File: LEDs.kicad_sch (KiCad schematic)
At the start: 31 parts

Commit message: update
Parts:
- D0, D1, D10, D11, D12, D13, D14, D15, D16, D17, D18, D19, D2, D20, D21, D22, D23, D24, D25, D26, D27, D28, D29, D3, D4, D5, D6, D7, D8, D9: footprint kicad-library:WS2812B_wider_pads -> easyeda2kicad:LED-SMD_4P-L5.0-W5.0-BL_XL-5050RGBC
Connections:
- net +5V renamed +5VP
Changed lines of the file:
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@@
 			)
 		)
-		(property "Footprint" "kicad-library:WS2812B_wider_pads"
+		(property "Footprint" "easyeda2kicad:LED-SMD_4P-L5.0-W5.0-BL_XL-5050RGBC"
 			(at 242.57 106.68 0)
 			(effects
@@
 			)
 		)
-		(property "Footprint" "kicad-library:WS2812B_wider_pads"
+		(property "Footprint" "easyeda2kicad:LED-SMD_4P-L5.0-W5.0-BL_XL-5050RGBC"
 			(at 255.27 109.22 0)
 			(effects
@@
 			)
 		)
-		(property "Footprint" "kicad-library:WS2812B_wider_pads"
+		(property "Footprint" "easyeda2kicad:LED-SMD_4P-L5.0-W5.0-BL_XL-5050RGBC"
 			(at 255.27 124.46 0)
 			(effects
@@
 			)
 		)
-		(property "Footprint" "kicad-library:WS2812B_wider_pads"
+		(property "Footprint" "easyeda2kicad:LED-SMD_4P-L5.0-W5.0-BL_XL-5050RGBC"
 			(at 255.27 139.7 0)
 			(effects
@@
 			)
 		)
-		(property "Footprint" "kicad-library:WS2812B_wider_pads"
+		(property "Footprint" "easyeda2kicad:LED-SMD_4P-L5.0-W5.0-BL_XL-5050RGBC"
 			(at 255.27 154.94 0)
 			(effects
@@
 			)
 		)
-		(property "Footprint" "kicad-library:WS2812B_wider_pads"
+		(property "Footprint" "easyeda2kicad:LED-SMD_4P-L5.0-W5.0-BL_XL-5050RGBC"
 			(at 255.27 170.18 0)
 			(effects
@@
 			)
 		)
-		(property "Footprint" "kicad-library:WS2812B_wider_pads"
+		(property "Footprint" "easyeda2kicad:LED-SMD_4P-L5.0-W5.0-BL_XL-5050RGBC"
 			(at 255.27 185.42 0)
 			(effects
@@
 			)
 		)
-		(property "Footprint" "kicad-library:WS2812B_wider_pads"
+		(property "Footprint" "easyeda2kicad:LED-SMD_4P-L5.0-W5.0-BL_XL-5050RGBC"
 			(at 298.45 182.88 0)
 			(effects
@@
 			)
 		)
-		(property "Footprint" "kicad-library:WS2812B_wider_pads"
+		(property "Footprint" "easyeda2kicad:LED-SMD_4P-L5.0-W5.0-BL_XL-5050RGBC"
 			(at 298.45 167.64 0)
 			(effects
@@
 			)
 		)
-		(property "Footprint" "kicad-library:WS2812B_wider_pads"
+		(property "Footprint" "easyeda2kicad:LED-SMD_4P-L5.0-W5.0-BL_XL-5050RGBC"
 			(at 298.45 152.4 0)
 			(effects
@@
 			)
 		)
-		(property "Footprint" "kicad-library:WS2812B_wider_pads"
+		(property "Footprint" "easyeda2kicad:LED-SMD_4P-L5.0-W5.0-BL_XL-5050RGBC"
 			(at 298.45 137.16 0)
 			(effects
@@
 			)
 		)
-		(property "Footprint" "kicad-library:WS2812B_wider_pads"
+		(property "Footprint" "easyeda2kicad:LED-SMD_4P-L5.0-W5.0-BL_XL-5050RGBC"
 			(at 298.45 121.92 0)
 			(effects
@@
 			)
 		)
-		(property "Footprint" "kicad-library:WS2812B_wider_pads"
+		(property "Footprint" "easyeda2kicad:LED-SMD_4P-L5.0-W5.0-BL_XL-5050RGBC"
 			(at 298.45 106.68 0)
 			(effects
@@
 			)
 		)
-		(property "Footprint" "kicad-library:WS2812B_wider_pads"
+		(property "Footprint" "easyeda2kicad:LED-SMD_4P-L5.0-W5.0-BL_XL-5050RGBC"
 			(at 311.15 109.22 0)
 			(effects
@@
 			)
 		)
-		(property "Footprint" "kicad-library:WS2812B_wider_pads"
+		(property "Footprint" "easyeda2kicad:LED-SMD_4P-L5.0-W5.0-BL_XL-5050RGBC"
 			(at 311.15 124.46 0)
 			(effects
@@
 			)
 		)
-		(property "Footprint" "kicad-library:WS2812B_wider_pads"
+		(property "Footprint" "easyeda2kicad:LED-SMD_4P-L5.0-W5.0-BL_XL-5050RGBC"
 			(at 311.15 139.7 0)
 			(effects
@@
 			)
 		)
-		(property "Footprint" "kicad-library:WS2812B_wider_pads"
+		(property "Footprint" "easyeda2kicad:LED-SMD_4P-L5.0-W5.0-BL_XL-5050RGBC"
 			(at 311.15 154.94 0)
 			(effects
@@
 			)
 		)
-		(property "Footprint" "kicad-library:WS2812B_wider_pads"
+		(property "Footprint" "easyeda2kicad:LED-SMD_4P-L5.0-W5.0-BL_XL-5050RGBC"
 			(at 311.15 170.18 0)
 			(effects
@@
 			)
 		)
-		(property "Footprint" "kicad-library:WS2812B_wider_pads"
+		(property "Footprint" "easyeda2kicad:LED-SMD_4P-L5.0-W5.0-BL_XL-5050RGBC"
 			(at 311.15 185.42 0)
 			(effects
@@
 			)
 		)
-		(property "Footprint" "kicad-library:WS2812B_wider_pads"
+		(property "Footprint" "easyeda2kicad:LED-SMD_4P-L5.0-W5.0-BL_XL-5050RGBC"
 			(at 354.33 182.88 0)
 			(effects
@@
 			)
 		)
-		(property "Footprint" "kicad-library:WS2812B_wider_pads"
+		(property "Footprint" "easyeda2kicad:LED-SMD_4P-L5.0-W5.0-BL_XL-5050RGBC"
 			(at 354.33 167.64 0)
 			(effects
@@
 			)
 		)
-		(property "Footprint" "kicad-library:WS2812B_wider_pads"
+		(property "Footprint" "easyeda2kicad:LED-SMD_4P-L5.0-W5.0-BL_XL-5050RGBC"
 			(at 354.33 152.4 0)
 			(effects
@@
 			)
 		)
-		(property "Footprint" "kicad-library:WS2812B_wider_pads"
+		(property "Footprint" "easyeda2kicad:LED-SMD_4P-L5.0-W5.0-BL_XL-5050RGBC"
 			(at 354.33 137.16 0)
 			(effects
@@
 			)
 		)
-		(property "Footprint" "kicad-library:WS2812B_wider_pads"
+		(property "Footprint" "easyeda2kicad:LED-SMD_4P-L5.0-W5.0-BL_XL-5050RGBC"
 			(at 354.33 121.92 0)
 			(effects
@@
 			)
 		)
-		(property "Footprint" "kicad-library:WS2812B_wider_pads"
+		(property "Footprint" "easyeda2kicad:LED-SMD_4P-L5.0-W5.0-BL_XL-5050RGBC"
 			(at 354.33 106.68 0)
 			(effects
@@
 			)
 		)
-		(property "Footprint" "kicad-library:WS2812B_wider_pads"
+		(property "Footprint" "easyeda2kicad:LED-SMD_4P-L5.0-W5.0-BL_XL-5050RGBC"
 			(at 242.57 152.4 0)
 			(effects
@@
 			)
 		)
-		(property "Value" "+5V"
+		(property "Value" "+5VP"
 			(at 332.74 189.23 0)
 			(effects
@@
 			)
 		)
-		(property "Value" "+5V"
-			(at 276.86 189.0196 0)
+		(property "Value" "+5VP"
+			(at 276.86 189.23 0)
 			(effects
 				(font
@@
 			)
 		)
-		(property "Footprint" "kicad-library:WS2812B_wider_pads"
+		(property "Footprint" "easyeda2kicad:LED-SMD_4P-L5.0-W5.0-BL_XL-5050RGBC"
 			(at 242.57 182.88 0)
 			(effects
@@
 			)
 		)
-		(property "Footprint" "kicad-library:WS2812B_wider_pads"
+		(property "Footprint" "easyeda2kicad:LED-SMD_4P-L5.0-W5.0-BL_XL-5050RGBC"
 			(at 242.57 121.92 0)
 			(effects
@@
 			)
 		)
-		(property "Value" "+5V"
-			(at 219.71 184.15 0)
-			(effects
-				(font
-					(size 1.27 1.27)
-				)
+		(property "Value" "+5VP"
+			(at 220.98 184.1499 90)
+			(effects
+				(font
+					(size 1.27 1.27)
+				)
+				(justify left)
 			)
 		)
@@
 			)
 		)
-		(property "Footprint" "kicad-library:WS2812B_wider_pads"
+		(property "Footprint" "easyeda2kicad:LED-SMD_4P-L5.0-W5.0-BL_XL-5050RGBC"
 			(at 242.57 137.16 0)
 			(effects
@@
 			)
 		)
-		(property "Value" "+5V"
+		(property "Value" "+5VP"
 			(at 374.65 129.54 0)
 			(effects
@@
 			)
 		)
-		(property "Footprint" "kicad-library:WS2812B_wider_pads"
+		(property "Footprint" "easyeda2kicad:LED-SMD_4P-L5.0-W5.0-BL_XL-5050RGBC"
 			(at 242.57 167.64 0)
 			(effects

Commit message: finished placing components
Parts:
- C31: footprint Capacitor_SMD:C_1206_3216Metric -> Capacitor_SMD:C_0603_1608Metric; LCSC Part C96123 -> C19702
Changed lines of the file:
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@@
 			)
 		)
-		(property "Footprint" "Capacitor_SMD:C_1206_3216Metric"
+		(property "Footprint" "Capacitor_SMD:C_0603_1608Metric"
 			(at 374.65 140.97 0)
 			(effects
@@
 			)
 		)
-		(property "LCSC Part" "C96123"
+		(property "LCSC Part" "C19702"
 			(at 374.65 140.97 0)
 			(effects
