File: Voided Oblivion.kicad_pcb (KiCad board)
At the start: 2 copper layers, 95.2 x 114.3 mm, 160 parts, among them J10 Conn_01x02, J13 Debug, J14 QWIIC, J6 TYPEC-304-ACP16, J8 RGB_LED_In, Q1 2N7002, Q2 AO3401A, Q3 AO3401A, SW1 TS24CA, SW2 TS24CA, U1 RP2350B, U105 MT9700, U28 W25Q128JVSIQ, Y1 3225_4P

Commit message: update
Parts:
- removed C1: 10u, Capacitor_SMD:C_0402_1005Metric
- removed C5: 100nF, Capacitor_SMD:C_0402_1005Metric
- removed D31: ZMMxx, Diode_SMD:D_MiniMELF
- removed DI2: B5819W, Diode_SMD:D_SOD-123
- removed F1: 500mA, Fuse:Fuse_0603_1608Metric
- removed FB1, FB2, FB4: 100 @ 100 MHz, Inductor_SMD:L_0805_2012Metric
- removed J6: TYPEC-304-ACP16, Connector_USB:USB_C_Receptacle_GCT_USB4105-xx-A_16P_TopMnt_Horizontal
- removed JP1: SolderJumper_2_Bridged, Jumper:SolderJumper-2_P1.3mm_Bridged_Pad1.0x1.5mm
- removed LDO2: AMS1117-3.3, Package_TO_SOT_SMD:SOT-223-3_TabPin2
- removed LED0: WS2812B, kicad-library:WS2812B_wider_pads
- removed Q1: 2N7002, Package_TO_SOT_SMD:SOT-23
- removed Q2, Q3: AO3401A, Package_TO_SOT_SMD:SOT-23
- removed R5: 1k, Resistor_SMD:R_0402_1005Metric
- removed SW1, SW2: TS24CA, kicad_misc_parts:SW-SMD_TS24CA
- removed U28: W25Q128JVSIQ, Package_SO:SOIC-8_5.23x5.23mm_P1.27mm
- removed Y1: 3225_4P, Crystal:Crystal_SMD_3225-4Pin_3.2x2.5mm
- added BT1: Battery_Cell, Connector_PinHeader_2.54mm:PinHeader_1x02_P2.54mm_Vertical, F.Cu at (188.9, 32.5)
- added BTN1: SW_Push, easyeda2kicad:SW-SMD_2P-TS24CA, F.Cu at (209.2, 25.2)
- added BTN2: SW_Push, easyeda2kicad:SW-SMD_2P-TS24CA, F.Cu at (202.6, 25.2)
- added C25: 1uf, Resistor_SMD:R_0402_1005Metric, F.Cu at (207.0, 58.5)
- added C26: 22uF, Capacitor_SMD:C_0201_0603Metric, F.Cu at (186.6, 60.2)
- added C27: 10nF, Capacitor_SMD:C_0402_1005Metric, F.Cu at (192.3, 58.2)
- added C28: 10pF, Capacitor_SMD:C_0201_0603Metric, F.Cu at (193.4, 61.0)
- added C29: 47uF, Capacitor_SMD:C_0805_2012Metric, F.Cu at (189.0, 57.8)
- added C30: 1uf, Resistor_SMD:R_0402_1005Metric, F.Cu at (205.0, 58.5)
- added D34: B5819W, Diode_SMD:D_SOD-123, F.Cu at (188.6, 52.7)
- added H1: MountingHole, MountingHole:MountingHole_3.2mm_M3_ISO14580_Pad, F.Cu at (132.7, 25.7)
- added H2: MountingHole, MountingHole:MountingHole_3.2mm_M3_ISO14580_Pad, F.Cu at (222.0, 25.7)
- added H3: MountingHole, MountingHole:MountingHole_3.2mm_M3_ISO14580_Pad, F.Cu at (132.7, 134.0)
- added H4: MountingHole, MountingHole:MountingHole_3.2mm_M3_ISO14580_Pad, F.Cu at (222.0, 134.0)
- added J1: Receive 1, kicad_misc_parts:Magnetis connenctor, F.Cu at (217.9, 79.9)
- added J2: Receive 2, kicad_misc_parts:Magnetis connenctor, F.Cu at (177.4, 29.8)
- added J3: Transmit 1, kicad_misc_parts:Magnetis connenctor, F.Cu at (136.7, 79.9)
- added J4: Transmit 1, kicad_misc_parts:spesial Magnetic connenctor, F.Cu at (177.4, 130.0)
- added J5: USB_C_Receptacle_USB2.0_16P, Connector_USB:USB_C_Receptacle_GCT_USB4105-xx-A_16P_TopMnt_Horizontal, F.Cu at (148.8, 26.4)
- added L2: 1uH, easyeda2kicad:IND-SMD_L5.4-W5.2_FXL0530, F.Cu at (189.4, 64.2)
- added R14: 1k, Resistor_SMD:R_0402_1005Metric, F.Cu at (203.4, 59.7)
- added R15: 2k, Resistor_SMD:R_0402_1005Metric, F.Cu at (203.7, 61.1)
- added R16: 1.5k, Resistor_SMD:R_0402_1005Metric, F.Cu at (206.0, 62.2)
- added R17: 1.5k, Resistor_SMD:R_0402_1005Metric, F.Cu at (209.0, 60.4)
- added R18: 316k, Resistor_SMD:R_0201_0603Metric, F.Cu at (192.8, 61.6)
- added R19: 100k, Resistor_SMD:R_0402_1005Metric, F.Cu at (193.9, 60.3)
- added U2: BQ24045DSQR, easyeda2kicad:WSON-10_L2.0-W2.0-P0.40-BL-EP, F.Cu at (206.0, 60.5)
- added U3: W25Q128JVS, easyeda2kicad:SOIC-8_L5.3-W5.3-P1.27-LS8.0-BL, F.Cu at (153.3, 42.0)
- added U4: ABM8-272-T3, easyeda2kicad:CRYSTAL-SMD_4P-L3.2-W2.5-BL, F.Cu at (168.4, 55.5)
- added U5: TPS61230ARNSR, easyeda2kicad:VQFN-7_L2.1-W2.1-P0.50-BL, F.Cu at (190.8, 59.4)
- C10, C6, C7, C9: value 100nF -> 4.7uf; moved to F.Cu
- C11, C12, C2: value 10u -> 100nf; moved to F.Cu
- C13, C14, C21, C8: value 100nF -> 100nf; moved to F.Cu
- C15: value 1µF -> 100nf; moved to F.Cu
- C16: value 1uf -> 100nf; moved to F.Cu
- C17, C20: value 4.7uf -> 100nf; moved to F.Cu
- C18: value 22pf 0402 -> 100nf; moved to F.Cu
- C19: value 22pf 0402 -> 10uf; footprint Capacitor_SMD:C_0402_1005Metric -> Capacitor_SMD:C_1206_3216Metric; moved to F.Cu
- C22: value 4.7uf -> 10u; moved to F.Cu
- C23: value 100nf -> 10u; moved to F.Cu
- C24: value 10nf -> 47u; footprint Capacitor_SMD:C_0402_1005Metric -> Capacitor_SMD:C_0603_1608Metric; moved to F.Cu
- C3: value 47u -> 15pf; footprint Capacitor_SMD:C_1206_3216Metric -> Capacitor_SMD:C_0402_1005Metric; moved to F.Cu
- C31, D30, ESD1, F2, FB3, J10, J13, J14, J8, LDO1, R13, U1, U105: moved to F.Cu
- C39: value 10u -> 10uf; moved to F.Cu
- C4: value 100nF -> 15pf; moved to F.Cu
- D0, D1, D10, D11, D12, D13, D14, D15, D16, D17, D18, D19, D2, D20, D21, D22, D23, D24, D25, D26, D27, D28, D29, D3, D4, D5, D6, D7, D8, D9: footprint kicad-library:WS2812B_wider_pads -> easyeda2kicad:LED-SMD_4P-L5.0-W5.0-BL_XL-5050RGBC
- L1: value 3.3u -> 3.3uH; footprint kicad_misc_parts:INDM3225X210N -> easyeda2kicad:IND-SMD_L4.0-W4.0; moved to F.Cu
- R1: value 2k2 -> DNF; moved to F.Cu
- R10: value 33Ω -> 0; footprint Resistor_SMD:R_0603_1608Metric -> Resistor_SMD:R_0402_1005Metric; moved to F.Cu
- R11: value 1K -> 5k; moved to F.Cu
- R12: value 330k -> 5k; moved to F.Cu
- R2: value 2k2 -> 1k; moved to F.Cu
- R3: value 5k1 -> 33Ω; moved to F.Cu
- R4: value 5k1 -> 1k; moved to F.Cu
- R6: value 330k -> 1k; moved to F.Cu
- R7, R8: footprint Resistor_SMD:R_0603_1608Metric -> Resistor_SMD:R_0402_1005Metric; moved to F.Cu
- R9: value 1k -> DNF; moved to F.Cu
- moved J10 164.1 mm to (46.7, 24.3), turned to 0 degrees
- moved C24 157.5 mm to (36.5, 44.4), turned to 0 degrees
- moved J13 156.0 mm to (23.5, 24.3), turned to 0 degrees
- moved R12 146.0 mm to (41.8, 40.2), turned to 0 degrees
- moved C9 140.7 mm to (22.6, 47.5), turned to 0 degrees
- moved C7 138.3 mm to (22.6, 43.6), turned to 0 degrees
- moved R11 135.0 mm to (41.8, 38.2), turned to 0 degrees
- moved R13 123.0 mm to (81.9, 64.5)
- moved U105 118.0 mm to (84.5, 64.0), turned to 0 degrees
- moved C31 114.8 mm to (24.0, 55.0)
- moved C39 113.0 mm to (87.1, 63.5)
- moved ESD1 108.1 mm to (41.5, 45.6)
- moved C19 107.4 mm to (70.3, 36.6), turned to 0 degrees
- moved J8 100.5 mm to (32.1, 39.0), turned to 0 degrees
- moved J14 91.0 mm to (98.2, 40.7), turned to 0 degrees
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- renumbered AM1:2 to AM1:0, AM1:0 to AM1:2, AM1:5 to AM1:3, AM1:3 to AM1:5, H1:2 to H1:0, H1:0 to H1:2
Connections:
- net Net-(U1-VREG_LX) renamed VREG LX
- net SWDIO renamed SWD
- C10 pad 1: +3V3 -> +1V1
- C11 pad 1: Net-(LDO2-VI) -> +1V1
- C15 pad 1: +3.3VA -> +3V3
- C16 pad 1: +1V1 -> +3V3
- C17 pad 1: Net-(U1-VREG_AVDD) -> +3V3
- C18 pad 1: GND -> +3V3
- C18 pad 2: XIN -> GND
- C19 pad 1: GND -> +3V3
- C19 pad 2: Net-(C19-Pad2) -> GND
- C2 pad 1: Net-(LDO1-VO) -> +3V3
- C20 pad 2: Net-(U1-VREG_PGND) -> GND
- C22 pad 1: +1V1 -> Net-(LDO1-VI)
- C22 pad 2: Net-(U1-VREG_PGND) -> GND
- C23 pad 1: +3.3VA -> +3V3
- C24 pad 1: +3.3VA -> +5V
- C3 pad 1: +5V -> GND
- C3 pad 2: GND -> XIN
- C31 pad 1: +5V -> +5VP
- C4 pad 1: +1V1 -> Net-(C4-Pad1)
- C7 pad 1: +3V3 -> +1V1
- C8 pad 1: +3V3 -> +1V1
- C9 pad 1: +3V3 -> VREG AVDD
- D0 pad 1: +5V -> +5VP
- D1 pad 1: +5V -> +5VP
- D10 pad 1: +5V -> +5VP
- D11 pad 1: +5V -> +5VP
- D12 pad 1: +5V -> +5VP
- D13 pad 1: +5V -> +5VP
- D14 pad 1: +5V -> +5VP
- D15 pad 1: +5V -> +5VP
- D16 pad 1: +5V -> +5VP
- D17 pad 1: +5V -> +5VP
- D18 pad 1: +5V -> +5VP
- D19 pad 1: +5V -> +5VP
- D2 pad 1: +5V -> +5VP
- D20 pad 1: +5V -> +5VP
- D21 pad 1: +5V -> +5VP
- D22 pad 1: +5V -> +5VP
- D23 pad 1: +5V -> +5VP
- D24 pad 1: +5V -> +5VP
- D25 pad 1: +5V -> +5VP
- D26 pad 1: +5V -> +5VP
- D27 pad 1: +5V -> +5VP
- D28 pad 1: +5V -> +5VP
- D29 pad 1: +5V -> +5VP
- D3 pad 1: +5V -> +5VP
- D30 pad 2: +5VD -> +5VP
- D4 pad 1: +5V -> +5VP
- D5 pad 1: +5V -> +5VP
- D6 pad 1: +5V -> +5VP
- D7 pad 1: +5V -> +5VP
- D8 pad 1: +5V -> +5VP
- D9 pad 1: +5V -> +5VP
- FB3 pad 1: Net-(LDO2-VI) -> Net-(LDO1-VI)
- H1:0 pad 2: AM1:2 -> AM1:0
- H1:2 pad 2: AM1:0 -> AM1:2
- LDO1 pad 2: Net-(LDO1-VO) -> +3V3
- R1 pad 2: SCL -> FLASH SS
- R10 pad 1: Net-(U1-VREG_AVDD) -> QSPI SS
- R10 pad 2: +3V3 -> FLASH SS
- R11 pad 1: XOUT -> DATA_CC1
- R11 pad 2: Net-(C19-Pad2) -> GND
- R12 pad 1: Net-(Q2-S) -> DATA_CC2
- R12 pad 2: Net-(Q1-D) -> GND
- R2 pad 1: +3V3 -> Net-(C4-Pad1)
- R2 pad 2: SDA -> XOUT
- R3 pad 1: DATA_CC1 -> +3V3
- R3 pad 2: GND -> VREG AVDD
- R4 pad 1: DATA_CC2 -> GND
- R4 pad 2: GND -> Net-(BTN2-Pad1)
- R6 pad 1: GND -> USB BOOT
- R6 pad 2: +5VP -> QSPI SS
- R7 pad 1: USB_D+ -> Net-(U1-USB_DP)
- R7 pad 2: Net-(U1-USB_DP) -> USB D+
- R8 pad 1: USB_D- -> Net-(U1-USB_DM)
- R8 pad 2: Net-(U1-USB_DM) -> USB D-
- R9 pad 1: /~{USB_BOOT} -> GPIO0
- R9 pad 2: QSPI_SS -> FLASH SS
- U1 pad 17: RGB_LED_MCU -> RGB_LED
- U1 pad 20: EXT_PWR_EN -> BAT_EN
- U1 pad 21: unconnected-(U1-GPIO21-Pad21) -> BAT_H/L
- U1 pad 22: unconnected-(U1-GPIO22-Pad22) -> BAT_PWR_EN
- U1 pad 23: unconnected-(U1-GPIO23-Pad23) -> BAT_PWR_GOOD?
- U1 pad 25: unconnected-(U1-GPIO24-Pad25) -> BAT_CHG_STAT
- U1 pad 53: GND -> Net-(U1-GPIO42_ADC2)
- U1 pad 54: GND -> Net-(U1-GPIO42_ADC2)
- U1 pad 55: GND -> unconnected-(U1-GPIO44_ADC4-Pad55)
- U1 pad 56: GND -> unconnected-(U1-GPIO45_ADC5-Pad56)
- U1 pad 57: GND -> unconnected-(U1-GPIO46_ADC6-Pad57)
- U1 pad 58: GND -> unconnected-(U1-GPIO47_ADC7-Pad58)
- U1 pad 59: +3.3VA -> +3V3
- U1 pad 61: Net-(U1-VREG_AVDD) -> VREG AVDD
- U1 pad 62: Net-(U1-VREG_PGND) -> GND
- U1 pad 70: SD3 -> QSPI SD3
- U1 pad 71: QSPI_CLK -> QSPI SCLK
- U1 pad 72: SD0 -> QSPI SD0
- U1 pad 73: SD2 -> QSPI SD2
- U1 pad 74: SD1 -> QSPI SD1
- U1 pad 75: QSPI_SS -> QSPI SS
- U1 pad 77: unconnected-(U1-GPIO0-Pad77) -> GPIO0
- U105 pad 4: EXT_PWR_EN -> 5V_PWR_EN
Routing:
- net RGB_LED_SIG: track 95.2 -> 0.00 mm, vias 1 -> 0
- net RGB_LED_MCU: track 70.5 -> 0.00 mm, vias 2 -> 0
- net +5VD: track 67.8 -> 0.00 mm
- net BAT_CHG_STAT: track 0.00 -> 65.8 mm, vias 0 -> 2
- net BAT_EN: track 0.00 -> 64.8 mm, vias 0 -> 2
- net +BATT: track 0.00 -> 63.9 mm, vias 0 -> 3
- net +3V3: track 149.0 -> 91.2 mm, vias 14 -> 5
- net BAT_H/L: track 0.00 -> 57.6 mm, vias 0 -> 2
- net BAT_PWR_GOOD?: track 0.00 -> 54.8 mm, vias 0 -> 2
- net GND: track 90.3 -> 38.1 mm, vias 33 -> 44
- net QSPI SS: track 0.00 -> 49.9 mm, vias 0 -> 2
- net VBUS: track 51.2 -> 1.39 mm, vias 4 -> 0
- net BAT_PWR_EN: track 0.00 -> 46.4 mm, vias 0 -> 4
- net AM1:2: track 50.6 -> 8.71 mm
- net AM1:0: track 8.18 -> 48.4 mm
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- added copper zone on F.Cu, net +3V3
- added copper zone on F.Cu, net +BATT
- added copper zone on F.Cu, net Net-(D34-A)
- added copper zone on F.Cu, net Net-(U5-CBST)
- added copper zone on F.Cu, net Net-(U5-FB)
- added copper zone on F.Cu, net Net-(U5-SW)
- removed copper zone on B.Cu, net +3V3
Other:
- board text removed: "GND 5V+"

Commit message: finished placing components
Parts:
- removed J8: RGB_LED_In, Connector_PinHeader_2.54mm:PinHeader_1x03_P2.54mm_Vertical
- added C5: 100nf, Capacitor_SMD:C_0402_1005Metric, F.Cu at (148.0, 51.6)
- added PSW1: MSK12C02, easyeda2kicad:SW-TH_MSK12C02, F.Cu at (205.9, 133.5)
- added R20: 0Ω, Resistor_SMD:R_0402_1005Metric, F.Cu at (163.6, 32.9)
- added R5: 10k, Resistor_SMD:R_0402_1005Metric, F.Cu at (146.5, 43.3)
- added U6: W25Q128JVS, easyeda2kicad:SOIC-8_L5.3-W5.3-P1.27-LS8.0-BL, F.Cu at (151.0, 47.9)
- C31: footprint Capacitor_SMD:C_1206_3216Metric -> Capacitor_SMD:C_0603_1608Metric
- J13: footprint Connector_PinHeader_2.54mm:PinHeader_1x05_P2.54mm_Horizontal -> Connector_PinHeader_2.54mm:PinHeader_1x05_P2.54mm_Vertical
- R10: value 0 -> 0Ω
- moved C31 172.2 mm to (195.7, 41.7), turned to 90 degrees
- moved J13 162.9 mm to (177.0, 78.9), turned to -90 degrees
- moved J10 159.6 mm to (206.0, 34.7)
- moved C7 156.4 mm to (179.0, 43.1), turned to 90 degrees
- moved C24 155.8 mm to (192.4, 41.7), turned to 90 degrees
- moved C9 154.9 mm to (177.2, 37.5)
- moved R13 110.6 mm to (191.0, 46.5), turned to -90 degrees
- moved R11 110.1 mm to (151.8, 32.7), turned to -90 degrees
- moved ESD1 107.9 mm to (148.7, 33.2), turned to 180 degrees
- moved U105 105.3 mm to (188.4, 47.0), turned to 180 degrees
- moved R12 101.7 mm to (142.8, 28.0), turned to -90 degrees
- moved C39 100.1 mm to (185.8, 47.5), turned to 90 degrees
- moved R3 90.4 mm to (176.5, 38.6), turned to 180 degrees
- moved C19 90.0 mm to (159.8, 46.2), turned to 180 degrees
- moved J14 55.0 mm to (149.8, 59.6)
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- renumbered BT1 to B1
Connections:
- C24 pad 1: +5V -> +5VP
- C26 pad 1: +BATT -> Net-(U5-VIN)
- ESD1 pad 1: USB_D- -> USB D-
- ESD1 pad 6: USB_D+ -> USB D+
- J10 pad 2: +5V -> +5VP
- J5 pad A6: USB_D+ -> USB D+
- J5 pad A7: USB_D- -> USB D-
- J5 pad B6: USB_D+ -> USB D+
- J5 pad B7: USB_D- -> USB D-
- L2 pad 1: +BATT -> Net-(U5-VIN)
- U1 pad 45: unconnected-(U1-GPIO36-Pad45) -> 5V_PWR_EN
- U5 pad 4: +BATT -> Net-(U5-VIN)
Routing:
- net Net-(U5-VIN): track 0.00 -> 80.6 mm, vias 0 -> 4
- net USB D+: track 0.00 -> 40.0 mm
- net SWD: track 0.00 -> 34.4 mm
- net USB D-: track 0.00 -> 34.2 mm, vias 0 -> 2
- net SWCLK: track 0.00 -> 33.5 mm
- net RUN: track 48.4 -> 81.7 mm, vias 4 -> 5
- net SDA: track 0.00 -> 30.9 mm, vias 0 -> 2
- net SCL: track 0.00 -> 27.9 mm, vias 0 -> 2
- net FLASH2 SS: track 0.00 -> 25.5 mm, vias 0 -> 2
- net +BATT: track 63.9 -> 78.6 mm, vias 3 -> 4
- net 5V_PWR_EN: track 0.00 -> 13.3 mm, vias 0 -> 2
- net +5VP: track 0.00 -> 12.2 mm
- net VBUS: track 1.39 -> 12.2 mm, vias 0 -> 2
- net QSPI SD3: track 25.9 -> 34.9 mm
- net QSPI SCLK: track 25.4 -> 34.3 mm
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- added copper zone on F.Cu, net Net-(U5-VIN)
- removed copper zone on F.Cu, net +BATT
Other:
- board text added: "5V+"
- board text added: "BAT+"
- board text added: "GND"

Commit message: schematic done?
Parts:
- moved D1 1.19 mm to (139.3, 108.5)
Routing:
- net +3.3VA: track 0.00 -> 104.5 mm
- net +5VP: track 12.2 -> 116.4 mm
- net +BATT: track 78.6 -> 110.5 mm
- net Net-(D10-DOUT): track 0.00 -> 25.3 mm
- net Net-(D2-DOUT): track 0.00 -> 14.0 mm
- net Net-(D1-DOUT): track 0.00 -> 14.0 mm
- net Net-(D0-DOUT): track 0.00 -> 14.0 mm
- net Net-(D4-DOUT): track 0.00 -> 14.0 mm
- net Net-(D3-DOUT): track 0.00 -> 14.0 mm
