File: Voided Oblivion.kicad_sch (KiCad schematic)
At the start: 81 parts, among them IC1 XL1509-5.0E1, J1 Receive 1, J10 Conn_01x02, J13 Debug, J14 QWIIC, J2 Receive 2, J3 Transmit 1, J4 Transmit 1, J5 5V_Barrel, J6 TYPEC-304-ACP16, J8 RGB_LED_In, Q1 2N7002, Q2 AO3401A, Q3 AO3401A, SW1 TS24CA, SW2 TS24CA, U1 RP2350B, U105 MT9700, U28 W25Q128JVSIQ, Y1 3225_4P

Commit message: update
Parts:
- removed C1, C2: 10u, Capacitor_SMD:C_0402_1005Metric, symbol Device:C_Small
- removed C10, C13, C14, C21, C4, C5, C6, C7, C8, C9: 100nF, Capacitor_SMD:C_0402_1005Metric, symbol Device:C_Small
- removed C15: 1µF, Capacitor_SMD:C_0402_1005Metric, symbol Device:C_Small
- removed C16: 1uf, Capacitor_SMD:C_0402_1005Metric, symbol Device:C_Small
- removed C17, C20, C22: 4.7uf, Capacitor_SMD:C_0402_1005Metric, symbol Device:C_Small
- removed C18: 22pf 0402, Capacitor_SMD:C_0402_1005Metric, symbol Device:C_Small
- removed C23: 100nf, Capacitor_SMD:C_0402_1005Metric, symbol Device:C_Small
- removed C24: 10nf, Capacitor_SMD:C_0402_1005Metric, symbol Device:C_Small
- removed C25: 470uF, Capacitor_SMD:C_Elec_10x10.2, symbol Device:C_Polarized_Small_US
- removed C27: 220uF, kicad_misc_parts:CAP-SMD_BD6.3-L6.6-W6.6-LS7.2-R-RD, symbol Device:C_Polarized_Small_US
- removed D31: ZMMxx, Diode_SMD:D_MiniMELF, symbol Diode:ZMMxx
- removed D89: SK34WA, kicad_misc_parts:SOD-123F_L2.8-W1.8-LS3.7-RD, symbol Device:D_Schottky
- removed D95: Display, Connector_PinSocket_2.54mm:PinSocket_1x08_P2.54mm_Vertical, symbol Connector_Generic:Conn_01x08
- removed DI2: B5819W, Diode_SMD:D_SOD-123, symbol Device:D_Schottky_Small
- removed F1: 500mA, Fuse:Fuse_0603_1608Metric, symbol Device:Fuse_Small
- removed FB1, FB2: 100 @ 100 MHz, Inductor_SMD:L_0805_2012Metric, symbol Device:FerriteBead_Small
- removed FB4: 100 @ 100 MHz, Inductor_SMD:L_0805_2012Metric, symbol Device:Ferrite_Bead_Small
- removed IC1: XL1509-5.0E1, Package_SO:SOIC-8_3.9x4.9mm_P1.27mm, symbol XL1509-5.0E1:XL1509-5.0E1
- removed J5: 5V_Barrel, kicad_misc_parts:DC-IN-TH_DC-470-2.1GP, symbol Connector:Barrel_Jack_Switch
- removed J6: TYPEC-304-ACP16, kicad_misc_parts:TYPEC-304-ACP16, symbol Connector:USB_C_Receptacle_USB2.0
- removed JP1: SolderJumper_2_Bridged, Jumper:SolderJumper-2_P1.3mm_Bridged_Pad1.0x1.5mm, symbol Jumper:SolderJumper_2_Bridged
- removed L2: 2A 6uH, kicad_misc_parts:IND-SMD_L11.5-W10.0_SMMS1040, symbol Device:L_Small
- removed LDO1: AMS1117-3.3, Package_TO_SOT_SMD:SOT-223-3_TabPin2, symbol Regulator_Linear:AMS1117-3.3
- removed LED0: WS2812B, kicad-library:WS2812B_wider_pads, symbol LED:WS2812B
- removed Q1: 2N7002, Package_TO_SOT_SMD:SOT-23, symbol Transistor_FET:2N7002
- removed Q2, Q3: AO3401A, Package_TO_SOT_SMD:SOT-23, symbol Transistor_FET:AO3401A
- removed R1, R2: 2k2, Resistor_SMD:R_0402_1005Metric, symbol Device:R_Small
- removed R11: 1K, Resistor_SMD:R_0402_1005Metric, symbol Device:R_Small
- removed R12, R6: 330k, Resistor_SMD:R_0402_1005Metric, symbol Device:R_Small
- removed R5, R9: 1k, Resistor_SMD:R_0402_1005Metric, symbol Device:R_Small
- removed SW1, SW2: TS24CA, kicad_misc_parts:SW-SMD_TS24CA, symbol Switch:SW_Push
- removed U28: W25Q128JVSIQ, Package_SO:SOIC-8_5.23x5.23mm_P1.27mm, symbol Memory_Flash:W25Q128JVS
- removed Y1: 3225_4P, Crystal:Crystal_SMD_3225-4Pin_3.2x2.5mm, symbol Device:Crystal_GND24
- added BT1: Battery_Cell, Connector_PinHeader_2.54mm:PinHeader_1x02_P2.54mm_Vertical, symbol Device:Battery_Cell
- added BTN1, BTN2: SW_Push, easyeda2kicad:SW-SMD_2P-TS24CA, symbol Switch:SW_Push_Shielded
- added C10, C6, C7, C9: 4.7uf, Capacitor_SMD:C_0402_1005Metric, symbol Device:C
- added C11, C12, C13, C14, C15, C16, C17, C18, C2, C20, C21, C8: 100nf, Capacitor_SMD:C_0402_1005Metric, symbol Device:C
- added C25, C30: 1uf, Resistor_SMD:R_0402_1005Metric, symbol Device:C
- added C27: 10nF, Capacitor_SMD:C_0402_1005Metric, symbol Device:C_Small
- added C28: 10pF, Capacitor_SMD:C_0201_0603Metric, symbol Device:C_Small
- added C29: 47uF, Capacitor_SMD:C_0805_2012Metric, symbol Device:C_Small
- added C3, C4: 15pf, Capacitor_SMD:C_0402_1005Metric, symbol Device:C
- added D34: B5819W, Diode_SMD:D_SOD-123, symbol Device:D_Schottky_Small
- added H1, H2, H3, H4: MountingHole, MountingHole:MountingHole_3.2mm_M3_ISO14580_Pad, symbol Mechanical:MountingHole
- added J5: USB_C_Receptacle_USB2.0_16P, Connector_USB:USB_C_Receptacle_GCT_USB4105-xx-A_16P_TopMnt_Horizontal, symbol Connector:USB_C_Receptacle_USB2.0_16P
- added L2: 1uH, easyeda2kicad:IND-SMD_L5.4-W5.2_FXL0530, symbol Device:L
- added R1, R9: DNF, Resistor_SMD:R_0402_1005Metric, symbol Device:R
- added R14: 1k, Resistor_SMD:R_0402_1005Metric, symbol Device:R_Small
- added R15: 2k, Resistor_SMD:R_0402_1005Metric, symbol Device:R_Small
- added R16, R17: 1.5k, Resistor_SMD:R_0402_1005Metric, symbol Device:R_Small
- added R18: 316k, Resistor_SMD:R_0201_0603Metric, symbol Device:R_Small
- added R19: 100k, Resistor_SMD:R_0402_1005Metric, symbol Device:R_Small
- added R2, R4, R6: 1k, Resistor_SMD:R_0402_1005Metric, symbol Device:R
- added R3: 33Ω, Resistor_SMD:R_0402_1005Metric, symbol Device:R
- added U2: BQ24045DSQR, easyeda2kicad:WSON-10_L2.0-W2.0-P0.40-BL-EP, symbol easyeda2kicad:BQ24045DSQR
- added U3: W25Q128JVS, easyeda2kicad:SOIC-8_L5.3-W5.3-P1.27-LS8.0-BL, symbol Memory_Flash:W25Q128JVS
- added U4: ABM8-272-T3, easyeda2kicad:CRYSTAL-SMD_4P-L3.2-W2.5-BL, symbol easyeda2kicad:ABM8-272-T3_C20625731
- added U5: TPS61230ARNSR, easyeda2kicad:VQFN-7_L2.1-W2.1-P0.50-BL, symbol easyeda2kicad:TPS61230ARNSR
- C19: value 22pf 0402 -> 10uf; footprint Capacitor_SMD:C_0402_1005Metric -> Capacitor_SMD:C_1206_3216Metric; Basic Part (none) -> True; LCSC C1555 -> (none); LCSC Part (none) -> C15525
- C24: renamed from C3; footprint Capacitor_SMD:C_1206_3216Metric -> Capacitor_SMD:C_0603_1608Metric; LCSC Part C96123 -> C19702
- C26: value 1uF -> 22uF; footprint Capacitor_SMD:C_0603_1608Metric -> Capacitor_SMD:C_0201_0603Metric; Basic Part (none) -> True; LCSC C15849 -> (none); LCSC Part (none) -> C77042; Value2 (none) -> 1mΩ; now fitted; now in the parts list
- C39: value 10u -> 10uf
- J1, J2, J3: footprint Connector_PinSocket_2.54mm:PinSocket_1x04_P2.54mm_Vertical -> kicad_misc_parts:Magnetis connenctor; now fitted; now in the parts list
- J4: footprint Connector_PinSocket_2.54mm:PinSocket_1x04_P2.54mm_Vertical -> kicad_misc_parts:spesial Magnetic connenctor; now fitted; now in the parts list
- L1: value 3.3u -> 3.3uH; footprint kicad_misc_parts:INDM3225X210N -> easyeda2kicad:IND-SMD_L4.0-W4.0; LCSC Part (none) -> C602030
- R10: value 33Ω -> 0; footprint Resistor_SMD:R_0603_1608Metric -> Resistor_SMD:R_0402_1005Metric; LCSC C25190 -> (none); LCSC Part (none) -> C17168
- R11: renamed from R3; value 5k1 -> 5k
- R12: renamed from R4; value 5k1 -> 5k
- R7: footprint Resistor_SMD:R_0603_1608Metric -> Resistor_SMD:R_0402_1005Metric; LCSC C25190 -> (none); LCSC Part (none) -> C25100
- R8: footprint Resistor_SMD:R_0603_1608Metric -> Resistor_SMD:R_0402_1005Metric; LCSC C25190 -> (none)
- renumbered C11 to C22, C12 to C23, LDO2 to LDO1
Connections:
- net +5VD is gone; now on net +5VP: D30.2 (A)
- net QSPI_SS is gone; now on net QSPI SS: U1.75 (QSPI_SS)
- net RGB_LED_MCU is gone; now on net RGB_LED: U1.17 (GPIO17)
- net +1V1: now also C10.1, C11.1, C7.1, C8.1
- net +3.3VA: no longer U1.59 (ADC_AVDD)
- net +3V3: now also C19.1, U1.59 (ADC_AVDD), C12.1, C13.1, C14.1, C15.1, C16.1, C17.1, C18.1, C2.1, C20.1, C21.1, C6.1, R1.1, R3.1, U3.8 (VCC); no longer R10.2
- net +5V: now also D34.1 (K)
- net DATA_CC1: now also J5.A5 (CC1)
- net DATA_CC2: now also J5.B5 (CC2)
- net GND: now also C19.2, U1.62 (VREG_PGND), BT1.1 (-), BTN1.1, BTN1.SH (B), BTN2.SH (B), C10.2, C11.2, C12.2, C13.2, C14.2, C15.2, C16.2, C17.2, C18.2, C2.2, C20.2, C21.2, C25.2, C29.2, C3.1, C30.2, C4.2, C6.2, C7.2, C8.2, C9.2, J5.A1 (GND), J5.A12 (GND), J5.B1 (GND), J5.B12 (GND), J5.S1 (SHIELD), R14.1, R15.1, R19.1, R4.1, U2.11 (EP), U2.3 (VSS), U3.4 (GND), U4.2 (GND), U4.4 (GND), U5.6 (GND); no longer C19.1, U1.53 (GPIO42_ADC2), U1.54 (GPIO43_ADC3), U1.55 (GPIO44_ADC4), U1.56 (GPIO45_ADC5), U1.57 (GPIO46_ADC6), U1.58 (GPIO47_ADC7)
- net RUN: now also BTN2.2
- net USB_D+: now also J5.A6 (D+), J5.B6 (D+); no longer R7.1
- net USB_D-: now also J5.A7 (D-), J5.B7 (D-); no longer R8.1
- net VBUS: now also C30.1, J5.A4 (VBUS), J5.A9 (VBUS), J5.B4 (VBUS), J5.B9 (VBUS), U2.1 (IN)
- net XIN: now also C3.2, U4.1
- net XOUT: now also R2.2
- net at U1.66 (USB_DM): now also R8.1; no longer R8.2
- net at U1.67 (USB_DP): now also R7.1; no longer R7.2
- net QSPI SS: now reaches R10.1
- net QSPI SS: now also R6.2; no longer U1.61 (VREG_AVDD)
- net VREG LX: now reaches L1.2, U1.63 (VREG_LX)
- net BAT_H/L: now reaches U1.21 (GPIO21)
- net BAT_H/L: now also U2.7 (ISET2)
- net BAT_PWR_EN: now reaches U1.22 (GPIO22)
- net BAT_PWR_EN: now also U5.2 (EN)
- net BAT_PWR_GOOD?: now reaches U1.23 (GPIO23)
- net BAT_PWR_GOOD?: now also R16.2, U2.5 (~{PG})
- net BAT_CHG_STAT: now reaches U1.25 (GPIO24)
- net BAT_CHG_STAT: now also R17.2, U2.8 (~{CHG})
- net GPIO0: now reaches U1.77 (GPIO0)
- net GPIO0: now also R9.1
- net EXT_PWR_EN renamed 5V_PWR_EN
- net 5V_PWR_EN: no longer U1.20 (GPIO20)
- net QSPI_CLK renamed QSPI SCLK
- net QSPI SCLK: now also U3.6 (CLK)
- net SD0 renamed QSPI SD0
- net QSPI SD0: now also U3.5 (DI/IO_{0})
- net SD1 renamed QSPI SD1
- net QSPI SD1: now also U3.2 (DO/IO_{1})
- net SD2 renamed QSPI SD2
- net QSPI SD2: now also U3.3 (~{WP}/IO_{2})
- net SD3 renamed QSPI SD3
- net QSPI SD3: now also U3.7 (~{HOLD}/~{RESET}/IO_{3})
- net SWDIO renamed SWD
- net VCC renamed +BATT
- net +BATT: now also BT1.2 (+), C25.1, L2.1, R16.1, R17.1, U2.10 (OUT), U5.4 (VIN)
- new net: BTN2.1, R4.2
- new net: C28.1, C29.1, D34.2 (A), R18.2, U5.7 (VOUT)
- new net: R14.2, U2.2 (ISET)
- new net: R15.2, U2.4 (PRETERM)
- new net: C4.1, R2.1, U4.3
- new net: C28.2, R18.1, R19.2, U5.3 (FB)
- new net: C27.1, L2.2, U5.5 (SW)
- new net: C27.2, U5.1 (CBST)
- new net: U1.53 (GPIO42_ADC2), U1.54 (GPIO43_ADC3)
- new net BAT_EN: U1.20 (GPIO20), U2.9 (TS)
- new net FLASH SS: R1.2, R10.2, R9.2, U3.1 (~{CS})
- new net USB BOOT: BTN1.2, R6.1
- new net USB D+: R7.2
- new net USB D-: R8.2
- new net VREG AVDD: C9.1, R3.2, U1.61 (VREG_AVDD)
Other:
- note added: "+5VP = 5V protected"
- note added: "12MHz Crystal"
- note added: "5V (from bat)"
- note added: "Battery managment"
- note added: "Decoupling caps, put one close to each +3v3 pin on the rp2350b"
- note added: "If you're that weird guy reviewing this, can you check the data sheet to see if i did this right, ti short hand confuses me."
- note added: "Make sure R7 and R8 are close to the rp2350b"
- note added: "Parts done"
- note added: "Primary Flash"
- note added: "Secondary Flash?"
- note removed: ""Fake" LED"
- note removed: ""Sacrificial LED": Diode drops the input voltage to approx 4v so the 3.3V signal from the MCU can work reliably. NOTE: Isn't really visibly noticeable."
- note removed: "+3.3VA should be used to power all analog components"
- note removed: "+5V is one half of the LEDs +5VL is for the other half"
- note removed: "+5VD is power-selected power +5V is primary 5V source +5VP is primary after reverse current protection IC +5VL is secondary 5V source (for 1/2 LEDs) VCC is barrel jack (external) power VBUS is USB C power"
- note removed: "5-20V Input"
- note removed: "Analog 3.3V LDO"
- note removed: "BUSY/BL"
- note removed: "Barrel Jack Power"
- note removed: "CLK"
- note removed: "CS"
- note removed: "Crystal"
- note removed: "DC"
- note removed: "DIN"
- note removed: "Display"
- note removed: "Dual 5V @2A Max Buck Converters"
- note removed: "I2C Pullups"
- note removed: "LED In/Out Swap Jumper"
- note removed: "Make sure C15 is close to pin 44 (VREG_IN) of RP2040"
- note removed: "Make sure C16 is close to pin 45 of RP2040"
- note removed: "Make sure these resistors are close to RP2040"
- note removed: "PWR_SENSE goes floating when external power is connected"
- note removed: "Power Selection"
- note removed: "QSPI Flash"
- note removed: "REQUIRED TO USE LEDS!"
- note removed: "RGB LED Stuff"
- note removed: "RST"
- note removed: "Reset Switch"
- note removed: "These decoupling capacitors are meant to be put close by each 3.3V pin of the RP2040"
- note removed: "Using a 12MHz because that's what you're supposed to use"
- note removed: "When VBUS is selected there's a 0.2V voltage drop because of the diodes inside the MOSFETS"
- moved on the sheet: AM0, AM1, C22, C23, C24, D30, F2, FB3, LDO1

Commit message: finished placing components
Parts:
- removed J8: RGB_LED_In, Connector_PinHeader_2.54mm:PinHeader_1x03_P2.54mm_Vertical, symbol Connector_Generic:Conn_01x03
- added C5: 100nf, Capacitor_SMD:C_0402_1005Metric, symbol Device:C
- added PSW1: MSK12C02, easyeda2kicad:SW-TH_MSK12C02, symbol easyeda2kicad:MSK12C02
- added R20: 0Ω, Resistor_SMD:R_0402_1005Metric, symbol Device:R
- added R5: 10k, Resistor_SMD:R_0402_1005Metric, symbol Device:R
- added U6: W25Q128JVS, easyeda2kicad:SOIC-8_L5.3-W5.3-P1.27-LS8.0-BL, symbol Memory_Flash:W25Q128JVS
- C24: MPN CL31A476MPHNNNE -> (none)
- J13: footprint Connector_PinHeader_2.54mm:PinHeader_1x05_P2.54mm_Horizontal -> Connector_PinHeader_2.54mm:PinHeader_1x05_P2.54mm_Vertical
- R1, R9: now left out of the parts list
- R10: value 0 -> 0Ω
- U3: LCSC Part (none) -> C97521
- renumbered BT1 to B1
Connections:
- net USB_D+ is gone; now on net USB D+: ESD1.6 (IO4), J5.A6 (D+), J5.B6 (D+)
- net USB_D- is gone; now on net USB D-: ESD1.1 (IO1), J5.A7 (D-), J5.B7 (D-)
- net +3V3: now also C5.1, R5.1, U6.8 (VCC)
- net +5V: no longer C24.1, J10.2 (Pin_2)
- net +5VP: now also C24.1, J10.2 (Pin_2)
- net +BATT: now also PSW1.2; no longer C26.1, L2.1, U5.4 (VIN)
- net 5V_PWR_EN: now also U1.45 (GPIO36)
- net GND: now also C5.2, PSW1.4, U6.4 (GND)
- net GPIO0: now also R20.1
- net QSPI SCLK: now also U6.6 (CLK)
- net QSPI SD0: now also U6.5 (DI/IO_{0})
- net QSPI SD1: now also U6.2 (DO/IO_{1})
- net QSPI SD2: now also U6.3 (~{WP}/IO_{2})
- net QSPI SD3: now also U6.7 (~{HOLD}/~{RESET}/IO_{3})
- new net: C26.1, L2.1, PSW1.1, U5.4 (VIN)
- new net FLASH2 SS: R20.2, R5.2, U6.1 (~{CS})
- no-connect marks 4 -> 5
Other:
- note removed: "LED Connectors"
- note removed: "LED In"

Commit message: schematic done?
Parts:
- removed D34: B5819W, Diode_SMD:D_SOD-123, symbol Device:D_Schottky_Small
- removed ESD1: SRV05-4, Package_TO_SOT_SMD:SOT-23-6_Handsoldering, symbol Power_Protection:SRV05-4
- removed R11, R12: 5k, Resistor_SMD:R_0402_1005Metric, symbol Device:R_Small
- added C32, C33, C34, C35: 100nf, Capacitor_SMD:C_0402_1005Metric, symbol Device:C
- added D31, D32: SMBJ5.0A, easyeda2kicad:SMB_L4.6-W3.6-LS5.3-RD, symbol easyeda2kicad:SMBJ5.0A-C113974
- added D35, D36: B5819W, Diode_SMD:D_SOD-123, symbol Device:D_Schottky_Small
- added J6: USB_C_Receptacle_USB2.0_16P, Connector_USB:USB_C_Receptacle_GCT_USB4105-xx-A_16P_TopMnt_Horizontal, symbol Connector:USB_C_Receptacle_USB2.0_16P
- added Q1, Q2, Q3: PMOS, Package_TO_SOT_SMD:SOT-23, symbol Simulation_SPICE:PMOS
- added R11: 10k, Resistor_SMD:R_0402_1005Metric, symbol Device:R
- added R21, R22, R23, R28, R30, R31: 4.7k, Resistor_SMD:R_0402_1005Metric, symbol Device:R_Small
- added R24, R29: 909k, Resistor_SMD:R_0402_1005Metric, symbol Device:R_Small
- added R25, R26, R27, R32: 200k, Resistor_SMD:R_0402_1005Metric, symbol Device:R_Small
- added R33: 51.1k, Resistor_SMD:R_0402_1005Metric, symbol Device:R_Small
- added R34: 13.7k, Resistor_SMD:R_0402_1005Metric, symbol Device:R_Small
- added R35, R37, R39: 5k, Resistor_SMD:R_0402_1005Metric, symbol Device:R_Small
- added R36: 23.7k, Resistor_SMD:R_0402_1005Metric, symbol Device:R_Small
- added R38: 10.2k, Resistor_SMD:R_0402_1005Metric, symbol Device:R_Small
- added U10: TPS2121RUXR, easyeda2kicad:VQFN-HR-12_L2.5-W2.0-P0.50-BL, symbol easyeda2kicad:TPS2121RUXR
- added U7, U9: TUSB320LAIRWBR, easyeda2kicad:X2QFN-12_L1.6-W1.6-P0.40-TL, symbol easyeda2kicad:TUSB320LAIRWBR
- added U8: TS3USB221ARSER, easyeda2kicad:UQFN-10_L2.0-W1.5-P0.50-BL, symbol easyeda2kicad:TS3USB221ARSER
Connections:
- net +3V3: now also R22.1, R23.1, R30.1, R31.1
- net +5V: now also U10.1 (OUT), U10.8 (OUT)
- net GND: now also C32.1, C33.1, C34.1, C35.2, J6.A1 (GND), J6.A12 (GND), J6.B1 (GND), J6.B12 (GND), J6.S1 (SHIELD), R11.1, R21.1, R28.1, R33.1, R35.2, R37.2, R39.1, U10.12 (GND), U10.9 (ST), U7.10 (GND), U7.11 (EN_N), U7.5 (ADDR), U8.5 (GND), U8.6 (~{OE}), U9.10 (GND), U9.11 (EN_N), U9.5 (ADDR)
- net USB D+: now also U8.8 (D+); no longer J5.A6 (D+), J5.B6 (D+)
- net USB D-: now also U8.7 (D-); no longer J5.A7 (D-), J5.B7 (D-)
- net VBUS: now also Q1.1 (D), Q1.2 (G), Q2.1 (D), Q2.2 (G), R36.1, R38.1, U10.7 (IN1); no longer J5.A4 (VBUS), J5.A9 (VBUS), J5.B4 (VBUS), J5.B9 (VBUS)
- net at C28.1, C29.1, R18.2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: now also Q3.3 (S)
- net DATA_CC1 renamed DATA_CC1-1
- net DATA_CC1-1: now also U7.1 (CC1)
- net DATA_CC2 renamed DATA_CC2-1
- net DATA_CC2-1: now also U7.2 (CC2)
- new net: R29.2, U9.4 (VBUS_DET)
- new net: R28.2, U9.3 (PORT)
- new net: R32.2, U9.9 (ID)
- new net: R21.2, U7.3 (PORT)
- new net: R24.2, U7.4 (VBUS_DET)
- new net: R25.2, U7.9 (ID)
- new net: R34.1, R35.1, U10.4 (OV2)
- new net: C33.2, U8.10 (VCC)
- new net: D32.2 (A), J6.A4 (VBUS), J6.A9 (VBUS), J6.B4 (VBUS), J6.B9 (VBUS)
- new net: R36.2, R39.2, U10.5 (OV1)
- new net: R33.2, U10.10 (ILM)
- new net: C35.1, U10.11 (SS)
- new net: R37.1, R38.2, U10.6 (PR1)
- new net: D31.2 (A), J5.A4 (VBUS), J5.A9 (VBUS), J5.B4 (VBUS), J5.B9 (VBUS)
- new net +5VBAT: Q3.1 (D), Q3.2 (G), R34.2, U10.2 (IN2)
- new net 5V SELECT: U10.3 (CP2)
- new net DATA_CC1-2: J6.A5 (CC1), U9.1 (CC1)
- new net DATA_CC2-2: J6.B5 (CC2), U9.2 (CC2)
- new net USB DM1: J5.A7 (D-), J5.B7 (D-), U8.2 (1D-)
- new net USB DM2: J6.A7 (D-), J6.B7 (D-), U8.4 (2D-)
- new net USB DP1: J5.A6 (D+), J5.B6 (D+), U8.1 (1D+)
- new net USB DP2: J6.A6 (D+), J6.B6 (D+), U8.3 (2D+)
- new net USB INT-1: R26.1, U7.6 (INT_N/OUT3)
- new net USB INT-2: R27.1, U9.6 (INT_N/OUT3)
- new net USB SCL1: R23.2, U7.8 (SCL/OUT2)
- new net USB SCL2: R30.2, U9.8 (SCL/OUT2)
- new net USB SDA1: R22.2, U7.7 (SDA/OUT1)
- new net USB SDA2: R31.2, U9.7 (SDA/OUT1)
- new net VBUS1: D31.1 (C), D35.2 (A), Q2.3 (S), R24.1
- new net VBUS2: D32.1 (C), D36.2 (A), Q1.3 (S), R11.2, R29.1, U8.9 (S)
- new net VDD 5V-1: R26.2
- new net VDD 5V-2: R27.2
- new net VDD 5V1: C32.2, D35.1 (K), R25.1, U7.12 (VDD)
- new net VDD 5V2: C34.2, D36.1 (K), R32.1, U9.12 (VDD)
- no-connect marks 5 -> 7
Other:
- note added: "Diode imposter"
- note added: "Negotiator 1"
- note added: "Negotiator 2"
- note added: "Not an "O-ring" a "Or'ing" device for if usb is wimpy"
- note added: "Port 1"
- note added: "Port 2"
- note added: "TVS 1"
- note added: "TVS 2"
- note added: "USB C Stuff"
- note added: "USB Switch"
- note removed: "Both CC lines get 5.1k so we can get as much non-negotiated power as possible"
- note removed: "ESD"
- note removed: "USB C Data"
- moved on the sheet: J5
