File: Voided-Oblivion/Voided-Oblivion.kicad_pcb (KiCad board)
At the start: 2 copper layers, 291 parts, among them J4 SM03B-SRSS-TB, Q1 AO3401, Q2 AO4407A, Q3 BC857, SW1 boot, SW2 reset, U1 RP2350_80QFN, U10 TLV431, U11 LM2903, U2 TS3USB30ERSWR, U3 W25Q128JVS, U4 W25Q128JVS, U5 TPS54302, U6 TPS54302, U7 XC6220B331MR, U9 MAX40203, Y1 ABM8-272-T3

Commit message: i think the schematic is acctualy done this time, (besides little tiny things)
Parts:
- added D3: BZV55B3V3, Diode_SMD:D_MiniMELF, F.Cu at (108.0, 216.7)
- added D5: BZX84C10, Package_TO_SOT_SMD:SOT-23, F.Cu at (110.7, 220.6)
- added J1: Top male, Pogo-Pins:PG-6P-2.5-5.5H-SM-RA-Male, F.Cu at (116.6, 103.3)
- added J2: Top female, Pogo-Pins:PG-6P-2.5-5.5H-SM-RA-Female, F.Cu at (127.5, 188.5)
- added J3: Right male, Pogo-Pins:PG-6P-2.5-5.5H-SM-RA-Male, F.Cu at (110.4, 195.2)
- added J4: Right female, Pogo-Pins:PG-6P-2.5-5.5H-SM-RA-Female, F.Cu at (127.5, 194.1)
- added J5: Left male, Pogo-Pins:PG-6P-2.5-5.5H-SM-RA-Male, F.Cu at (110.4, 201.8)
- added J6: Left female, Pogo-Pins:PG-6P-2.5-5.5H-SM-RA-Female, F.Cu at (127.5, 199.7)
- added J7: Bottom male, Pogo-Pins:PG-6P-2.5-5.5H-SM-RA-Male, F.Cu at (110.4, 208.5)
- added J8: Bottom female, Pogo-Pins:PG-6P-2.5-5.5H-SM-RA-Female, F.Cu at (127.5, 205.3)
- added R48: 100Ω, Resistor_SMD:R_0402_1005Metric, F.Cu at (103.3, 216.0)
- added R49: 100Ω, Resistor_SMD:R_0402_1005Metric, F.Cu at (103.3, 218.0)
- added R50: 100Ω, Resistor_SMD:R_0402_1005Metric, F.Cu at (103.3, 220.0)
- added R51: 100Ω, Resistor_SMD:R_0402_1005Metric, F.Cu at (103.3, 222.0)
- added R62: 0Ω, Resistor_SMD:R_0402_1005Metric, F.Cu at (116.6, 216.0)
- added R63: 33Ω, Resistor_SMD:R_0402_1005Metric, F.Cu at (116.6, 218.0)
- added R64: 33Ω, Resistor_SMD:R_0402_1005Metric, F.Cu at (116.6, 220.0)
- added R65: 0Ω, Resistor_SMD:R_0402_1005Metric, F.Cu at (116.6, 222.0)
- added R66: 0Ω, Resistor_SMD:R_0402_1005Metric, F.Cu at (116.6, 224.0)
- added U13: TPD2E2U06DRL, Package_TO_SOT_SMD:SOT-553, F.Cu at (106.5, 220.1)
- added U14: TPD2E2U06DRL, Package_TO_SOT_SMD:SOT-553, F.Cu at (106.5, 223.2)
- added U7: TLV76733DRVR, Package_SON:WSON-6-1EP_2x2mm_P0.65mm_EP1x1.6mm_ThermalVias, F.Cu at (110.1, 224.7)
- added U8: SN74LVC2T45DCUR, Package_SO:VSSOP-8_2.3x2mm_P0.5mm, F.Cu at (120.9, 217.0)
- C24: value 10µF -> 1µF
- R44, R45: value 100kΩ -> 4.7kΩ
- U10: value TLV431 -> TLV431B
- moved C100 222.8 mm to (128.5, 235.4)
- moved C101 222.8 mm to (148.2, 238.2)
- moved C102 222.8 mm to (146.3, 238.2)
- moved C103 222.8 mm to (144.3, 238.2)
- moved C104 222.8 mm to (142.3, 238.2)
- moved C105 222.8 mm to (140.4, 238.2)
- moved C106 222.8 mm to (138.4, 238.2)
- moved C107 222.8 mm to (136.4, 238.2)
- moved C81 222.8 mm to (144.3, 232.5)
- moved C82 222.8 mm to (142.3, 232.5)
- moved C83 222.8 mm to (140.4, 232.5)
- moved C84 222.8 mm to (138.4, 232.5)
- moved C85 222.8 mm to (136.4, 232.5)
- moved C86 222.8 mm to (134.4, 232.5)
- moved C87 222.8 mm to (132.5, 232.5)
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- renumbered J4 to J9
Connections:
- net Net-(U2-D1+) renamed /power/USB1 D+
- net Net-(U2-D1-) renamed /power/USB1 D-
- net Net-(U2-D2+) renamed /power/USB2 D+
- net Net-(U2-D2-) renamed /power/USB2 D-
- AM0 pad 16: AM0:15 -> Net-(AM0-I15)
- AM1 pad 16: AM1:15 -> Net-(AM1-I15)
- LED11 pad 3: Net-(LED11-SDI) -> Net-(LED10-SDO)
- LED11 pad 4: Net-(LED11-CKI) -> Net-(LED10-CKO)
- LED12 pad 2: +5VP -> GND
- LED12 pad 3: Net-(LED12-SDI) -> Net-(LED11-SDO)
- LED12 pad 4: Net-(LED12-CKI) -> Net-(LED11-CKO)
- LED12 pad 5: GND -> +5VP
- LED13 pad 3: Net-(LED13-SDI) -> Net-(LED12-SDO)
- LED13 pad 4: Net-(LED13-CKI) -> Net-(LED12-CKO)
- LED14 pad 2: +5VP -> GND
- LED14 pad 3: Net-(LED14-SDI) -> Net-(LED13-SDO)
- LED14 pad 4: Net-(LED14-CKI) -> Net-(LED13-CKO)
- LED14 pad 5: GND -> +5VP
- LED15 pad 3: Net-(LED10-SDO) -> Net-(LED14-SDO)
- LED15 pad 4: Net-(LED10-CKO) -> Net-(LED14-CKO)
- LED16 pad 3: Net-(LED11-SDO) -> Net-(LED15-SDO)
- LED16 pad 4: Net-(LED11-CKO) -> Net-(LED15-CKO)
- LED17 pad 1: Net-(LED12-SDI) -> Net-(LED17-SDO)
- LED17 pad 2: +5VP -> GND
- LED17 pad 3: Net-(LED17-SDI) -> Net-(LED16-SDO)
- LED17 pad 4: Net-(LED17-CKI) -> Net-(LED16-CKO)
- LED17 pad 5: GND -> +5VP
- LED17 pad 6: Net-(LED12-CKI) -> Net-(LED17-CKO)
- LED18 pad 3: Net-(LED13-SDO) -> Net-(LED17-SDO)
- LED18 pad 4: Net-(LED13-CKO) -> Net-(LED17-CKO)
- LED19 pad 2: +5VP -> GND
- LED19 pad 3: Net-(LED14-SDO) -> Net-(LED18-SDO)
- LED19 pad 4: Net-(LED14-CKO) -> Net-(LED18-CKO)
- LED19 pad 5: GND -> +5VP
- LED2 pad 2: +5VP -> GND
- LED2 pad 3: Net-(LED2-SDI) -> Net-(LED1-SDO)
- LED2 pad 4: Net-(LED2-CKI) -> Net-(LED1-CKO)
- LED2 pad 5: GND -> +5VP
- LED20 pad 3: Net-(LED15-SDO) -> Net-(LED19-SDO)
- LED20 pad 4: Net-(LED15-CKO) -> Net-(LED19-CKO)
- LED21 pad 3: Net-(LED16-SDO) -> Net-(LED20-SDO)
- LED21 pad 4: Net-(LED16-CKO) -> Net-(LED20-CKO)
- LED22 pad 1: Net-(LED17-SDI) -> Net-(LED22-SDO)
- LED22 pad 2: +5VP -> GND
- LED22 pad 3: Net-(LED22-SDI) -> Net-(LED21-SDO)
- LED22 pad 4: Net-(LED22-CKI) -> Net-(LED21-CKO)
- LED22 pad 5: GND -> +5VP
- LED22 pad 6: Net-(LED17-CKI) -> Net-(LED22-CKO)
- LED23 pad 3: Net-(LED18-SDO) -> Net-(LED22-SDO)
- LED23 pad 4: Net-(LED18-CKO) -> Net-(LED22-CKO)
- LED24 pad 2: +5VP -> GND
- LED24 pad 3: Net-(LED19-SDO) -> Net-(LED23-SDO)
- LED24 pad 4: Net-(LED19-CKO) -> Net-(LED23-CKO)
- LED24 pad 5: GND -> +5VP
- LED25 pad 3: Net-(LED20-SDO) -> Net-(LED24-SDO)
- LED25 pad 4: Net-(LED20-CKO) -> Net-(LED24-CKO)
- LED26 pad 3: Net-(LED21-SDO) -> Net-(LED25-SDO)
- LED26 pad 4: Net-(LED21-CKO) -> Net-(LED25-CKO)
- LED27 pad 1: Net-(LED22-SDI) -> Net-(LED27-SDO)
- LED27 pad 2: +5VP -> GND
- LED27 pad 5: GND -> +5VP
- LED27 pad 6: Net-(LED22-CKI) -> Net-(LED27-CKO)
- LED28 pad 3: Net-(LED23-SDO) -> Net-(LED27-SDO)
- LED28 pad 4: Net-(LED23-CKO) -> Net-(LED27-CKO)
- LED29 pad 2: +5VP -> GND
- LED29 pad 3: Net-(LED24-SDO) -> Net-(LED28-SDO)
- LED29 pad 4: Net-(LED24-CKO) -> Net-(LED28-CKO)
- LED29 pad 5: GND -> +5VP
- LED30 pad 3: Net-(LED25-SDO) -> Net-(LED29-SDO)
- LED30 pad 4: Net-(LED25-CKO) -> Net-(LED29-CKO)
- LED4 pad 2: +5VP -> GND
- LED4 pad 3: Net-(LED28-SDO) -> Net-(LED3-SDO)
- LED4 pad 4: Net-(LED28-CKO) -> Net-(LED3-CKO)
- LED4 pad 5: GND -> +5VP
- LED5 pad 1: Net-(LED10-SDI) -> Net-(LED5-SDO)
- LED5 pad 3: Net-(LED29-SDO) -> Net-(LED4-SDO)
- LED5 pad 4: Net-(LED29-CKO) -> Net-(LED4-CKO)
- LED5 pad 6: Net-(LED10-CKI) -> Net-(LED5-CKO)
- LED6 pad 1: Net-(LED11-SDI) -> Net-(LED6-SDO)
- LED6 pad 3: Net-(LED1-SDO) -> Net-(LED5-SDO)
- LED6 pad 4: Net-(LED1-CKO) -> Net-(LED5-CKO)
- LED6 pad 6: Net-(LED11-CKI) -> Net-(LED6-CKO)
- LED7 pad 1: Net-(LED2-SDI) -> Net-(LED7-SDO)
- LED7 pad 2: +5VP -> GND
- LED7 pad 3: Net-(LED12-SDO) -> Net-(LED6-SDO)
- LED7 pad 4: Net-(LED12-CKO) -> Net-(LED6-CKO)
- LED7 pad 5: GND -> +5VP
- LED7 pad 6: Net-(LED2-CKI) -> Net-(LED7-CKO)
- LED8 pad 1: Net-(LED13-SDI) -> Net-(LED8-SDO)
- LED8 pad 3: Net-(LED3-SDO) -> Net-(LED7-SDO)
- LED8 pad 4: Net-(LED3-CKO) -> Net-(LED7-CKO)
- LED8 pad 6: Net-(LED13-CKI) -> Net-(LED8-CKO)
- LED9 pad 1: Net-(LED14-SDI) -> Net-(LED10-SDI)
- LED9 pad 2: +5VP -> GND
- LED9 pad 3: Net-(LED4-SDO) -> Net-(LED8-SDO)
- LED9 pad 4: Net-(LED4-CKO) -> Net-(LED8-CKO)
- LED9 pad 5: GND -> +5VP
- LED9 pad 6: Net-(LED14-CKI) -> Net-(LED10-CKI)
- PD1 pad 1: Net-(USB1-CC1) -> Net-(PD1-CC2-Pad1)
- PD1 pad 10: Net-(USB1-CC2) -> Net-(PD1-CC1-Pad10)
- PD1 pad 11: Net-(USB1-CC2) -> Net-(PD1-CC1-Pad10)
- PD1 pad 14: Net-(USB1-CC1) -> Net-(PD1-CC2-Pad1)
- PD2 pad 1: Net-(USB2-CC1) -> Net-(PD2-CC2-Pad1)
- PD2 pad 10: Net-(USB2-CC2) -> Net-(PD2-CC1-Pad10)
- PD2 pad 11: Net-(USB2-CC2) -> Net-(PD2-CC1-Pad10)
- PD2 pad 14: Net-(USB2-CC1) -> Net-(PD2-CC2-Pad1)
- R12 pad 1: BS+ -> Net-(U7-EN)
- R12 pad 2: Net-(U7-CE) -> BS+
Other:
- board outline added: 95.3 x 114.3 mm

Commit message: drc rules and stuff
Parts:
- removed the D3 at (169.4, 171.7)
- removed the R48 at (126.5, 167.1)
- removed the R49 at (126.5, 169.1)
- removed the R50 at (129.4, 163.1)
- removed the R51 at (129.4, 165.1)
- removed R9: DNP, Resistor_SMD:R_0402_1005Metric
- removed the U7 at (172.4, 187.7)
- added C116: 100nF, Capacitor_SMD:C_0402_1005Metric, F.Cu at (30.6, 201.9)
- added C117: 100nF, Capacitor_SMD:C_0402_1005Metric, F.Cu at (33.5, 194.0)
- added C118: 100nF, Capacitor_SMD:C_0402_1005Metric, F.Cu at (33.5, 196.0)
- added C119: 100nF, Capacitor_SMD:C_0402_1005Metric, F.Cu at (33.5, 198.0)
- added C120: 1µF, Capacitor_SMD:C_0402_1005Metric, F.Cu at (33.5, 199.9)
- added C121: 10µF, Capacitor_SMD:C_1206_3216Metric, F.Cu at (33.5, 201.9)
- added C122: 100nF, Capacitor_SMD:C_0402_1005Metric, F.Cu at (28.7, 208.7)
- added C123: 100nF, Capacitor_SMD:C_0402_1005Metric, F.Cu at (28.7, 210.7)
- added C124: 100nF, Capacitor_SMD:C_0402_1005Metric, F.Cu at (28.7, 212.6)
- added C125: 100nF, Capacitor_SMD:C_0402_1005Metric, F.Cu at (28.7, 214.6)
- added H1: MountingHole, MountingHole:MountingHole_2.2mm_M2_DIN965, F.Cu at (100.0, 100.0)
- added H2: MountingHole, MountingHole:MountingHole_2.2mm_M2_DIN965, F.Cu at (100.0, 135.7)
- added H3: MountingHole, MountingHole:MountingHole_2.2mm_M2_DIN965, F.Cu at (100.0, 26.2)
- added H4: MountingHole, MountingHole:MountingHole_2.2mm_M2_DIN965, F.Cu at (116.7, 42.9)
- added H5: MountingHole, MountingHole:MountingHole_2.2mm_M2_DIN965, F.Cu at (116.7, 119.1)
- added H6: MountingHole, MountingHole:MountingHole_2.2mm_M2_DIN965, F.Cu at (61.9, 42.9)
- added H7: MountingHole, MountingHole:MountingHole_2.2mm_M2_DIN965, F.Cu at (42.9, 135.7)
- added H8: MountingHole_Pad, MountingHole:MountingHole_2.2mm_M2_DIN965_Pad, F.Cu at (42.9, 61.9)
- added J10: Sub-Module TL, Voided-Oblivion-misc:5-pin-machined-female-pin-headers-sunk, F.Cu at (33.3, 25.6)
- added J11: Sub-Module LT, Voided-Oblivion-misc:5-pin-machined-female-pin-headers-sunk, F.Cu at (25.6, 33.3)
- added J12: Sub-Module TR, Voided-Oblivion-misc:5-pin-machined-female-pin-headers-sunk, F.Cu at (109.5, 25.6)
- added J16: Sub-Module BL, Voided-Oblivion-misc:5-pin-machined-female-pin-headers-sunk, F.Cu at (33.3, 136.3)
- added J17: Sub-Module LB, Voided-Oblivion-misc:5-pin-machined-female-pin-headers-sunk, F.Cu at (25.6, 128.6)
- added J18: Sub-Module BR, Voided-Oblivion-misc:5-pin-machined-female-pin-headers-sunk, F.Cu at (109.5, 136.3)
- added J19: Sub-Module RB, Voided-Oblivion-misc:5-pin-machined-female-pin-headers-sunk, F.Cu at (117.3, 128.6)
- added J20: Sub-Module RT, Voided-Oblivion-misc:5-pin-machined-female-pin-headers-sunk, F.Cu at (117.3, 33.3)
- added L2: 10µH, Inductor_SMD:L_APV_APH0630, F.Cu at (114.7, 196.9)
- added L3: 10µH, Inductor_SMD:L_APV_APH0630, F.Cu at (114.7, 205.0)
- added Q10: BC847B, Package_TO_SOT_SMD:SOT-23, F.Cu at (26.7, 190.2)
- added Q11: BC847B, Package_TO_SOT_SMD:SOT-23, F.Cu at (26.7, 194.7)
- added Q4: AO4407A, Package_SO:SOP-8_3.76x4.96mm_P1.27mm, F.Cu at (20.0, 182.5)
- added Q5: AO4407A, Package_SO:SOP-8_3.76x4.96mm_P1.27mm, F.Cu at (20.0, 189.2)
- added Q6: AO4407A, Package_SO:SOP-8_3.76x4.96mm_P1.27mm, F.Cu at (20.0, 195.8)
- added Q7: AO4407A, Package_SO:SOP-8_3.76x4.96mm_P1.27mm, F.Cu at (20.0, 202.4)
- added Q8: BC847B, Package_TO_SOT_SMD:SOT-23, F.Cu at (26.7, 181.3)
- added Q9: BC847B, Package_TO_SOT_SMD:SOT-23, F.Cu at (26.7, 185.8)
- added R100: 10kΩ, Resistor_SMD:R_0402_1005Metric, F.Cu at (25.9, 214.7)
- added R5: 1kΩ, Resistor_SMD:R_0402_1005Metric, F.Cu at (17.1, 208.7)
- added R67: 100kΩ, Resistor_SMD:R_0402_1005Metric, F.Cu at (30.6, 182.1)
- added R68: 100kΩ, Resistor_SMD:R_0402_1005Metric, F.Cu at (30.6, 184.1)
- added R69: 100kΩ, Resistor_SMD:R_0402_1005Metric, F.Cu at (30.6, 186.1)
- added R70: 100kΩ, Resistor_SMD:R_0402_1005Metric, F.Cu at (30.6, 188.1)
- added R71: 4.7kΩ, Resistor_SMD:R_0402_1005Metric, F.Cu at (30.6, 190.1)
- added R72: 4.7kΩ, Resistor_SMD:R_0402_1005Metric, F.Cu at (30.6, 192.1)
- added R73: 4.7kΩ, Resistor_SMD:R_0402_1005Metric, F.Cu at (33.6, 180.1)
- added R74: 4.7kΩ, Resistor_SMD:R_0402_1005Metric, F.Cu at (33.6, 182.1)
- added R75: 10kΩ, Resistor_SMD:R_0402_1005Metric, F.Cu at (33.6, 184.1)
- added R76: 10kΩ, Resistor_SMD:R_0402_1005Metric, F.Cu at (33.6, 186.1)
- added R77: 10kΩ, Resistor_SMD:R_0402_1005Metric, F.Cu at (33.6, 188.1)
- added R78: 10kΩ, Resistor_SMD:R_0402_1005Metric, F.Cu at (33.6, 190.1)
- added R79: 100kΩ, Resistor_SMD:R_0402_1005Metric, F.Cu at (33.6, 192.1)
- added R80: 100kΩ, Resistor_SMD:R_0402_1005Metric, F.Cu at (36.5, 180.1)
- added R81: 100kΩ, Resistor_SMD:R_0402_1005Metric, F.Cu at (36.5, 182.1)
- added R82: 100kΩ, Resistor_SMD:R_0402_1005Metric, F.Cu at (36.5, 184.1)
- added R83: 100kΩ, Resistor_SMD:R_0402_1005Metric, F.Cu at (36.5, 186.1)
- added R84: 0Ω, Resistor_SMD:R_0402_1005Metric, F.Cu at (17.1, 212.7)
- added R85: 0Ω, Resistor_SMD:R_0402_1005Metric, F.Cu at (17.1, 214.7)
- added R86: 0Ω, Resistor_SMD:R_0402_1005Metric, F.Cu at (20.0, 208.7)
- added R87: 0Ω, Resistor_SMD:R_0402_1005Metric, F.Cu at (20.0, 210.7)
- added R88: 4.7kΩ, Resistor_SMD:R_0402_1005Metric, F.Cu at (20.0, 212.7)
- added R89: 4.7kΩ, Resistor_SMD:R_0402_1005Metric, F.Cu at (20.0, 214.7)
- added R90: 4.7kΩ, Resistor_SMD:R_0402_1005Metric, F.Cu at (22.9, 208.7)
- added R91: 4.7kΩ, Resistor_SMD:R_0402_1005Metric, F.Cu at (22.9, 210.7)
- added R92: 4.7kΩ, Resistor_SMD:R_0402_1005Metric, F.Cu at (36.5, 188.1)
- added R93: 10kΩ, Resistor_SMD:R_0402_1005Metric, F.Cu at (22.9, 212.7)
- added R94: 10kΩ, Resistor_SMD:R_0402_1005Metric, F.Cu at (22.9, 214.7)
- added R95: 4.7kΩ, Resistor_SMD:R_0402_1005Metric, F.Cu at (36.5, 190.1)
- added R96: 100kΩ, Resistor_SMD:R_0402_1005Metric, F.Cu at (36.5, 192.1)
- added R97: 10kΩ, Resistor_SMD:R_0402_1005Metric, F.Cu at (25.9, 208.7)
- added R98: 1kΩ, Resistor_SMD:R_0402_1005Metric, F.Cu at (25.9, 210.7)
- added R99: 1kΩ, Resistor_SMD:R_0402_1005Metric, F.Cu at (25.9, 212.7)
- added U12: AP2171WG-7, Package_TO_SOT_SMD:SOT-23-5, F.Cu at (37.5, 195.5)
- added U15: LM66100DCKT, Package_TO_SOT_SMD:SOT-363_SC-70-6, F.Cu at (26.3, 202.3)
- added U16: AP2171WG-7, Package_TO_SOT_SMD:SOT-23-5, F.Cu at (37.5, 200.1)
- C10, C6, C7, C9: value 4.7u -> 4.7µF
- C11, C110, C111, C112, C113, C12, C13, C14, C15, C16, C17, C18, C2, C20, C21, C8: value 100n -> 100nF
- C114, C76: value 100nF -> 1µF
- C19: value 10u -> 10µF; footprint Capacitor_SMD:C_0805_2012Metric -> Capacitor_SMD:C_1206_3216Metric
- C22: value DNP -> 100nF
- C25, C27, C32, C33, C42, C43: value 0.1µF -> 100nF
- C26, C28, C29, C31, C34, C35, C40: footprint Capacitor_SMD:C_0402_1005Metric -> Capacitor_SMD:C_1206_3216Metric
- C41: value 100µF -> 1µF
- C77: value 1µF -> 10µF; footprint Capacitor_SMD:C_0402_1005Metric -> Capacitor_SMD:C_1206_3216Metric
- R1, R13: value DNP -> 10kΩ
- R10: value 0 -> 0Ω
- R11: value DNP -> 0Ω
- R2, R4, R6: value 1k -> 1kΩ
- R22: value 10kΩ -> 5.1kΩ
- R23: value 0Ω -> 1kΩ
- R3: value 33 -> 33Ω
- R30: value 44.2kΩ -> 35.7kΩ
- R31: value 12.2kΩ -> 10kΩ
- R7, R8: value 27 -> 27Ω
- U10: value TLV431B -> TLV431BQDBZR
- U9: value MAX40203 -> LM66100DCKT; footprint Package_BGA:WLP-4_0.728x0.728mm_Layout2x2_P0.35mm -> Package_TO_SOT_SMD:SOT-363_SC-70-6
- USB1, USB2: value USB_C_Receptacle -> USB_C_Receptacle_USB2.0_16P; footprint Connector_USB:USB_C_Receptacle_Molex_105450-0101 -> Connector_USB:USB_C_Receptacle_HCTL_HC-TYPE-C-16P-01A
- moved C83 205.8 mm to (34.1, 56.3)
- moved C81 202.4 mm to (91.2, 37.2)
- moved C82 197.9 mm to (110.3, 37.2)
- moved U13 195.9 mm to (45.0, 34.1), turned to -90 degrees
- moved C84 195.8 mm to (53.1, 56.3)
- moved C85 187.6 mm to (72.2, 56.3)
- moved C88 184.4 mm to (34.1, 75.3)
- moved C86 181.5 mm to (91.2, 56.3)
- moved C93 177.8 mm to (34.1, 94.4)
- moved C87 177.6 mm to (110.3, 56.3)
- moved C90 177.2 mm to (72.2, 75.3)
- moved C89 174.3 mm to (53.1, 75.3)
- moved USB1 169.6 mm to (45.2, 28.0), turned to 180 degrees
- moved C91 169.3 mm to (91.2, 75.3)
- moved J6 169.2 mm to (26.3, 64.1), turned to -90 degrees
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Connections:
- net /power/USB1 D+ renamed USB1 D+
- net /power/USB1 D- renamed USB1 D-
- net /power/USB2 D+ renamed USB2 D+
- net /power/USB2 D- renamed USB2 D-
- net Net-(U1-USB_DM) renamed /MCU D-
- net Net-(U1-USB_DP) renamed /MCU D+
- net Net-(U5-SW) renamed SW CLEAN
- net Net-(U6-SW) renamed SW NOISY
- C114 pad 1: +5VA -> +5VP
- C41 pad 1: GND -> +5VA
- C41 pad 2: BS+ -> GND
- C76 pad 1: GND -> BS+
- C76 pad 2: +5VP -> GND
- C77 pad 2: +5VP -> /power/SM BUS
- J1 pad 3: unconnected-(J1-Pin_3-Pad3) -> PD+ TOP
- J1 pad 4: unconnected-(J1-Pin_4-Pad4) -> PD+ TOP
- J1 pad 6: unconnected-(J1-Pin_6-Pad6) -> Net-(J1-Pin_6)
- J2 pad 1: unconnected-(J2-Pin_1-Pad1) -> Rx TOP
- J2 pad 3: unconnected-(J2-Pin_3-Pad3) -> PD+ TOP
- J2 pad 4: unconnected-(J2-Pin_4-Pad4) -> PD+ TOP
- J3 pad 3: unconnected-(J3-Pin_3-Pad3) -> PD+ RIGHT
- J3 pad 4: unconnected-(J3-Pin_4-Pad4) -> PD+ RIGHT
- J3 pad 6: unconnected-(J3-Pin_6-Pad6) -> Net-(J3-Pin_6)
- J4 pad 1: unconnected-(J4-Pin_1-Pad1) -> Rx RIGHT
- J4 pad 3: unconnected-(J4-Pin_3-Pad3) -> PD+ RIGHT
- J4 pad 4: unconnected-(J4-Pin_4-Pad4) -> PD+ RIGHT
- J5 pad 3: unconnected-(J5-Pin_3-Pad3) -> PD+ LEFT
- J5 pad 4: unconnected-(J5-Pin_4-Pad4) -> PD+ LEFT
- J5 pad 6: unconnected-(J5-Pin_6-Pad6) -> Net-(J5-Pin_6)
- J6 pad 1: unconnected-(J6-Pin_1-Pad1) -> Rx LEFT
- J6 pad 3: unconnected-(J6-Pin_3-Pad3) -> PD+ LEFT
- J6 pad 4: unconnected-(J6-Pin_4-Pad4) -> PD+ LEFT
- J7 pad 3: unconnected-(J7-Pin_3-Pad3) -> PD+ BOTTOM
- J7 pad 4: unconnected-(J7-Pin_4-Pad4) -> PD+ BOTTOM
- J7 pad 6: unconnected-(J7-Pin_6-Pad6) -> Net-(J7-Pin_6)
- J8 pad 1: unconnected-(J8-Pin_1-Pad1) -> Rx BOTTOM
- J8 pad 3: unconnected-(J8-Pin_3-Pad3) -> PD+ BOTTOM
- J8 pad 4: unconnected-(J8-Pin_4-Pad4) -> PD+ BOTTOM
- R11 pad 1: /GPIO0 -> FLASH CS1n
- R15 pad 1: +5VA -> BS+
- R15 pad 2: Net-(U9-EN) -> Net-(U9-~{CE})
- R16 pad 1: Net-(R16-Pad1) -> /power/SM BUS
- R16 pad 2: GND -> Net-(U15-~{CE})
- R23 pad 1: Net-(R23-Pad1) -> BL ID
- R23 pad 2: GND -> Net-(J16-Pin_1)
- R48 pad 2: Net-(PD1-CC1-Pad10) -> Net-(PD1-CC2-Pad1)
- R49 pad 1: Net-(PD1-CC2-Pad1) -> Net-(PD1-CC1-Pad10)
- R50 pad 2: Net-(PD2-CC1-Pad10) -> Net-(PD2-CC2-Pad1)
- R51 pad 1: Net-(PD2-CC2-Pad1) -> Net-(PD2-CC1-Pad10)
- U1 pad 1: unconnected-(U1-GPIO4-Pad1) -> Tx TOP
- U1 pad 11: unconnected-(U1-GPIO12-Pad11) -> Tx BOTTOM
- U1 pad 12: unconnected-(U1-GPIO13-Pad12) -> Rx BOTTOM
- U1 pad 16: unconnected-(U1-GPIO16-Pad16) -> Tx LEFT
- U1 pad 17: unconnected-(U1-GPIO17-Pad17) -> Rx LEFT
- U1 pad 19: unconnected-(U1-GPIO19-Pad19) -> FLASH CS1n
- U1 pad 2: unconnected-(U1-GPIO5-Pad2) -> Rx TOP
- U1 pad 22: unconnected-(U1-GPIO22-Pad22) -> TL Tx
- U1 pad 23: unconnected-(U1-GPIO23-Pad23) -> TL Rx
- U1 pad 25: unconnected-(U1-GPIO24-Pad25) -> TR Tx
- U1 pad 26: unconnected-(U1-GPIO25-Pad26) -> TR Rx
- U1 pad 27: unconnected-(U1-GPIO26-Pad27) -> BR Tx
- U1 pad 28: unconnected-(U1-GPIO27-Pad28) -> BR Rx
- U1 pad 3: unconnected-(U1-GPIO6-Pad3) -> Tx RIGHT
- U1 pad 36: unconnected-(U1-GPIO28-Pad36) -> BL Tx
- U1 pad 37: unconnected-(U1-GPIO29-Pad37) -> BL Rx
- U1 pad 4: unconnected-(U1-GPIO7-Pad4) -> Rx RIGHT
- U1 pad 40: unconnected-(U1-GPIO32-Pad40) -> SM BS EN
- U1 pad 42: unconnected-(U1-GPIO33-Pad42) -> SM+ EN
- U1 pad 45: unconnected-(U1-GPIO36-Pad45) -> BS+ SRC
- U1 pad 46: unconnected-(U1-GPIO37-Pad46) -> SM+ FLT
- U1 pad 53: unconnected-(U1-GPIO42_ADC2-Pad53) -> TL ID
- U1 pad 54: unconnected-(U1-GPIO43_ADC3-Pad54) -> TR ID
- U1 pad 55: unconnected-(U1-GPIO44_ADC4-Pad55) -> BR ID
- U1 pad 56: unconnected-(U1-GPIO45_ADC5-Pad56) -> BL ID
- U1 pad 77: unconnected-(U1-GPIO0-Pad77) -> PD EN TOP
- U1 pad 78: unconnected-(U1-GPIO1-Pad78) -> PD EN RIGHT
- U1 pad 79: unconnected-(U1-GPIO2-Pad79) -> PD EN BOTTOM
- U1 pad 80: unconnected-(U1-GPIO3-Pad80) -> PD EN LEFT
- U10 pad 1: (no net) -> +1V24ref
- U10 pad 2: (no net) -> Net-(U10-REF)
- U10 pad 3: +1V24ref -> GND
Routing:
- net USB1 D-: track 0.00 -> 5.67 mm
- net USB1 D+: track 0.00 -> 4.36 mm
- added copper zone on B.Cu, net GND
- added copper zone on F.Cu, net GND
- added copper zone on In1.Cu, net GND
- added copper zone on In2.Cu, net GND
Other:
- copper layers 2 -> 4

Commit message: checkpoint
Parts:
- added TP1: TestPoint, TestPoint:TestPoint_Pad_D1.0mm, F.Cu at (124.4, 168.9)
- added TP10: TestPoint, TestPoint:TestPoint_Pad_D1.0mm, F.Cu at (127.4, 178.0)
- added TP11: TestPoint, TestPoint:TestPoint_Pad_D1.0mm, F.Cu at (127.4, 181.1)
- added TP12: TestPoint, TestPoint:TestPoint_Pad_D1.0mm, F.Cu at (127.4, 184.1)
- added TP13: TestPoint, TestPoint:TestPoint_Pad_D1.0mm, F.Cu at (130.5, 168.9)
- added TP14: TestPoint, TestPoint:TestPoint_Pad_D1.0mm, F.Cu at (130.5, 171.9)
- added TP15: TestPoint, TestPoint:TestPoint_Pad_D1.0mm, F.Cu at (130.5, 175.0)
- added TP16: TestPoint, TestPoint:TestPoint_Pad_D1.0mm, F.Cu at (130.5, 178.0)
- added TP17: TestPoint, TestPoint:TestPoint_Pad_D1.0mm, F.Cu at (130.5, 181.1)
- added TP18: TestPoint, TestPoint:TestPoint_Pad_D1.0mm, F.Cu at (130.5, 184.1)
- added TP19: TestPoint, TestPoint:TestPoint_Pad_D1.0mm, F.Cu at (133.5, 168.9)
- added TP2: TestPoint, TestPoint:TestPoint_Pad_D1.0mm, F.Cu at (124.4, 171.9)
- added TP20: TestPoint, TestPoint:TestPoint_Pad_D1.0mm, F.Cu at (133.5, 171.9)
- added TP21: TestPoint, TestPoint:TestPoint_Pad_D1.0mm, F.Cu at (133.5, 175.0)
- added TP22: TestPoint, TestPoint:TestPoint_Pad_D1.0mm, F.Cu at (133.5, 178.0)
- added TP23: TestPoint, TestPoint:TestPoint_Pad_D1.0mm, F.Cu at (133.5, 181.1)
- added TP24: TestPoint, TestPoint:TestPoint_Pad_D1.0mm, F.Cu at (133.5, 184.1)
- added TP25: TestPoint, TestPoint:TestPoint_Pad_D1.0mm, F.Cu at (136.6, 168.9)
- added TP26: TestPoint, TestPoint:TestPoint_Pad_D1.0mm, F.Cu at (136.6, 171.9)
- added TP27: TestPoint, TestPoint:TestPoint_Pad_D1.0mm, F.Cu at (136.6, 175.0)
- added TP28: TestPoint, TestPoint:TestPoint_Pad_D1.0mm, F.Cu at (136.6, 178.0)
- added TP29: TestPoint, TestPoint:TestPoint_Pad_D1.0mm, F.Cu at (136.6, 181.1)
- added TP3: TestPoint, TestPoint:TestPoint_Pad_D1.0mm, F.Cu at (124.4, 175.0)
- added TP30: TestPoint, TestPoint:TestPoint_Pad_D1.0mm, F.Cu at (136.6, 184.1)
- added TP31: TestPoint, TestPoint:TestPoint_Pad_D1.0mm, F.Cu at (139.6, 168.9)
- added TP32: TestPoint, TestPoint:TestPoint_Pad_D1.0mm, F.Cu at (139.6, 171.9)
- added TP33: TestPoint, TestPoint:TestPoint_Pad_D1.0mm, F.Cu at (139.6, 175.0)
- added TP34: TestPoint, TestPoint:TestPoint_Pad_D1.0mm, F.Cu at (139.6, 178.0)
- added TP35: TestPoint, TestPoint:TestPoint_Pad_D1.0mm, F.Cu at (139.6, 181.1)
- added TP36: TestPoint, TestPoint:TestPoint_Pad_D1.0mm, F.Cu at (139.6, 184.1)
- added TP37: TestPoint, TestPoint:TestPoint_Pad_D1.0mm, F.Cu at (124.4, 189.2)
- added TP4: TestPoint, TestPoint:TestPoint_Pad_D1.0mm, F.Cu at (124.4, 178.0)
- added TP5: TestPoint, TestPoint:TestPoint_Pad_D1.0mm, F.Cu at (124.4, 181.1)
- added TP6: TestPoint, TestPoint:TestPoint_Pad_D1.0mm, F.Cu at (124.4, 184.1)
- added TP7: TestPoint, TestPoint:TestPoint_Pad_D1.0mm, F.Cu at (127.4, 168.9)
- added TP8: TestPoint, TestPoint:TestPoint_Pad_D1.0mm, F.Cu at (127.4, 171.9)
- added TP9: TestPoint, TestPoint:TestPoint_Pad_D1.0mm, F.Cu at (127.4, 175.0)
- moved C21 152.2 mm to (59.5, 66.8), turned to 180 degrees
- moved U3 149.8 mm to (57.2, 47.6)
- moved C13 147.3 mm to (62.4, 68.5), turned to -90 degrees
- moved Y1 142.4 mm to (63.8, 73.9)
- moved C10 140.9 mm to (65.3, 68.5), turned to -90 degrees
- moved C4 140.6 mm to (65.3, 70.3)
- moved C3 139.2 mm to (62.4, 70.3), turned to 180 degrees
- moved R2 131.9 mm to (64.0, 68.6), turned to -90 degrees
- moved C11 129.8 mm to (144.7, 88.7)
- moved C110 129.8 mm to (150.4, 86.7)
- moved C111 129.8 mm to (150.4, 88.7)
- moved C112 129.8 mm to (150.4, 90.6)
- moved C113 129.8 mm to (150.4, 92.6)
- moved C12 129.8 mm to (144.7, 90.6)
- moved C14 129.8 mm to (144.7, 94.6)
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Routing:
- net AM0:11: track 0.00 -> 61.8 mm
- net AM0:12: track 0.00 -> 58.9 mm
- net AM0:6: track 0.00 -> 54.9 mm
- net AM0:0: track 0.00 -> 52.0 mm
- net AM0:5: track 0.00 -> 47.9 mm
- net AM0:10: track 0.00 -> 43.4 mm
- net AM0:9: track 0.00 -> 43.0 mm
- net AM0:13: track 0.00 -> 38.8 mm
- net AM0:7: track 0.00 -> 38.5 mm
- net AM0:1: track 0.00 -> 33.6 mm
- net +1V1: track 0.00 -> 30.1 mm, vias 0 -> 9
- net AM0:4: track 0.00 -> 29.5 mm
- net AM0:2: track 0.00 -> 15.2 mm
- net AM0:14: track 0.00 -> 13.8 mm
- net AM0:8: track 0.00 -> 13.6 mm
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- added copper zone on F.Cu, net +1V1
- added copper zone on F.Cu, net /VREG_LX
- added copper zone on F.Cu, net VBUS

Commit message: blaaa why does placeing and routing things take so looonnggggggggg >:c
Parts:
- added H10: MountingHole, MountingHole:MountingHole_2.2mm_M2_DIN965, F.Cu at (42.9, 100.0)
- added H11: MountingHole, MountingHole:MountingHole_2.2mm_M2_DIN965, F.Cu at (81.0, 42.9)
- added H12: MountingHole, MountingHole:MountingHole_2.2mm_M2_DIN965, F.Cu at (81.0, 119.1)
- added H13: MountingHole, MountingHole:MountingHole_2.2mm_M2_DIN965, F.Cu at (26.2, 81.0)
- added H14: MountingHole, MountingHole:MountingHole_2.2mm_M2_DIN965, F.Cu at (116.7, 81.0)
- added H15: MountingHole, MountingHole:MountingHole_2.2mm_M2_DIN965, F.Cu at (61.9, 119.1)
- added H9: MountingHole, MountingHole:MountingHole_2.2mm_M2_DIN965, F.Cu at (26.2, 42.9)
- C110: footprint Capacitor_SMD:C_0402_1005Metric -> RP2350_80QFN_minimal:C_0402_1005Metric_small_pads
- moved U7 174.6 mm to (71.0, 43.9)
- moved L2 152.4 mm to (99.3, 45.3), turned to -90 degrees
- moved L3 141.7 mm to (99.2, 64.2), turned to -90 degrees
- moved C29 139.3 mm to (93.4, 48.3), turned to 180 degrees
- moved R34 138.5 mm to (87.2, 42.1)
- moved R20 138.1 mm to (86.5, 44.0), turned to 90 degrees
- moved C26 137.6 mm to (94.5, 44.2), turned to -90 degrees
- moved C27 136.5 mm to (87.7, 46.7)
- moved R19 136.2 mm to (85.5, 44.0), turned to -90 degrees
- moved C25 135.6 mm to (92.8, 44.0), turned to -90 degrees
- moved C28 134.9 mm to (96.6, 51.0), turned to 180 degrees
- moved C24 134.0 mm to (72.8, 43.4), turned to -90 degrees
- moved R18 132.2 mm to (85.5, 46.0), turned to -90 degrees
- moved C23 131.6 mm to (69.0, 44.2), turned to -90 degrees
- moved C30 131.2 mm to (84.5, 44.0), turned to 90 degrees
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- renumbered AM1:14 to AM1:12, AM1:12 to AM1:14, AM1:5 to AM1:3, AM1:3 to AM1:5
Connections:
- U2 pad 1: USB1 D+ -> USB2 D+
- U2 pad 2: USB2 D+ -> USB1 D+
- U2 pad 6: USB2 D- -> USB1 D-
- U2 pad 7: USB1 D- -> USB2 D-
Routing:
- net AM1:0: track 0.00 -> 64.5 mm
- net AM1:5: track 0.00 -> 63.6 mm
- net AM1:12: track 0.00 -> 62.1 mm
- net USB2 D+: track 0.00 -> 61.3 mm, vias 0 -> 4
- net USB2 D-: track 0.00 -> 59.8 mm, vias 0 -> 4
- net USB D-: track 0.00 -> 53.8 mm, vias 0 -> 4
- net USB1 D+: track 4.36 -> 58.0 mm, vias 0 -> 2
- net AM1:6: track 0.00 -> 53.1 mm
- net USB1 D-: track 5.67 -> 58.1 mm, vias 0 -> 2
- net USB D+: track 0.00 -> 51.7 mm, vias 0 -> 4
- net AM1:11: track 0.00 -> 50.1 mm
- net AM1:1: track 0.00 -> 45.3 mm
- net AM1:4: track 0.00 -> 40.9 mm
- net AM1:13: track 0.00 -> 38.4 mm
- net GND: track 4.35 -> 40.9 mm, vias 6 -> 46
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- added copper zone on F.Cu, net +3V3
- added copper zone on F.Cu, net +5VA
- added copper zone on F.Cu, net +5VP
- added copper zone on F.Cu, net BS+
- added copper zone on F.Cu, net PD+
- added copper zone on F.Cu, net SW CLEAN
- added copper zone on F.Cu, net SW NOISY
- removed copper zone on F.Cu, net VBUS

Commit message: the letter "gay"
Parts:
- TP1, TP10, TP11, TP12, TP13, TP14, TP15, TP16, TP17, TP18, TP19, TP2, TP20, TP21, TP22, TP23, TP24, TP25, TP26, TP27, TP28, TP29, TP3, TP30, TP31, TP32, TP33, TP34, TP35, TP36, TP37, TP4, TP5, TP6, TP7, TP8, TP9: moved to B.Cu
- moved Q6 57.7 mm to (65.5, 128.9), turned to -90 degrees
- moved R69 45.8 mm to (65.1, 124.3), turned to 180 degrees
- moved R73 41.2 mm to (65.3, 122.3), turned to 90 degrees
- moved TP1 15.2 mm to (139.6, 168.9), turned to 180 degrees
- moved TP2 15.2 mm to (139.6, 171.9), turned to 180 degrees
- moved TP3 15.2 mm to (139.6, 175.0), turned to 180 degrees
- moved TP31 15.2 mm to (124.4, 168.9), turned to 180 degrees
- moved TP32 15.2 mm to (124.4, 171.9), turned to 180 degrees
- moved TP33 15.2 mm to (124.4, 175.0), turned to 180 degrees
- moved TP34 15.2 mm to (124.4, 178.0), turned to 180 degrees
- moved TP35 15.2 mm to (124.4, 181.1), turned to 180 degrees
- moved TP36 15.2 mm to (124.4, 184.1), turned to 180 degrees
- moved TP37 15.2 mm to (139.6, 189.2), turned to 180 degrees
- moved TP4 15.2 mm to (139.6, 178.0), turned to 180 degrees
- moved TP5 15.2 mm to (139.6, 181.1), turned to 180 degrees
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Routing:
- net Net-(Q6-G): track 0.00 -> 4.23 mm
