File: Voided-Oblivion/Voided-Oblivion.kicad_pcb (KiCad board)
At the start: 4 copper layers, 95.3 x 114.3 mm, 425 parts, among them J1 Top male, J10 Sub-Module TL, J11 Sub-Module LT, J12 Sub-Module TR, J16 Sub-Module BL, J17 Sub-Module LB, J18 Sub-Module BR, J19 Sub-Module RB, J2 Top female, J20 Sub-Module RT, J3 Right male, J4 Right female, J5 Left male, J6 Left female, J7 Bottom male, J8 Bottom female, J9 SM03B-SRSS-TB, Q1 AO3401, Q10 BC847B, Q11 BC847B, Q2 AO4407A, Q3 BC857, Q4 AO4407A, Q5 AO4407A, Q6 AO4407A, Q7 AO4407A, Q8 BC847B, Q9 BC847B, SW1 boot, SW2 reset, U1 RP2350_80QFN, U10 TLV431BQDBZR, U11 LM2903, U12 AP2171WG-7, U13 TPD2E2U06DRL, U14 TPD2E2U06DRL, U15 LM66100DCKT, U16 AP2171WG-7, U2 TS3USB30ERSWR, U3 W25Q128JVS, U4 W25Q128JVS, U5 TPS54302, U6 TPS54302, U7 TLV76733DRVR, U8 SN74LVC2T45DCUR, U9 LM66100DCKT, Y1 ABM8-272-T3

Commit message: i swear bro its for the smaller hitbot
Parts:
- added C126: 100nF, Capacitor_SMD:C_0402_1005Metric, F.Cu at (67.7, 68.3)
- added R101: 10kΩ, Resistor_SMD:R_0402_1005Metric, F.Cu at (66.7, 68.4)
- SW1, SW2: footprint Button_Switch_SMD:SW_Push_1P1T_NO_Vertical_Wuerth_434133025816 -> Button_Switch_SMD:SW_Push_1P1T-MP_NO_Horizontal_Alps_SKRTLAE010
- moved H1:5 102.6 mm to (74.7, 36.6)
- moved PD2 83.9 mm to (35.9, 121.2)
- moved H1:6 78.5 mm to (74.7, 55.6)
- moved H1:4 78.5 mm to (93.7, 36.6)
- moved D2 68.6 mm to (48.7, 121.5), turned to 180 degrees
- moved R51 67.0 mm to (34.1, 115.2), turned to 180 degrees
- moved SW1 63.7 mm to (25.9, 86.0)
- moved R50 61.4 mm to (36.1, 118.5)
- moved H1:0 60.2 mm to (93.7, 93.7)
- moved H1:1 60.2 mm to (93.7, 112.8)
- moved H1:12 60.2 mm to (112.8, 93.7)
- moved H1:14 60.2 mm to (112.8, 131.8)
- moved H1:13 60.2 mm to (112.8, 112.8)
- moved H1:2 60.2 mm to (93.7, 131.8)
- moved H1:11 53.9 mm to (112.8, 74.7)
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- renumbered AM1:8 to AM1:0, AM1:7 to AM1:1, AM1:1 to AM1:10, AM1:2 to AM1:11, AM1:3 to AM1:12, AM1:4 to AM1:13, AM1:5 to AM1:14, AM1:6 to AM1:2, AM1:13 to AM1:3, AM1:12 to AM1:4, AM1:11 to AM1:5, AM1:10 to AM1:6, AM1:9 to AM1:7, AM1:14 to AM1:8, AM1:0 to AM1:9
Connections:
- net Net-(D1-A) renamed VBUS1
- net Net-(D2-A) renamed VBUS2
- J1 pad 2: GND -> PD+ TOP
- J1 pad 4: PD+ TOP -> BS+
- J1 pad 5: BS+ -> Net-(J1-Pin_5)
- J1 pad 6: Net-(J1-Pin_6) -> GND
- J2 pad 1: Rx TOP -> GND
- J2 pad 2: BS+ -> Rx TOP
- J2 pad 3: PD+ TOP -> BS+
- J2 pad 5: GND -> PD+ TOP
- J3 pad 2: GND -> PD+ RIGHT
- J3 pad 4: PD+ RIGHT -> BS+
- J3 pad 5: BS+ -> Net-(J3-Pin_5)
- J3 pad 6: Net-(J3-Pin_6) -> GND
- J4 pad 1: Rx RIGHT -> GND
- J4 pad 2: BS+ -> Rx RIGHT
- J4 pad 3: PD+ RIGHT -> BS+
- J4 pad 5: GND -> PD+ RIGHT
- J5 pad 2: GND -> PD+ LEFT
- J5 pad 4: PD+ LEFT -> BS+
- J5 pad 5: BS+ -> Net-(J5-Pin_5)
- J5 pad 6: Net-(J5-Pin_6) -> GND
- J6 pad 1: Rx LEFT -> GND
- J6 pad 2: BS+ -> Rx LEFT
- J6 pad 3: PD+ LEFT -> BS+
- J6 pad 5: GND -> PD+ LEFT
- J7 pad 2: GND -> PD+ BOTTOM
- J7 pad 4: PD+ BOTTOM -> BS+
- J7 pad 5: BS+ -> Net-(J7-Pin_5)
- J7 pad 6: Net-(J7-Pin_6) -> GND
- J8 pad 1: Rx BOTTOM -> GND
- J8 pad 2: BS+ -> Rx BOTTOM
- J8 pad 3: PD+ BOTTOM -> BS+
- J8 pad 5: GND -> PD+ BOTTOM
- R84 pad 1: Net-(J1-Pin_6) -> Net-(J1-Pin_5)
- R85 pad 1: Net-(J3-Pin_6) -> Net-(J3-Pin_5)
- R86 pad 1: Net-(J7-Pin_6) -> Net-(J7-Pin_5)
- R87 pad 1: Net-(J5-Pin_6) -> Net-(J5-Pin_5)
Routing:
- net /~{USB_BOOT}: track 4.12 -> 54.1 mm, vias 0 -> 4
- net AM1:9: track 13.3 -> 62.8 mm
- net /RUN: track 1.10 -> 48.4 mm, vias 0 -> 4
- net AM1:14: track 21.1 -> 67.2 mm
- net AM0: track 0.00 -> 45.2 mm
- net AM1:0: track 64.5 -> 28.7 mm
- net AM1:2: track 27.7 -> 60.7 mm
- net AM1: track 0.00 -> 28.9 mm
- net AM1:12: track 62.1 -> 34.7 mm
- net AM1:7: track 32.9 -> 8.07 mm
- net AM1:4: track 40.9 -> 63.8 mm
- net AM1:6: track 53.1 -> 30.2 mm
- net AM1:11: track 50.1 -> 27.4 mm
- net VBUS2: track 0.00 -> 16.4 mm, vias 0 -> 16
- net /SWCLK: track 16.3 -> 1.40 mm
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- added copper zone on F.Cu, net VBUS2
- added copper zone on In2.Cu, net VBUS2

Commit message: still cis tho
Parts:
- removed D1, D2: SS54, Diode_SMD:D_SMC
- removed R17, R57, R58, R59, R60: 0Ω, Resistor_SMD:R_0402_1005Metric
- added C127: 100nF, Capacitor_SMD:C_0402_1005Metric, F.Cu at (36.0, 121.0)
- added C128: 100nF, Capacitor_SMD:C_0402_1005Metric, F.Cu at (41.6, 120.4)
- added C129: 100nF, Capacitor_SMD:C_0402_1005Metric, F.Cu at (50.9, 35.3)
- added C130: 100nF, Capacitor_SMD:C_0402_1005Metric, F.Cu at (54.1, 38.1)
- added Q13: NCE4009S, Package_SO:SOP-8_3.76x4.96mm_P1.27mm, F.Cu at (40.7, 124.7)
- added Q14: NCE4009S, Package_SO:SOP-8_3.76x4.96mm_P1.27mm, F.Cu at (44.7, 48.0)
- added R102: 0Ω, Resistor_SMD:R_0402_1005Metric, F.Cu at (46.1, 118.9)
- added R103: 0Ω, Resistor_SMD:R_0402_1005Metric, F.Cu at (52.9, 37.9)
- added U17: LM74700QDDF, Package_TO_SOT_SMD:SOT-23-8, F.Cu at (43.8, 119.6)
- added U18: LM74700QDDF, Package_TO_SOT_SMD:SOT-23-8, F.Cu at (49.8, 37.6)
- moved C42 154.5 mm to (44.9, 36.5)
- moved R85 153.6 mm to (124.2, 72.3)
- moved C116 150.8 mm to (95.7, 32.6), turned to -90 degrees
- moved R100 148.5 mm to (73.5, 40.4), turned to -90 degrees
- moved C125 147.2 mm to (75.5, 41.4), turned to 90 degrees
- moved R99 146.1 mm to (74.5, 41.4), turned to 90 degrees
- moved C121 145.2 mm to (112.3, 47.0)
- moved U16 143.8 mm to (112.1, 44.1), turned to 180 degrees
- moved Q4 143.4 mm to (101.0, 31.3)
- moved C120 143.1 mm to (109.5, 45.8), turned to -90 degrees
- moved C124 143.0 mm to (74.3, 43.5), turned to 90 degrees
- moved R98 141.8 mm to (73.3, 43.5), turned to 90 degrees
- moved R97 141.0 mm to (72.2, 42.0)
- moved R71 140.4 mm to (99.4, 34.6)
- moved R96 140.1 mm to (113.2, 41.9), turned to 180 degrees
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Connections:
- AM0 pad 10: Net-(AM0-S0) -> AS0
- AM0 pad 11: Net-(AM0-S1) -> AS1
- AM0 pad 13: Net-(AM0-S3) -> AS3
- AM0 pad 14: Net-(AM0-S2) -> AS2
- AM1 pad 10: Net-(AM1-S0) -> AS0
- AM1 pad 11: Net-(AM1-S1) -> AS1
- AM1 pad 13: Net-(AM1-S3) -> AS3
- AM1 pad 14: Net-(AM1-S2) -> AS2
- R53 pad 1: Net-(AM1-S3) -> AS3
- R53 pad 2: AS3 -> Net-(U1-GPIO11)
- R54 pad 1: Net-(AM1-S2) -> AS2
- R54 pad 2: AS2 -> Net-(U1-GPIO10)
- R55 pad 1: Net-(AM1-S1) -> AS1
- R55 pad 2: AS1 -> Net-(U1-GPIO9)
- R56 pad 1: Net-(AM1-S0) -> AS0
- R56 pad 2: AS0 -> Net-(U1-GPIO8)
- U1 pad 6: AS0 -> Net-(U1-GPIO8)
- U1 pad 7: AS1 -> Net-(U1-GPIO9)
- U1 pad 8: AS2 -> Net-(U1-GPIO10)
- U1 pad 9: AS3 -> Net-(U1-GPIO11)
- U2 pad 8: Net-(U2-~{OE}) -> GND
Routing:
- net VBUS: track 0.00 -> 133.7 mm, vias 0 -> 84
- net Net-(J16-Pin_1): track 0.00 -> 130.4 mm, vias 0 -> 1
- net Net-(J18-Pin_1): track 0.00 -> 87.3 mm, vias 0 -> 1
- net VBUS2: track 16.4 -> 81.4 mm, vias 16 -> 20
- net Net-(J10-Pin_1): track 0.00 -> 62.3 mm, vias 0 -> 1
- net Net-(J12-Pin_1): track 0.00 -> 54.5 mm, vias 0 -> 1
- net AS3: track 0.00 -> 51.6 mm, vias 0 -> 3
- net AS2: track 0.00 -> 50.0 mm, vias 0 -> 3
- net AS1: track 0.00 -> 46.7 mm, vias 0 -> 3
- net SM+: track 0.00 -> 46.0 mm
- net AS0: track 0.00 -> 45.0 mm, vias 0 -> 3
- net Net-(U1-GPIO8): track 0.00 -> 33.0 mm, vias 0 -> 2
- net Net-(U1-GPIO9): track 0.00 -> 32.7 mm, vias 0 -> 2
- net TL ID: track 0.00 -> 32.1 mm, vias 0 -> 2
- net Net-(U1-GPIO10): track 0.00 -> 31.9 mm, vias 0 -> 2
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- added copper zone on B.Cu, net BS+
- added copper zone on B.Cu, net PD+
- added copper zone on F.Cu, net PD+ BOTTOM
- added copper zone on B.Cu, net PD+ LEFT
- added copper zone on F.Cu, net PD+ LEFT
- added copper zone on F.Cu, net PD+ RIGHT
- added copper zone on F.Cu, net PD+ TOP
- added copper zone on B.Cu, net VBUS
- added copper zone on F.Cu, net VBUS
- added copper zone on B.Cu, net VBUS1
- added copper zone on F.Cu, net VBUS1
- added copper zone on In1.Cu, net VBUS1
- added copper zone on In2.Cu, net VBUS1
- added copper zone on B.Cu, net VBUS2
- added copper zone on In1.Cu, net VBUS2
