File: Voided-Oblivion/Voided-Oblivion.kicad_pcb (KiCad board)
At the start: 4 copper layers, 95.3 x 114.3 mm, 427 parts, among them J1 Top male, J10 Sub-Module TL, J11 Sub-Module LT, J12 Sub-Module TR, J16 Sub-Module BL, J17 Sub-Module LB, J18 Sub-Module BR, J19 Sub-Module RB, J2 Top female, J20 Sub-Module RT, J3 Right male, J4 Right female, J5 Left male, J6 Left female, J7 Bottom male, J8 Bottom female, J9 SM03B-SRSS-TB, Q1 AO3401, Q10 BC847B, Q11 BC847B, Q13 NCE4009S, Q14 NCE4009S, Q2 AO4407A, Q3 BC857, Q4 AO4407A, Q5 AO4407A, Q6 AO4407A, Q7 AO4407A, Q8 BC847B, Q9 BC847B, SW1 boot, SW2 reset, U1 RP2350_80QFN, U10 TLV431BQDBZR, U11 LM2903, U12 AP2171WG-7, U13 TPD2E2U06DRL, U14 TPD2E2U06DRL, U15 LM66100DCKT, U16 AP2171WG-7, U17 LM74700QDDF, U18 LM74700QDDF, U2 TS3USB30ERSWR, U3 W25Q128JVS, U4 W25Q128JVS, U5 TPS54302, U6 TPS54302, U7 TLV76733DRVR, U8 SN74LVC2T45DCUR, U9 LM66100DCKT, Y1 ABM8-272-T3

Commit message: BOMB update  (ignore the "B" on the end of that first word, it has no significant meaning) and some library linking
Parts:
- R75, R76, R77, R78: value 10kΩ -> 4.7kΩ
Routing:
- net GND: track 515.6 -> 539.7 mm
- net +3V3: track 435.7 -> 438.5 mm, vias 111 -> 110
