File: Voided-Oblivion/Voided-Oblivion.kicad_sch (KiCad schematic)
At the start: 39 parts, among them J4 SM03B-SRSS-TB, SW1 boot, SW2 reset, U1 RP2350_80QFN, U3 W25Q128JVS, U4 W25Q128JVS, Y1 ABM8-272-T3

Commit message: update.com
Parts:
- added C110, C111, C112, C113: 100n, Capacitor_SMD:C_0402_1005Metric, symbol Device:C
Connections:
- net +1V1: now also C110.1, C111.1
- net +3V3: now also C112.1, C113.1
- net GND: now also C110.2, C111.2, C112.2, C113.2
- net LED SCK: now reaches U1.43 (GPIO34)
- net LED TX: now reaches U1.44 (GPIO35)
- net AM0: now reaches U1.49 (GPIO40_ADC0)
- net AM1: now reaches U1.52 (GPIO41_ADC1)
- net AS0: now reaches U1.6 (GPIO8)
- net AS1: now reaches U1.7 (GPIO9)
- net AS2: now reaches U1.8 (GPIO10)
- net AS3: now reaches U1.9 (GPIO11)

Commit message: update
Parts:
- C10, C6, C7, C9: LCSC (none) -> C23733; MPN (none) -> CL05A475MP5NRNC; Manufacturer (none) -> Samsung Electro-Mechanics
- C11, C110, C111, C112, C113, C12, C13, C14, C15, C16, C17, C18, C2, C20, C21, C8: LCSC (none) -> C307331; MPN (none) -> CL05B104KB54PNC; Manufacturer (none) -> Samsung Electro-Mechanics
- C19: LCSC (none) -> C95841; MPN (none) -> CL21B106KOQNNNE; Manufacturer (none) -> Samsung Electro-Mechanics
- C22, R1, R11, R13, R9, U4: BOM Comments (none) -> DNP - do not populate; DNP (none) -> DNP
- C3, C4: LCSC (none) -> C1548; MPN (none) -> 0402CG150J500NT; Manufacturer (none) -> Guangdong Fenghua (FH)
- J4: LCSC (none) -> C160403; MPN (none) -> SM03B-SRSS-TB(LF)(SN); Manufacturer (none) -> JST
- L1: LCSC (none) -> C3221749; MPN (none) -> VLS201610CX-3R3M-1; Manufacturer (none) -> TDK
- R10: LCSC (none) -> C17168; MPN (none) -> 0402WGF0000TCE; Manufacturer (none) -> UNI-ROYAL
- R2, R4, R6: LCSC (none) -> C11702; MPN (none) -> 0402WGF1001TCE; Manufacturer (none) -> UNI-ROYAL
- R3: LCSC (none) -> C138002; MPN (none) -> RC0402FR-0733RL; Manufacturer (none) -> Yageo
- R7, R8: LCSC (none) -> C138021; MPN (none) -> RC0402FR-0727RL; Manufacturer (none) -> Yageo
- U1: LCSC (none) -> C42415655; MPN (none) -> RP2350B; Manufacturer (none) -> Raspberry Pi
- U3: LCSC (none) -> C97521; MPN (none) -> W25Q128JVSIQ; Manufacturer (none) -> Winbond
- Y1: LCSC (none) -> C20625731; MPN (none) -> ABM8-272-T3; Manufacturer (none) -> Abracon

Commit message: i think the schematic is acctualy done this time, (besides little tiny things)
Parts:
- removed R9: DNP, Resistor_SMD:R_0402_1005Metric, symbol Device:R
- added C122, C123, C124, C125: 100nF, Capacitor_SMD:C_0402_1005Metric, symbol Device:C
- added J1: Top male, Pogo-Pins:PG-6P-2.5-5.5H-SM-RA-Male, symbol Connector:Conn_01x06_Pin
- added J10: Sub-Module TL, symbol Connector:Conn_01x05_Socket
- added J11: Sub-Module LT, symbol Connector:Conn_01x05_Socket
- added J12: Sub-Module TR, symbol Connector:Conn_01x05_Socket
- added J16: Sub-Module BL, symbol Connector:Conn_01x05_Socket
- added J17: Sub-Module LB, symbol Connector:Conn_01x05_Socket
- added J18: Sub-Module BR, symbol Connector:Conn_01x05_Socket
- added J19: Sub-Module RB, symbol Connector:Conn_01x05_Socket
- added J2: Top female, Pogo-Pins:PG-6P-2.5-5.5H-SM-RA-Female, symbol Connector:Conn_01x06_Socket
- added J20: Sub-Module RT, symbol Connector:Conn_01x05_Socket
- added J3: Right male, Pogo-Pins:PG-6P-2.5-5.5H-SM-RA-Male, symbol Connector:Conn_01x06_Pin
- added J4: Right female, Pogo-Pins:PG-6P-2.5-5.5H-SM-RA-Female, symbol Connector:Conn_01x06_Socket
- added J5: Left male, Pogo-Pins:PG-6P-2.5-5.5H-SM-RA-Male, symbol Connector:Conn_01x06_Pin
- added J6: Left female, Pogo-Pins:PG-6P-2.5-5.5H-SM-RA-Female, symbol Connector:Conn_01x06_Socket
- added J7: Bottom male, Pogo-Pins:PG-6P-2.5-5.5H-SM-RA-Male, symbol Connector:Conn_01x06_Pin
- added J8: Bottom female, Pogo-Pins:PG-6P-2.5-5.5H-SM-RA-Female, symbol Connector:Conn_01x06_Socket
- added R100, R93, R94, R97: 10kΩ, Resistor_SMD:R_0402_1005Metric, symbol Device:R
- added R23, R5, R98, R99: 1kΩ, Resistor_SMD:R_0402_1005Metric, symbol Device:R
- added R84, R85, R86, R87: 0Ω, Resistor_SMD:R_0402_1005Metric, symbol Device:R
- added R88, R89, R90, R91: 4.7kΩ, Resistor_SMD:R_0402_1005Metric, symbol Device:R
- C10, C6, C7, C9: LCSC C23733 -> (none); MPN CL05A475MP5NRNC -> (none); Manufacturer Samsung Electro-Mechanics -> (none)
- C11, C110, C111, C112, C113, C12, C13, C14, C15, C16, C17, C18, C2, C20, C21, C8: LCSC C307331 -> (none); MPN CL05B104KB54PNC -> (none); Manufacturer Samsung Electro-Mechanics -> (none)
- C19: LCSC C95841 -> (none); MPN CL21B106KOQNNNE -> (none); Manufacturer Samsung Electro-Mechanics -> (none)
- C22, U4: BOM Comments DNP - do not populate -> (none); DNP DNP -> (none)
- C3, C4: LCSC C1548 -> (none); MPN 0402CG150J500NT -> (none); Manufacturer Guangdong Fenghua (FH) -> (none)
- J9: renamed from J4; LCSC C160403 -> (none); MPN SM03B-SRSS-TB(LF)(SN) -> (none); Manufacturer JST -> (none)
- L1: LCSC C3221749 -> (none); MPN VLS201610CX-3R3M-1 -> (none); Manufacturer TDK -> (none)
- R1, R13: value DNP -> 10kΩ; BOM Comments DNP - do not populate -> (none); DNP DNP -> (none)
- R10: value 0 -> 0Ω; LCSC C17168 -> (none); MPN 0402WGF0000TCE -> (none); Manufacturer UNI-ROYAL -> (none)
- R11: value DNP -> 0Ω; BOM Comments DNP - do not populate -> (none); DNP DNP -> (none)
- R2, R4, R6: value 1k -> 1kΩ; LCSC C11702 -> (none); MPN 0402WGF1001TCE -> (none); Manufacturer UNI-ROYAL -> (none)
- R3: value 33 -> 33Ω; LCSC C138002 -> (none); MPN RC0402FR-0733RL -> (none); Manufacturer Yageo -> (none)
- R7, R8: value 27 -> 27Ω; LCSC C138021 -> (none); MPN RC0402FR-0727RL -> (none); Manufacturer Yageo -> (none)
- U1: LCSC C42415655 -> (none); MPN RP2350B -> (none); Manufacturer Raspberry Pi -> (none)
- U3: LCSC C97521 -> (none); MPN W25Q128JVSIQ -> (none); Manufacturer Winbond -> (none)
- Y1: LCSC C20625731 -> (none); MPN ABM8-272-T3 -> (none); Manufacturer Abracon -> (none)
Connections:
- net GPIO0 is gone; now on net FLASH CS1n: R11.1
- net +3V3: now also R100.1, R93.1, R94.1, R97.1
- net GND: now also C122.2, C123.2, C124.2, C125.2, J1.1 (Pin_1), J1.2 (Pin_2), J10.2 (Pin_2), J11.2 (Pin_2), J12.2 (Pin_2), J16.2 (Pin_2), J17.2 (Pin_2), J18.2 (Pin_2), J19.2 (Pin_2), J2.5 (Pin_5), J2.6 (Pin_6), J20.2 (Pin_2), J3.1 (Pin_1), J3.2 (Pin_2), J4.5 (Pin_5), J4.6 (Pin_6), J5.1 (Pin_1), J5.2 (Pin_2), J6.5 (Pin_5), J6.6 (Pin_6), J7.1 (Pin_1), J7.2 (Pin_2), J8.5 (Pin_5), J8.6 (Pin_6), R88.2, R89.2, R90.2, R91.2
- net Tx TOP: now reaches U1.1 (GPIO4)
- net Tx TOP: now also R84.2
- net Tx BOTTOM: now reaches U1.11 (GPIO12)
- net Tx BOTTOM: now also R86.2
- net Rx BOTTOM: now reaches U1.12 (GPIO13)
- net Rx BOTTOM: now also J8.1 (Pin_1), R89.1
- net Tx LEFT: now reaches U1.16 (GPIO16)
- net Tx LEFT: now also R87.2
- net Rx LEFT: now reaches U1.17 (GPIO17)
- net Rx LEFT: now also J6.1 (Pin_1), R90.1
- net FLASH CS1n: now reaches U1.19 (GPIO19)
- net Rx TOP: now reaches U1.2 (GPIO5)
- net Rx TOP: now also J2.1 (Pin_1), R91.1
- net TL Tx: now reaches U1.22 (GPIO22)
- net TL Tx: now also J10.5 (Pin_5), J11.5 (Pin_5)
- net TL Rx: now reaches U1.23 (GPIO23)
- net TL Rx: now also J10.4 (Pin_4), J11.4 (Pin_4)
- net TR Tx: now reaches U1.25 (GPIO24)
- net TR Tx: now also J12.5 (Pin_5), J20.5 (Pin_5)
- net TR Rx: now reaches U1.26 (GPIO25)
- net TR Rx: now also J12.4 (Pin_4), J20.4 (Pin_4)
- net BR Tx: now reaches U1.27 (GPIO26)
- net BR Tx: now also J18.5 (Pin_5), J19.5 (Pin_5)
- net BR Rx: now reaches U1.28 (GPIO27)
- net BR Rx: now also J18.4 (Pin_4), J19.4 (Pin_4)
- net Tx RIGHT: now reaches U1.3 (GPIO6)
- net Tx RIGHT: now also R85.2
- net BL Tx: now reaches U1.36 (GPIO28)
- net BL Tx: now also J16.5 (Pin_5), J17.5 (Pin_5)
- net BL Rx: now reaches U1.37 (GPIO29)
- net BL Rx: now also J16.4 (Pin_4), J17.4 (Pin_4)
- net Rx RIGHT: now reaches U1.4 (GPIO7)
- net Rx RIGHT: now also J4.1 (Pin_1), R88.1
- net SM BS EN: now reaches U1.40 (GPIO32)
- net SM+ EN: now reaches U1.42 (GPIO33)
- net BS+ SRC: now reaches U1.45 (GPIO36)
- net SM+ FLT: now reaches U1.46 (GPIO37)
- net TL ID: now reaches U1.53 (GPIO42_ADC2)
- net TL ID: now also C125.1, R99.1
- net TR ID: now reaches U1.54 (GPIO43_ADC3)
- net TR ID: now also C124.1, R98.1
- net BR ID: now reaches U1.55 (GPIO44_ADC4)
- net BR ID: now also C122.1, R5.1
- net BL ID: now reaches U1.56 (GPIO45_ADC5)
- net BL ID: now also C123.1, R23.1
- net PD EN TOP: now reaches U1.77 (GPIO0)
- net PD EN RIGHT: now reaches U1.78 (GPIO1)
- net PD EN BOTTOM: now reaches U1.79 (GPIO2)
- net PD EN LEFT: now reaches U1.80 (GPIO3)
- new net: J12.1 (Pin_1), J20.1 (Pin_1), R97.2, R98.2
- new net: J3.6 (Pin_6), R85.1
- new net: J1.6 (Pin_6), R84.1
- new net: J16.1 (Pin_1), J17.1 (Pin_1), R23.2, R94.2
- new net: J10.1 (Pin_1), J11.1 (Pin_1), R100.2, R99.2
- new net: J18.1 (Pin_1), J19.1 (Pin_1), R5.2, R93.2
- new net: J5.6 (Pin_6), R87.1
- new net: J7.6 (Pin_6), R86.1
- new net BS+: J1.5 (Pin_5), J2.2 (Pin_2), J3.5 (Pin_5), J4.2 (Pin_2), J5.5 (Pin_5), J6.2 (Pin_2), J7.5 (Pin_5), J8.2 (Pin_2)
- new net PD BOTTOM: J7.3 (Pin_3), J7.4 (Pin_4), J8.3 (Pin_3), J8.4 (Pin_4)
- new net PD LEFT: J5.3 (Pin_3), J5.4 (Pin_4), J6.3 (Pin_3), J6.4 (Pin_4)
- new net PD RIGHT: J3.3 (Pin_3), J3.4 (Pin_4), J4.3 (Pin_3), J4.4 (Pin_4)
- new net PD TOP: J1.3 (Pin_3), J1.4 (Pin_4), J2.3 (Pin_3), J2.4 (Pin_4)
- new net SM+: J10.3 (Pin_3), J11.3 (Pin_3), J12.3 (Pin_3), J16.3 (Pin_3), J17.3 (Pin_3), J18.3 (Pin_3), J19.3 (Pin_3), J20.3 (Pin_3)
Other:
- note added: "Inter tile/Sub-Module connections"
- note added: "Optional Secondary flash or PSRAM (U4), using the second chip select (XIP_SS_N[1]) on GPIO19. N.B. Pull-up R13 will be required as GPIOs default to pull-downs at power-up."
- note removed: "Optional Secondary flash or PSRAM (U4), using the second chip select (XIP_SS_N[1]) on GPIO0. N.B. Pull-up R13 will be required as GPIOs default to pull-downs at power-up."
- moved on the sheet: C10, C11, C110, C111, C112, C113, C12, C13, C14, C15, C16, C17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

Commit message: drc rules and stuff
Parts:
- added H1, H2, H3, H4, H5, H6, H7: MountingHole, MountingHole:MountingHole_2.2mm_M2_DIN965, symbol Mechanical:MountingHole
- added H8: MountingHole_Pad, MountingHole:MountingHole_2.2mm_M2_DIN965_Pad, symbol Mechanical:MountingHole_Pad
- C10, C6, C7, C9: value 4.7u -> 4.7µF; LCSC (none) -> C23733; MPN (none) -> CL05A475MP5NRNC; Manufacturer (none) -> Samsung Electro-Mechanics
- C11, C110, C111, C112, C113, C12, C13, C14, C15, C16, C17, C18, C2, C20, C21, C8: value 100n -> 100nF; LCSC (none) -> C307331; MPN (none) -> CL05B104KB54PNC; Manufacturer (none) -> Samsung Electro-Mechanics
- C122, C123, C124, C125: LCSC (none) -> C307331; MPN (none) -> CL05B104KB54PNC; Manufacturer (none) -> Samsung Electro-Mechanics
- C19: value 10u -> 10µF; footprint Capacitor_SMD:C_0805_2012Metric -> Capacitor_SMD:C_1206_3216Metric; LCSC (none) -> C95841; MPN (none) -> CL21B106KOQNNNE; Manufacturer (none) -> Samsung Electro-Mechanics
- C22: value DNP -> 100nF; LCSC (none) -> C307331
- C3, C4: LCSC (none) -> C1548; MPN (none) -> 0402CG150J500NT; Manufacturer (none) -> FH (Guangdong Fenghua)
- J10, J11, J12, J16, J17, J18, J19, J20: footprint (none) -> Voided-Oblivion-misc:5-pin-machined-female-pin-headers-sunk
- J9: LCSC (none) -> C160403; MPN (none) -> SM03B-SRSS-TB(LF)(SN); Manufacturer (none) -> JST Sales America
- L1: LCSC (none) -> C3221749; MPN (none) -> VLS201610CX-3R3M-1; Manufacturer (none) -> TDK
- R1: now in the parts list
- R10, R84, R85, R86, R87: LCSC (none) -> C17168; MPN (none) -> 0402WGF0000TCE; Manufacturer (none) -> UNI-ROYAL(Uniroyal Elec)
- R100, R93, R94, R97: LCSC (none) -> C25744; MPN (none) -> 0402WGF1002TCE; Manufacturer (none) -> UNI-ROYAL(Uniroyal Elec)
- R2, R23, R4, R5, R6, R98, R99: LCSC (none) -> C11702; MPN (none) -> 0402WGF1001TCE; Manufacturer (none) -> UNI-ROYAL(Uniroyal Elec)
- R3: LCSC (none) -> C138002; MPN (none) -> RC0402FR-0733RL; Manufacturer (none) -> YAGEO
- R7, R8: LCSC (none) -> C138021; MPN (none) -> RC0402FR-0727RL; Manufacturer (none) -> YAGEO
- R88, R89, R90, R91: LCSC (none) -> C25900; MPN (none) -> 0402WGF4701TCE; Manufacturer (none) -> UNI-ROYAL(Uniroyal Elec)
- U1: LCSC (none) -> C42415655; MPN (none) -> RP2350B; Manufacturer (none) -> Raspberry Pi
- U3: LCSC (none) -> C97521; MPN (none) -> W25Q128JVSIQ; Manufacturer (none) -> Winbond Elec
- Y1: LCSC (none) -> C20625731; MPN (none) -> ABM8-272-T3; Manufacturer (none) -> Abracon LLC
Connections:
- net GND: now also H8.1
- net MCU D+: now reaches R7.2, U1.67 (USB_DP)
- net MCU D-: now reaches R8.2, U1.66 (USB_DM)
- net PD BOTTOM renamed PD+ BOTTOM
- net PD LEFT renamed PD+ LEFT
- net PD RIGHT renamed PD+ RIGHT
- net PD TOP renamed PD+ TOP

Commit message: checkpoint
Parts:
- added TP1, TP10, TP11, TP12, TP13, TP14, TP15, TP16, TP17, TP18, TP19, TP2, TP20, TP21, TP22, TP23, TP24, TP25, TP26, TP27, TP28, TP29, TP3, TP30, TP31, TP32, TP33, TP34, TP35, TP36, TP4, TP5, TP6, TP7, TP8, TP9: TestPoint, TestPoint:TestPoint_Pad_D1.0mm, symbol Connector:TestPoint
Connections:
- net +1V1: now also TP7.1
- net +3V3: now also TP6.1
- net +5VP EN: now also TP21.1
- net AS0: now also TP29.1
- net AS1: now also TP30.1
- net AS2: now also TP31.1
- net AS3: now also TP32.1
- net BS+: now also TP2.1
- net BS+ SRC: now also TP3.1
- net GND: now also TP10.1, TP11.1, TP12.1, TP13.1
- net LED SCK: now also TP33.1
- net LED TX: now also TP34.1
- net PD EN BOTTOM: now also TP24.1
- net PD EN LEFT: now also TP25.1
- net PD EN RIGHT: now also TP23.1
- net PD EN TOP: now also TP22.1
- net PD1 INT: now also TP16.1
- net PD1 SCL: now also TP15.1
- net PD1 SDA: now also TP14.1
- net PD2 INT: now also TP19.1
- net PD2 SCL: now also TP18.1
- net PD2 SDA: now also TP17.1
- net RUN: now also TP35.1
- net SM BS EN: now also TP26.1
- net SM+: now also TP8.1
- net SM+ EN: now also TP27.1
- net ~{USB_BOOT}: now also TP36.1
- new net +5VA: TP4.1
- new net +5VA EN: TP20.1
- new net +5VP: TP5.1
- new net PD+: TP1.1
- new net USB SEL: TP28.1
- new net VBUS: TP9.1

Commit message: blaaa why does placeing and routing things take so looonnggggggggg >:c
Parts:
- added H10, H11, H12, H13, H14, H15, H9: MountingHole, MountingHole:MountingHole_2.2mm_M2_DIN965, symbol Mechanical:MountingHole
- C110: footprint Capacitor_SMD:C_0402_1005Metric -> RP2350_80QFN_minimal:C_0402_1005Metric_small_pads

Commit message: i swear bro its for the smaller hitbot
Parts:
- added C126: 100nF, Capacitor_SMD:C_0402_1005Metric, symbol Device:C
- added R101: 10kΩ, Resistor_SMD:R_0402_1005Metric, symbol Device:R
- SW1, SW2: footprint Button_Switch_SMD:SW_Push_1P1T_NO_Vertical_Wuerth_434133025816 -> Button_Switch_SMD:SW_Push_1P1T-MP_NO_Horizontal_Alps_SKRTLAE010; symbol Switch:SW_Push -> Voided-Oblivion-misc:SW_Push_Shielded; LCSC (none) -> C110293
Connections:
- net +3V3: now also R101.1
- net BS+: now also J1.4 (Pin_4), J2.3 (Pin_3), J3.4 (Pin_4), J4.3 (Pin_3), J5.4 (Pin_4), J6.3 (Pin_3), J7.4 (Pin_4), J8.3 (Pin_3); no longer J1.5 (Pin_5), J2.2 (Pin_2), J3.5 (Pin_5), J4.2 (Pin_2), J5.5 (Pin_5), J6.2 (Pin_2), J7.5 (Pin_5), J8.2 (Pin_2)
- net GND: now also J1.6 (Pin_6), J2.1 (Pin_1), J3.6 (Pin_6), J4.1 (Pin_1), J5.6 (Pin_6), J6.1 (Pin_1), J7.6 (Pin_6), J8.1 (Pin_1), SW1.MP (B), SW2.MP (B), C126.1; no longer J1.2 (Pin_2), J2.5 (Pin_5), J3.2 (Pin_2), J4.5 (Pin_5), J5.2 (Pin_2), J6.5 (Pin_5), J7.2 (Pin_2), J8.5 (Pin_5)
- net PD+ BOTTOM: now also J7.2 (Pin_2), J8.5 (Pin_5); no longer J7.4 (Pin_4), J8.3 (Pin_3)
- net PD+ LEFT: now also J5.2 (Pin_2), J6.5 (Pin_5); no longer J5.4 (Pin_4), J6.3 (Pin_3)
- net PD+ RIGHT: now also J3.2 (Pin_2), J4.5 (Pin_5); no longer J3.4 (Pin_4), J4.3 (Pin_3)
- net PD+ TOP: now also J1.2 (Pin_2), J2.5 (Pin_5); no longer J1.4 (Pin_4), J2.3 (Pin_3)
- net RUN: now also C126.2, R101.2
- net Rx BOTTOM: now also J8.2 (Pin_2); no longer J8.1 (Pin_1)
- net Rx LEFT: now also J6.2 (Pin_2); no longer J6.1 (Pin_1)
- net Rx RIGHT: now also J4.2 (Pin_2); no longer J4.1 (Pin_1)
- net Rx TOP: now also J2.2 (Pin_2); no longer J2.1 (Pin_1)
- net at R85.1: now also J3.5 (Pin_5); no longer J3.6 (Pin_6)
- net at R84.1: now also J1.5 (Pin_5); no longer J1.6 (Pin_6)
- net at R87.1: now also J5.5 (Pin_5); no longer J5.6 (Pin_6)
- net at R86.1: now also J7.5 (Pin_5); no longer J7.6 (Pin_6)
Other:
- moved on the sheet: C122, C123, C125, R5, R84, R85, R86, R87, R88, R89, R90, R91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

Commit message: still cis tho
Parts:
- added R53, R54, R55, R56: 0Ω, Resistor_SMD:R_0402_1005Metric, symbol Device:R
Connections:
- net AS0: now also R56.1; no longer U1.6 (GPIO8)
- net AS1: now also R55.1; no longer U1.7 (GPIO9)
- net AS2: now also R54.1; no longer U1.8 (GPIO10)
- net AS3: now also R53.1; no longer U1.9 (GPIO11)
- new net: R56.2, U1.6 (GPIO8)
- new net: R55.2, U1.7 (GPIO9)
- new net: R53.2, U1.9 (GPIO11)
- new net: R54.2, U1.8 (GPIO10)
