File: Voided-Oblivion/Voided-Oblivion.kicad_sch (KiCad schematic)
At the start: 135 parts, among them J1 Top male, J10 Sub-Module TL, J11 Sub-Module LT, J12 Sub-Module TR, J16 Sub-Module BL, J17 Sub-Module LB, J18 Sub-Module BR, J19 Sub-Module RB, J2 Top female, J20 Sub-Module RT, J3 Right male, J4 Right female, J5 Left male, J6 Left female, J7 Bottom male, J8 Bottom female, J9 SM03B-SRSS-TB, SW1 boot, SW2 reset, U1 RP2350_80QFN, U3 W25Q128JVS, U4 W25Q128JVS, Y1 ABM8-272-T3

Commit message: pcb almooost done
Parts:
- removed H1, H10: MountingHole, MountingHole:MountingHole_2.2mm_M2_DIN965, symbol Mechanical:MountingHole
Connections:
- no-connect marks 0 -> 1
Changed lines of the file:
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@@
 		(color 0 0 0 0)
 	)
+	(no_connect
+		(at 250.19 273.05)
+	)
 	(wire
 		(pts
@@
 	)
 	(symbol
-		(lib_id "Mechanical:MountingHole")
-		(at 314.96 180.34 0)
-		(unit 1)
-		(body_style 1)
-		(exclude_from_sim no)
-		(in_bom no)
-		(on_board yes)
-		(in_pos_files yes)
-		(dnp no)
-		(fields_autoplaced yes)
-		(property "Reference" "H1"
-			(at 317.5 179.0699 0)
-			(show_name no)
-			(do_not_autoplace no)
-			(effects
-				(font
-					(size 1.27 1.27)
-				)
-				(justify left)
-			)
-		)
-		(property "Value" "MountingHole"
-			(at 317.5 181.6099 0)
-			(hide yes)
-			(show_name no)
-			(do_not_autoplace no)
-			(effects
-				(font
-					(size 1.27 1.27)
-				)
-				(justify left)
-			)
-		)
-		(property "Footprint" "MountingHole:MountingHole_2.2mm_M2_DIN965"
-			(at 314.96 180.34 0)
-			(hide yes)
-			(show_name no)
-			(do_not_autoplace no)
-			(effects
-				(font
-					(size 1.27 1.27)
-				)
-			)
-		)
-		(property "Datasheet" ""
-			(at 314.96 180.34 0)
-			(hide yes)
-			(show_name no)
-			(do_not_autoplace no)
-			(effects
-				(font
-					(size 1.27 1.27)
-				)
-			)
-		)
-		(property "Description" "Mounting Hole without connection"
-			(at 314.96 180.34 0)
-			(hide yes)
-			(show_name no)
-			(do_not_autoplace no)
-			(effects
-				(font
-					(size 1.27 1.27)
-				)
-			)
-		)
-		(instances
-			(project "Voided-Oblivion"
-				(path "/d39297fe-343b-4cf0-9c31-a16e101c76da"
-					(reference "H1")
-					(unit 1)
-				)
-			)
-		)
-	)
-	(symbol
 		(lib_id "Voided-Oblivion-misc:SW_Push_Shielded")
 		(at 130.81 180.34 0)
@@
 					(unit 1)
 				)
-			)
-		)
-	)
-	(symbol
-		(lib_id "Mechanical:MountingHole")
-		(at 335.28 185.42 0)
-		(unit 1)
-		(body_style 1)
-		(exclude_from_sim no)
-		(in_bom no)
-		(on_board yes)
-		(in_pos_files yes)
-		(dnp no)
-		(fields_autoplaced yes)
-		(property "Reference" "H10"
-			(at 337.82 184.1499 0)
-			(show_name no)
-			(do_not_autoplace no)
-			(effects
-				(font
-					(size 1.27 1.27)
-				)
-				(justify left)
-			)
-		)
-		(property "Value" "MountingHole"
-			(at 337.82 186.6899 0)
-			(hide yes)
-			(show_name no)
-			(do_not_autoplace no)
-			(effects
-				(font
-					(size 1.27 1.27)
-				)
-				(justify left)
-			)
-		)
-		(property "Footprint" "MountingHole:MountingHole_2.2mm_M2_DIN965"
-			(at 335.28 185.42 0)
-			(hide yes)
-			(show_name no)
-			(do_not_autoplace no)
-			(effects
-				(font
-					(size 1.27 1.27)
-				)
-			)
-		)
-		(property "Datasheet" ""
-			(at 335.28 185.42 0)
-			(hide yes)
-			(show_name no)
-			(do_not_autoplace no)
-			(effects
-				(font
-					(size 1.27 1.27)
-				)
-			)
-		)
-		(property "Description" "Mounting Hole without connection"
-			(at 335.28 185.42 0)
-			(hide yes)
-			(show_name no)
-			(do_not_autoplace no)
-			(effects
-				(font
-					(size 1.27 1.27)
-				)
-			)
-		)
-		(instances
-			(project "Voided-Oblivion"
-				(path "/d39297fe-343b-4cf0-9c31-a16e101c76da"
-					(reference "H10")
-					(unit 1)
-				)

Commit message: THE PCB IS FINAWWYY (electricaly) DONE YAAAAAAAAAAAAAA :33333 ^w^ >w<
Connections:
- no-connect marks 1 -> 0
Changed lines of the file:
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@@
 		(color 0 0 0 0)
-	)
-	(no_connect
-		(at 250.19 273.05)
 	)
 	(wire

Commit message: small changes
Parts:
- removed H6: MountingHole, MountingHole:MountingHole_2.2mm_M2_DIN965, symbol Mechanical:MountingHole
- C10, C11, C111, C112, C113, C12, C122, C123, C124, C125, C126, C13, C14, C15, C16, C17, C18, C2, C20, C21, C22, C3, C4, C8, C9: footprint Capacitor_SMD:C_0402_1005Metric -> Voided-Oblivion-misc:C_0402_1005Metric-no-silkscreen-text
- R1, R10, R100, R101, R11, R13, R2, R23, R3, R4, R5, R53, R54, R55, R56, R6, R7, R8, R84, R85, R86, R87, R88, R89, R90, R91, R93, R94, R97, R98, R99: footprint Resistor_SMD:R_0402_1005Metric -> Voided-Oblivion-misc:R_0402_1005Metric-no-silkscreen-text

Commit message: BOMB update  (ignore the "B" on the end of that first word, it has no significant meaning) and some library linking
Parts:
- C19: LCSC C95841 -> C89632; MPN CL21B106KOQNNNE -> CL31B106KBHNNNE
- SW1, SW2: MPN (none) -> SKRTLAE010; Manufacturer (none) -> ALPSALPINE
Connections:
- no-connect marks 0 -> 4
Changed lines of the file:
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@@
 		(color 0 0 0 0)
 	)
+	(no_connect
+		(at 232.41 223.52)
+	)
+	(no_connect
+		(at 232.41 248.92)
+	)
+	(no_connect
+		(at 232.41 246.38)
+	)
+	(no_connect
+		(at 232.41 226.06)
+	)
 	(wire
 		(pts
@@
 			)
 		)
-		(property "LCSC" "C95841"
+		(property "LCSC" "C89632"
 			(at 259.08 138.43 0)
 			(hide yes)
@@
 			)
 		)
-		(property "MPN" "CL21B106KOQNNNE"
+		(property "MPN" "CL31B106KBHNNNE"
 			(at 259.08 138.43 0)
 			(hide yes)
@@
 			)
 		)
+		(property "Manufacturer" "ALPSALPINE"
+			(at 0 0 0)
+			(hide yes)
+			(show_name no)
+			(do_not_autoplace no)
+			(effects
+				(font
+					(size 1.27 1.27)
+				)
+			)
+		)
+		(property "MPN" "SKRTLAE010"
+			(at 0 0 0)
+			(hide yes)
+			(show_name no)
+			(do_not_autoplace no)
+			(effects
+				(font
+					(size 1.27 1.27)
+				)
+			)
+		)
 		(pin "1"
 		)
@@
 			(hide yes)
 			(show_name no)
+			(do_not_autoplace no)
+			(effects
+				(font
+					(size 1.27 1.27)
+				)
+			)
+		)
+		(property "Manufacturer" "ALPSALPINE"
+			(at 0 0 0)
+			(hide yes)
+			(show_name no)
+			(do_not_autoplace no)
+			(effects
+				(font
+					(size 1.27 1.27)
+				)
+			)
+		)
+		(property "MPN" "SKRTLAE010"
+			(at 0 0 0)
+			(hide yes)
+			(show_name no)

Commit message: this is gonna be a fun murge :meltingface:
Parts:
- removed TP20: TestPoint, TestPoint:TestPoint_Pad_D1.0mm, symbol Connector:TestPoint
- added FID1, FID2, FID3, FID4, FID5, FID6: Fiducial, Fiducial:Fiducial_1mm_Mask3mm, symbol Mechanical:Fiducial
- added H1, H10, H6: ToolingHole, MountingHole:ToolingHole_1.152mm, symbol Mechanical:MountingHole

Commit message: UwU
Parts:
- added TP37: SM BUS, TestPoint:TestPoint_Pad_D1.0mm, symbol Connector:TestPoint
- TP1: value TestPoint -> PD+
- TP10, TP11, TP12, TP13: value TestPoint -> GND
- TP14: value TestPoint -> PD1 SDA
- TP15: value TestPoint -> PD1 SCL
- TP16: value TestPoint -> PD1 INT
- TP17: value TestPoint -> PD2 SDA
- TP18: value TestPoint -> PD2 SCL
- TP19: value TestPoint -> PD2 INT
- TP2: value TestPoint -> BS+
- TP21: value TestPoint -> 5VP EN
- TP22: value TestPoint -> PD T
- TP23: value TestPoint -> PD R
- TP24: value TestPoint -> PD B
- TP25: value TestPoint -> PD L
- TP26: value TestPoint -> SM BS EN
- TP27: value TestPoint -> SM+ EN
- TP28: value TestPoint -> USB SEL
- TP29: value TestPoint -> AS0
- TP3: value TestPoint -> BS+ SRC
- TP30: value TestPoint -> AS1
- TP31: value TestPoint -> AS2
- TP32: value TestPoint -> AS3
- TP33: value TestPoint -> LED SCK
- TP34: value TestPoint -> LED TX
- TP35: value TestPoint -> RUN
- TP36: value TestPoint -> BOOT
- TP4: value TestPoint -> +5VA
- TP5: value TestPoint -> +5VP
- TP6: value TestPoint -> +3V3
- TP7: value TestPoint -> +1V1
- TP8: value TestPoint -> SM+
- TP9: value TestPoint -> VBUS
Connections:
- net ~{USB_BOOT} renamed USB BOOT
- new net SM BUS: TP37.1
Other:
- note added: "Misc."
- moved on the sheet: C122, C123, C124, C125, FID1, FID2, FID3, FID4, FID5, FID6, J1, J10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

Commit message: production files i think.com
Parts:
- C110: footprint RP2350_80QFN_minimal:C_0402_1005Metric_small_pads -> Voided-Oblivion-misc:C_0402_1005Metric-no-silkscreen-text
- C22, U4: now left out of the parts list
- L1: LCSC C3221749 -> C42411119; MPN VLS201610CX-3R3M-1 -> AOTA-B201610S3R3-101-T; Manufacturer TDK -> Abracon LLC
- R1, R13: LCSC (none) -> C25744; now left out of the parts list
- R11: LCSC (none) -> C17168
- SW1: value boot -> (none); footprint Button_Switch_SMD:SW_Push_1P1T-MP_NO_Horizontal_Alps_SKRTLAE010 -> Button_Switch_SMD:SW_SPST_EVQP7C; symbol Voided-Oblivion-misc:SW_Push_Shielded -> Switch:SW_Push; LCSC C110293 -> C388883; MPN SKRTLAE010 -> EVQ-P7C01P; Manufacturer ALPSALPINE -> Panasonic
- SW2: value reset -> (none); footprint Button_Switch_SMD:SW_Push_1P1T-MP_NO_Horizontal_Alps_SKRTLAE010 -> Button_Switch_SMD:SW_SPST_EVQP7C; symbol Voided-Oblivion-misc:SW_Push_Shielded -> Switch:SW_Push; LCSC C110293 -> C388883; MPN SKRTLAE010 -> EVQ-P7C01P; Manufacturer ALPSALPINE -> Panasonic
Connections:
- net GND: no longer SW1.MP (B), SW2.MP (B)
Changed lines of the file:
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@@
 		(body_style 1)
 		(exclude_from_sim no)
-		(in_bom yes)
+		(in_bom no)
 		(on_board yes)
-		(in_pos_files yes)
+		(in_pos_files no)
 		(dnp yes)
 		(property "Reference" "R1"
@@
 			)
 		)
+		(property "LCSC" "C25744"
+			(at 50.8 129.54 90)
+			(hide yes)
+			(show_name no)
+			(do_not_autoplace no)
+			(effects
+				(font
+					(size 1.27 1.27)
+				)
+			)
+		)
 		(pin "1"
 		)
@@
 		(body_style 1)
 		(exclude_from_sim no)
-		(in_bom yes)
+		(in_bom no)
 		(on_board yes)
-		(in_pos_files yes)
+		(in_pos_files no)
 		(dnp yes)
 		(property "Reference" "C22"
@@
 	)
 	(symbol
-		(lib_id "Voided-Oblivion-misc:SW_Push_Shielded")
+		(lib_id "Switch:SW_Push")
 		(at 130.81 180.34 0)
 		(unit 1)
@@
 			)
 		)
-		(property "Value" "reset"
+		(property "Value" ""
 			(at 130.81 175.26 0)
 			(show_name no)
@@
 			)
 		)
-		(property "Footprint" "Button_Switch_SMD:SW_Push_1P1T-MP_NO_Horizontal_Alps_SKRTLAE010"
+		(property "Footprint" "Button_Switch_SMD:SW_SPST_EVQP7C"
 			(at 130.81 175.26 0)
 			(hide yes)
@@
 			)
 		)
-		(property "Description" ""
-			(at 130.81 180.34 0)
+		(property "Description" "reset"
+			(at 130.81 175.26 0)
 			(show_name no)
 			(do_not_autoplace no)
@@
 			)
 		)
-		(property "LCSC" "C110293"
+		(property "LCSC" "C388883"
 			(at 130.81 180.34 0)
 			(hide yes)
@@
 			)
 		)
-		(property "Manufacturer" "ALPSALPINE"
+		(property "Manufacturer" "Panasonic"
 			(at 0 0 0)
 			(hide yes)
@@
 			)
 		)
-		(property "MPN" "SKRTLAE010"
+		(property "MPN" "EVQ-P7C01P"
 			(at 0 0 0)
 			(hide yes)
@@
 		(pin "2"
 		)
-		(pin "MP"
-		)
 		(instances
 			(project "Voided-Oblivion"
@@
 			)
 		)
+		(property "LCSC" "C17168"
+			(at 35.56 195.58 90)
+			(hide yes)
+			(show_name no)
+			(do_not_autoplace no)
+			(effects
+				(font
+					(size 1.27 1.27)
+				)
+			)
+		)
 		(pin "1"
 		)
@@
 			)
 		)
-		(property "LCSC" "C3221749"
+		(property "LCSC" "C42411119"
 			(at 132.08 123.19 0)
 			(hide yes)
@@
 			)
 		)
-		(property "MPN" "VLS201610CX-3R3M-1"
+		(property "MPN" "AOTA-B201610S3R3-101-T"
 			(at 132.08 123.19 0)
 			(hide yes)
@@
 			)
 		)
-		(property "Manufacturer" "TDK"
+		(property "Manufacturer" "Abracon LLC"
 			(at 132.08 123.19 0)
 			(hide yes)
@@
 		(body_style 1)
 		(exclude_from_sim no)
-		(in_bom yes)
+		(in_bom no)
 		(on_board yes)
-		(in_pos_files yes)
+		(in_pos_files no)
 		(dnp yes)
 		(fields_autoplaced yes)
@@
 	(symbol
 		(lib_id "power:GND")
-		(at 130.81 184.15 0)
-		(unit 1)
-		(body_style 1)
-		(exclude_from_sim no)
-		(in_bom yes)
-		(on_board yes)
-		(in_pos_files yes)
-		(dnp no)
-		(property "Reference" "#PWR0227"
-			(at 130.81 190.5 0)
-			(hide yes)
-			(show_name no)
-			(do_not_autoplace no)
-			(effects
-				(font
-					(size 1.27 1.27)
-				)
-			)
-		)
-		(property "Value" "GND"
-			(at 130.937 188.5442 0)
-			(show_name no)
-			(do_not_autoplace no)
-			(effects
-				(font
-					(size 1.27 1.27)
-				)
-			)
-		)
-		(property "Footprint" ""
-			(at 130.81 184.15 0)
-			(hide yes)
-			(show_name no)
-			(do_not_autoplace no)
-			(effects
-				(font
-					(size 1.27 1.27)
-				)
-			)
-		)
-		(property "Datasheet" ""
-			(at 130.81 184.15 0)
-			(hide yes)
-			(show_name no)
-			(do_not_autoplace no)
-			(effects
-				(font
-					(size 1.27 1.27)
-				)
-			)
-		)
-		(property "Description" ""
-			(at 130.81 184.15 0)
-			(show_name no)
-			(do_not_autoplace no)
-			(effects
-				(font
-					(size 1.27 1.27)
-				)
-			)
-		)
-		(pin "1"
-		)
-		(instances
-			(project "Voided-Oblivion"
-				(path "/d39297fe-343b-4cf0-9c31-a16e101c76da"
-					(reference "#PWR0227")
-					(unit 1)
-				)
-			)
-		)
-	)
-	(symbol
-		(lib_id "power:GND")
 		(at 105.41 133.35 0)
 		(mirror y)
@@
 	)
 	(symbol
-		(lib_id "power:GND")
-		(at 130.81 146.05 90)
-		(unit 1)
-		(body_style 1)
-		(exclude_from_sim no)
-		(in_bom yes)
-		(on_board yes)
-		(in_pos_files yes)
-		(dnp no)
-		(property "Reference" "#PWR0226"
-			(at 137.16 146.05 0)
-			(hide yes)
-			(show_name no)
-			(do_not_autoplace no)
-			(effects
-				(font
-					(size 1.27 1.27)
-				)
-			)
-		)
-		(property "Value" "GND"
-			(at 135.2042 145.923 0)
-			(show_name no)
-			(do_not_autoplace no)
-			(effects
-				(font
-					(size 1.27 1.27)
-				)
-			)
-		)
-		(property "Footprint" ""
-			(at 130.81 146.05 0)
-			(hide yes)
-			(show_name no)
-			(do_not_autoplace no)
-			(effects
-				(font
-					(size 1.27 1.27)
-				)
-			)
-		)
-		(property "Datasheet" ""
-			(at 130.81 146.05 0)
-			(hide yes)
-			(show_name no)
-			(do_not_autoplace no)
-			(effects
-				(font
-					(size 1.27 1.27)
-				)
-			)
-		)
-		(property "Description" ""
-			(at 130.81 146.05 0)
-			(show_name no)
-			(do_not_autoplace no)
-			(effects
-				(font
-					(size 1.27 1.27)
-				)
-			)
-		)
-		(pin "1"
-		)
-		(instances
-			(project "Voided-Oblivion"
-				(path "/d39297fe-343b-4cf0-9c31-a16e101c76da"
-					(reference "#PWR0226")
-					(unit 1)
-				)
-			)
-		)
-	)
-	(symbol
 		(lib_id "Mechanical:MountingHole")
 		(at 314.96 190.5 0)
@@
 	)
 	(symbol
-		(lib_id "Voided-Oblivion-misc:SW_Push_Shielded")
+		(lib_id "Switch:SW_Push")
 		(at 127 146.05 90)
 		(unit 1)
@@
 		(in_pos_files yes)
 		(dnp no)
+		(fields_autoplaced yes)
 		(property "Reference" "SW1"
-			(at 119.888 144.272 90)
+			(at 128.27 144.7799 90)
 			(show_name no)
 			(do_not_autoplace no)
@@
 			)
 		)
-		(property "Value" "boot"
-			(at 119.634 148.082 90)
+		(property "Value" ""
+			(at 128.27 147.3199 90)
 			(show_name no)
 			(do_not_autoplace no)
@@
 			)
 		)
-		(property "Footprint" "Button_Switch_SMD:SW_Push_1P1T-MP_NO_Horizontal_Alps_SKRTLAE010"
+		(property "Footprint" "Button_Switch_SMD:SW_SPST_EVQP7C"
 			(at 121.92 146.05 0)
 			(hide yes)
@@
 			)
 		)
-		(property "Description" ""
-			(at 127 146.05 0)
+		(property "Description" "boot"
+			(at 128.27 147.3199 90)
 			(show_name no)
 			(do_not_autoplace no)
@@
 					(size 1.27 1.27)
 				)
+				(justify right)
 			)
 		)
-		(property "LCSC" "C110293"
+		(property "LCSC" "C388883"
 			(at 127 146.05 90)
 			(hide yes)
@@
 			)
 		)
-		(property "Manufacturer" "ALPSALPINE"
+		(property "Manufacturer" "Panasonic"
 			(at 0 0 0)
 			(hide yes)
@@
 			)
 		)
-		(property "MPN" "SKRTLAE010"
+		(property "MPN" "EVQ-P7C01P"
 			(at 0 0 0)
 			(hide yes)
@@
 		(pin "2"
 		)
-		(pin "MP"
-		)
 		(instances
 			(project "Voided-Oblivion"
@@
 			)
 		)
-		(property "Footprint" "RP2350_80QFN_minimal:C_0402_1005Metric_small_pads"
+		(property "Footprint" "Voided-Oblivion-misc:C_0402_1005Metric-no-silkscreen-text"
 			(at 130.5052 85.09 0)
 			(hide yes)
@@
 		(body_style 1)
 		(exclude_from_sim no)
-		(in_bom yes)
+		(in_bom no)
 		(on_board yes)
-		(in_pos_files yes)
+		(in_pos_files no)
 		(dnp yes)
 		(property "Reference" "R13"
@@
 			(show_name no)
 			(do_not_autoplace no)
+			(effects
+				(font
+					(size 1.27 1.27)
+				)
+			)
+		)
+		(property "LCSC" "C25744"
+			(at 52.07 187.96 90)
+			(hide yes)
+			(show_name no)
+			(do_not_autoplace no)

Commit message: boring licence stuff
Parts:
- C22: now fitted; now in the parts list
- R11: now fitted
- R13: now in the parts list
- U4: LCSC (none) -> C97521; now fitted; now in the parts list
Other:
- note added: "not nessisary for this spisific flash"
Changed lines of the file:
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@@
 		)
 	)
+	(text "not nessisary for \nthis spisific flash"
+		(exclude_from_sim no)
+		(at 35.56 187.96 0)
+		(effects
+			(font
+				(size 1.27 1.27)
+			)
+		)
+	)
 	(text "Secondary Flash/PSRAM"
 		(exclude_from_sim no)
@@
 		)
 	)
+	(text "not nessisary for \nthis spisific flash"
+		(exclude_from_sim no)
+		(at 34.29 129.54 0)
+		(effects
+			(font
+				(size 1.27 1.27)
+			)
+		)
+	)
 	(text "JST Debug Connector"
 		(exclude_from_sim no)
@@
 		)
 	)
+	(polyline
+		(pts
+			(xy 46.99 186.69) (xy 48.26 187.96)
+		)
+		(stroke
+			(width 0)
+			(type default)
+		)
+	)
 	(wire
 		(pts
@@
 		)
 	)
+	(polyline
+		(pts
+			(xy 43.18 129.54) (xy 46.99 129.54)
+		)
+		(stroke
+			(width 0)
+			(type default)
+		)
+	)
 	(wire
 		(pts
@@
 		)
 	)
+	(polyline
+		(pts
+			(xy 45.72 128.27) (xy 46.99 129.54)
+		)
+		(stroke
+			(width 0)
+			(type default)
+		)
+	)
 	(wire
 		(pts
@@
 		)
 	)
+	(polyline
+		(pts
+			(xy 48.26 187.96) (xy 46.99 189.23)
+		)
+		(stroke
+			(width 0)
+			(type default)
+		)
+	)
 	(wire
 		(pts
@@
 		)
 	)
+	(polyline
+		(pts
+			(xy 46.99 129.54) (xy 45.72 130.81)
+		)
+		(stroke
+			(width 0)
+			(type default)
+		)
+	)
 	(wire
 		(pts
@@
 		)
 	)
+	(polyline
+		(pts
+			(xy 44.45 187.96) (xy 48.26 187.96)
+		)
+		(stroke
+			(width 0)
+			(type default)
+		)
+	)
 	(wire
 		(pts
@@
 		(body_style 1)
 		(exclude_from_sim no)
-		(in_bom no)
+		(in_bom yes)
 		(on_board yes)
-		(in_pos_files no)
-		(dnp yes)
+		(in_pos_files yes)
+		(dnp no)
 		(property "Reference" "C22"
 			(at 75.311 182.9816 0)
@@
 		(on_board yes)
 		(in_pos_files yes)
-		(dnp yes)
+		(dnp no)
 		(property "Reference" "R11"
 			(at 37.465 195.58 90)
@@
 		(body_style 1)
 		(exclude_from_sim no)
-		(in_bom no)
+		(in_bom yes)
 		(on_board yes)
-		(in_pos_files no)
-		(dnp yes)
+		(in_pos_files yes)
+		(dnp no)
 		(fields_autoplaced yes)
 		(property "Reference" "U4"
@@
 			)
 		)
+		(property "LCSC" "C97521"
+			(at 66.04 203.2 0)
+			(hide yes)
+			(show_name no)
+			(do_not_autoplace no)
+			(effects
+				(font
+					(size 1.27 1.27)
+				)
+			)
+		)
 		(pin "4"
 		)
@@
 		(body_style 1)
 		(exclude_from_sim no)
-		(in_bom no)
+		(in_bom yes)
 		(on_board yes)
 		(in_pos_files no)
