File: Voided-Oblivion/power.kicad_sch (KiCad schematic)
At the start: 76 parts, among them Q1 AO3401, Q2 AO4407A, Q3 BC857, U10 TLV431, U11 LM2903, U2 TS3USB30ERSWR, U5 TPS54302, U6 TPS54302, U7 XC6220B331MR, U9 MAX40203

Commit message: update.com
Parts:
- added C114, C115: 100nF, Capacitor_SMD:C_0402_1005Metric, symbol Device:C
- C23, C24, C25, C26, C27, C28, C29, C30, C31, C32, C33, C34, C35, C36, C37, C38, C39, C40, C41, C42, C43, C44, C45: footprint (none) -> Capacitor_SMD:C_0402_1005Metric
- R12, R14, R15, R17, R18, R19, R20, R21, R22, R24, R25, R26, R27, R28, R29, R30, R31, R32, R33, R34, R35, R36, R37, R38, R39, R40, R41, R42, R43, R44, R45, R46, R47: footprint (none) -> Resistor_SMD:R_0402_1005Metric
- USB1, USB2: footprint (none) -> Connector_USB:USB_C_Receptacle_Molex_105450-0101
Connections:
- net +3V3: now also C115.2
- net +5VA: now also C114.1
- net GND: now also C114.2, C115.1

Commit message: update
Parts:
- removed C41: 100µF, Capacitor_SMD:C_0402_1005Metric, symbol Device:C
- removed D3: BZV55B5V1, Diode_SMD:D_MiniMELF, symbol Diode:BZV55B5V1
- removed U7: XC6220B331MR, Package_TO_SOT_SMD:SOT-23-5, symbol Regulator_Linear:XC6220B331MR
- added D3: BZV55B3V3, Diode_SMD:D_MiniMELF, symbol Diode:BZV55B3V3
- added D5: BZX84C10, Package_TO_SOT_SMD:SOT-23, symbol Diode:BZX84Cxx
- added R48, R49, R50, R51: 100Ω, Resistor_SMD:R_0402_1005Metric, symbol Device:R
- added U13, U14: TPD2E2U06DRL, Package_TO_SOT_SMD:SOT-553, symbol Power_Protection:TPD2E2U06DRL
- added U7: TLV76733DRVR, Package_SON:WSON-6-1EP_2x2mm_P0.65mm_EP1x1.6mm_ThermalVias, symbol Regulator_Linear:TLV76733DRVx
- C114, C115, C25, C27, C32, C33, C38, C39, C42, C43, C44: LCSC (none) -> C307331; MPN (none) -> CL05B104KB54PNC; Manufacturer (none) -> Samsung Electro-Mechanics
- C23: LCSC (none) -> C23733; MPN (none) -> CL05A475MP5NRNC; Manufacturer (none) -> Samsung Electro-Mechanics
- C24: value 10µF -> 1µF; footprint Capacitor_SMD:C_0402_1005Metric -> Capacitor_SMD:C_0805_2012Metric; LCSC (none) -> C24123; MPN (none) -> CL21B105KOFNNNE; Manufacturer (none) -> Samsung Electro-Mechanics
- C26, C31: footprint Capacitor_SMD:C_0402_1005Metric -> Capacitor_SMD:C_1206_3216Metric; LCSC (none) -> C89632; MPN (none) -> CL31B106KBHNNNE; Manufacturer (none) -> Samsung Electro-Mechanics
- C28, C29, C34, C35: footprint Capacitor_SMD:C_0402_1005Metric -> Capacitor_SMD:C_1206_3216Metric; LCSC (none) -> C12891; MPN (none) -> CL31A226KAHNNNE; Manufacturer (none) -> Samsung Electro-Mechanics
- C30, C36: LCSC (none) -> C83711; MPN (none) -> 0402CGR75C500NT; Manufacturer (none) -> Guangdong Fenghua (FH)
- C37: LCSC (none) -> C53547; MPN (none) -> 0402CG102J500NT; Manufacturer (none) -> Guangdong Fenghua (FH); now not fitted; now left out of the parts list
- C40: LCSC (none) -> C315248; MPN (none) -> CL05A106MP5NUNC; Manufacturer (none) -> Samsung Electro-Mechanics
- C45: LCSC (none) -> C53547; MPN (none) -> 0402CG102J500NT; Manufacturer (none) -> Guangdong Fenghua (FH)
- D1, D2: LCSC (none) -> C18199188; MPN (none) -> SS54C; Manufacturer (none) -> R+O
- D4: LCSC (none) -> C19077470; MPN (none) -> BZX84C10; Manufacturer (none) -> R+O
- PD1, PD2: LCSC (none) -> C132291; MPN (none) -> FUSB302BMPX; Manufacturer (none) -> onsemi
- Q1: LCSC C181091 -> C15127; MPN (none) -> AO3401A; Manufacturer (none) -> Alpha & Omega Semiconductor
- Q2: MPN (none) -> AO4407A; Manufacturer (none) -> Alpha & Omega Semiconductor
- Q3: LCSC (none) -> C20069137; MPN (none) -> BC857C; Manufacturer (none) -> R+O
- R12, R14, R15, R17, R27: LCSC (none) -> C17168; MPN (none) -> 0402WGF0000TCE; Manufacturer (none) -> UNI-ROYAL
- R18, R24: LCSC (none) -> C49654456; MPN (none) -> GR0402F49R9TAG00; Manufacturer (none) -> GiantOhm
- R19, R25, R32, R34, R38, R39, R47: LCSC (none) -> C25741; MPN (none) -> 0402WGF1003TCE; Manufacturer (none) -> UNI-ROYAL
- R20, R26: LCSC (none) -> C2974007; MPN (none) -> FRC0402F1332TS; Manufacturer (none) -> FOJAN
- R21: LCSC (none) -> C25765; MPN (none) -> 0402WGF2002TCE; Manufacturer (none) -> UNI-ROYAL
- R22, R29, R33, R36, R37: LCSC (none) -> C25744; MPN (none) -> 0402WGF1002TCE; Manufacturer (none) -> UNI-ROYAL
- R28: BOM Comments (none) -> DNP - do not populate; DNP (none) -> DNP
- R35, R46: LCSC (none) -> C26083; MPN (none) -> 0402WGF1004TCE; Manufacturer (none) -> UNI-ROYAL
- R40, R41, R42, R43: LCSC (none) -> C25900; MPN (none) -> 0402WGF4701TCE; Manufacturer (none) -> UNI-ROYAL
- R44, R45: value 100kΩ -> 4.7kΩ; LCSC (none) -> C25900; MPN (none) -> 0402WGF4701TCE; Manufacturer (none) -> UNI-ROYAL
- U10: value TLV431 -> TLV431B; LCSC (none) -> C398374; MPN (none) -> TLV431BQDBZR; Manufacturer (none) -> Texas Instruments
- U11: MPN (none) -> LM2903DR; Manufacturer (none) -> Texas Instruments
- U2: LCSC (none) -> C73880; MPN (none) -> TS3USB30ERSWR; Manufacturer (none) -> Texas Instruments
- U5, U6: LCSC (none) -> C311983; MPN (none) -> TPS54302DDCR; Manufacturer (none) -> Texas Instruments
- U9: LCSC (none) -> C5668579; MPN (none) -> MAX40203ANS+T; Manufacturer (none) -> Analog Devices (Maxim)
- USB1, USB2: LCSC (none) -> C134092; MPN (none) -> 1054500101; Manufacturer (none) -> Molex
Connections:
- net +3V3: now also U7.1 (OUT), U7.2 (SNS)
- net BS+: now also R12.2, U7.6 (IN); no longer R12.1
- net GND: now also D3.2 (A), U13.4, U14.4, U7.3 (GND), U7.5 (GND), U7.7 (PAD)
- net USB SEL: now also D3.1 (K)
- net VBUS: now also D5.3 (K)
- net at PD1.1 (CC2), PD1.14 (CC2): now also R49.1; no longer USB1.A5 (CC1)
- net USB1 D+: now reaches U2.1 (D1+), USB1.A6 (D+), USB1.B6 (D+)
- net USB1 D+: now also U13.3
- net USB1 D-: now reaches U2.7 (D1-), USB1.A7 (D-), USB1.B7 (D-)
- net USB1 D-: now also U13.5
- net at PD1.10 (CC1), PD1.11 (CC1): now also R48.2; no longer USB1.B5 (CC2)
- net at C45.1, Q1.1 (G), R35.2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: now also D5.1 (A)
- net at PD2.1 (CC2), PD2.14 (CC2): now also R51.1; no longer USB2.A5 (CC1)
- net USB2 D+: now reaches U2.2 (D2+), USB2.A6 (D+), USB2.B6 (D+)
- net USB2 D+: now also U14.3
- net USB2 D-: now reaches U2.6 (D2-), USB2.A7 (D-), USB2.B7 (D-)
- net USB2 D-: now also U14.5
- net at PD2.10 (CC1), PD2.11 (CC1): now also R50.2; no longer USB2.B5 (CC2)
- new net: R12.1, U7.4 (EN)
- new net: R49.2, USB1.A5 (CC1)
- new net: R48.1, USB1.B5 (CC2)
- new net: R51.2, USB2.A5 (CC1)
- new net: R50.1, USB2.B5 (CC2)
- no-connect marks 20 -> 24
Other:
- note added: "place as close to the connector as physically possible"
- moved on the sheet: R12

Commit message: i think the schematic is acctualy done this time, (besides little tiny things)
Parts:
- removed U9: MAX40203, Package_BGA:WLP-4_0.728x0.728mm_Layout2x2_P0.35mm, symbol Analog_Switch:MAX40200ANS
- added C116, C117, C118, C119: 100nF, Capacitor_SMD:C_0402_1005Metric, symbol Device:C
- added C120, C41, C76: 1µF, Capacitor_SMD:C_0402_1005Metric, symbol Device:C
- added C121, C77: 10µF, Capacitor_SMD:C_0402_1005Metric, symbol Device:C
- added Q10, Q11, Q8, Q9: BC847B, Package_TO_SOT_SMD:SOT-23, symbol Transistor_BJT:BC847
- added Q4, Q5, Q6, Q7: AO4407A, Package_SO:SOP-8_3.76x4.96mm_P1.27mm, symbol Transistor_FET:FDS9435A
- added R16: 0Ω, Resistor_SMD:R_0402_1005Metric, symbol Device:R
- added R67, R68, R69, R70, R79, R80, R81, R82, R83, R96: 100kΩ, Resistor_SMD:R_0402_1005Metric, symbol Device:R
- added R71, R72, R73, R74, R92, R95: 4.7kΩ, Resistor_SMD:R_0402_1005Metric, symbol Device:R
- added R75, R76, R77, R78: 10kΩ, Resistor_SMD:R_0402_1005Metric, symbol Device:R
- added U12, U16: AP2171WG-7, Package_TO_SOT_SMD:SOT-23-5, symbol Power_Management:AP2171W
- added U15, U9: LM66100DCKT, Package_TO_SOT_SMD:SOT-363_SC-70-6, symbol Power_Management:LM66100DCK
- C114: value 100nF -> 1µF; LCSC C307331 -> (none); MPN CL05B104KB54PNC -> (none); Manufacturer Samsung Electro-Mechanics -> (none)
- C115, C25, C27, C32, C33, C38, C39, C42, C43, C44: LCSC C307331 -> (none); MPN CL05B104KB54PNC -> (none); Manufacturer Samsung Electro-Mechanics -> (none)
- C23: LCSC C23733 -> (none); MPN CL05A475MP5NRNC -> (none); Manufacturer Samsung Electro-Mechanics -> (none)
- C24: footprint Capacitor_SMD:C_0805_2012Metric -> Capacitor_SMD:C_0402_1005Metric; LCSC C24123 -> (none); MPN CL21B105KOFNNNE -> (none); Manufacturer Samsung Electro-Mechanics -> (none)
- C26, C31: footprint Capacitor_SMD:C_1206_3216Metric -> Capacitor_SMD:C_0402_1005Metric; LCSC C89632 -> (none); MPN CL31B106KBHNNNE -> (none); Manufacturer Samsung Electro-Mechanics -> (none)
- C28, C29, C34, C35: footprint Capacitor_SMD:C_1206_3216Metric -> Capacitor_SMD:C_0402_1005Metric; LCSC C12891 -> (none); MPN CL31A226KAHNNNE -> (none); Manufacturer Samsung Electro-Mechanics -> (none)
- C30, C36: LCSC C83711 -> (none); MPN 0402CGR75C500NT -> (none); Manufacturer Guangdong Fenghua (FH) -> (none)
- C37, C45: LCSC C53547 -> (none); MPN 0402CG102J500NT -> (none); Manufacturer Guangdong Fenghua (FH) -> (none)
- C40: LCSC C315248 -> (none); MPN CL05A106MP5NUNC -> (none); Manufacturer Samsung Electro-Mechanics -> (none)
- D1, D2: LCSC C18199188 -> (none); MPN SS54C -> (none); Manufacturer R+O -> (none)
- D3: LCSC C545375 -> (none); MPN BZV55B3V3 -> (none); Manufacturer LGE -> (none)
- D4, D5: LCSC C19077470 -> (none); MPN BZX84C10 -> (none); Manufacturer R+O -> (none)
- PD1, PD2: LCSC C132291 -> (none); MPN FUSB302BMPX -> (none); Manufacturer onsemi -> (none)
- Q1: LCSC C15127 -> C181091; MPN AO3401A -> (none); Manufacturer Alpha & Omega Semiconductor -> (none)
- Q2: MPN AO4407A -> (none); Manufacturer Alpha & Omega Semiconductor -> (none)
- Q3: LCSC C20069137 -> (none); MPN BC857C -> (none); Manufacturer R+O -> (none)
- R12, R14, R15, R17, R27: LCSC C17168 -> (none); MPN 0402WGF0000TCE -> (none); Manufacturer UNI-ROYAL -> (none)
- R18, R24: LCSC C49654456 -> (none); MPN GR0402F49R9TAG00 -> (none); Manufacturer GiantOhm -> (none)
- R19, R25, R32, R34, R38, R39, R47: LCSC C25741 -> (none); MPN 0402WGF1003TCE -> (none); Manufacturer UNI-ROYAL -> (none)
- R20, R26: LCSC C2974007 -> (none); MPN FRC0402F1332TS -> (none); Manufacturer FOJAN -> (none)
- R21: LCSC C25765 -> (none); MPN 0402WGF2002TCE -> (none); Manufacturer UNI-ROYAL -> (none)
- R22, R29, R33, R36, R37: LCSC C25744 -> (none); MPN 0402WGF1002TCE -> (none); Manufacturer UNI-ROYAL -> (none)
- R28: BOM Comments DNP - do not populate -> (none); DNP DNP -> (none)
- R35, R46: LCSC C26083 -> (none); MPN 0402WGF1004TCE -> (none); Manufacturer UNI-ROYAL -> (none)
- R40, R41, R42, R43, R44, R45: LCSC C25900 -> (none); MPN 0402WGF4701TCE -> (none); Manufacturer UNI-ROYAL -> (none)
- R48, R49, R50, R51: LCSC C25076 -> (none); MPN 0402WGF1000TCE -> (none); Manufacturer UNI-ROYAL -> (none)
- U10: LCSC C398374 -> (none); MPN TLV431BQDBZR -> (none); Manufacturer Texas Instruments -> (none)
- U11: MPN LM2903DR -> (none); Manufacturer Texas Instruments -> (none)
- U13, U14: LCSC C1972959 -> (none); MPN TPD2E2U06DRLR -> (none); Manufacturer Texas Instruments -> (none)
- U2: LCSC C73880 -> (none); MPN TS3USB30ERSWR -> (none); Manufacturer Texas Instruments -> (none)
- U5, U6: LCSC C311983 -> (none); MPN TPS54302DDCR -> (none); Manufacturer Texas Instruments -> (none)
- U7: LCSC C2848334 -> (none); MPN TLV76733DRVR -> (none); Manufacturer Texas Instruments -> (none)
- USB1, USB2: LCSC C134092 -> (none); MPN 1054500101 -> (none); Manufacturer Molex -> (none)
Connections:
- net +3V3: now also R83.2, R96.1
- net +5VA: now also C41.1, U9.1 (VIN); no longer C114.1, R15.1
- net +5VP: now also C114.1, U15.1 (VIN)
- net BS+: now also R15.1, C76.1, U12.5 (IN), U9.6 (VOUT)
- net GND: now also C120.2, C121.1, C41.2, C76.2, C77.1, Q10.2 (E), Q11.2 (E), Q8.2 (E), Q9.2 (E), R79.2, R80.2, R81.2, R82.2, R92.1, R95.1, U12.2 (GND), U15.2 (GND), U16.2 (GND), U9.2 (GND)
- net PD+: now also C116.1, C117.1, C118.1, C119.1, Q4.1 (S), Q4.2 (S), Q4.3 (S), Q5.1 (S), Q5.2 (S), Q5.3 (S), Q6.1 (S), Q6.2 (S), Q6.3 (S), Q7.1 (S), Q7.2 (S), Q7.3 (S), R67.1, R68.1, R69.1, R70.1
- net at R15.2: now also U9.3 (~{CE})
- new net: C120.1, C77.2, R16.1, U12.1 (OUT), U15.6 (VOUT), U16.5 (IN)
- new net: Q9.1 (B), R76.1, R80.1
- new net: Q9.3 (C), R72.2
- new net: R16.2, U15.3 (~{CE})
- new net: C118.2, Q6.4 (G), R69.2, R73.1
- new net: Q8.1 (B), R75.1, R79.1
- new net: Q8.3 (C), R71.2
- new net: C116.2, Q4.4 (G), R67.2, R71.1
- new net: C117.2, Q5.4 (G), R68.2, R72.1
- new net: C119.2, Q7.4 (G), R70.2, R74.1
- new net: Q11.3 (C), R74.2
- new net: Q10.1 (B), R77.1, R81.1
- new net: Q10.3 (C), R73.2
- new net: Q11.1 (B), R78.1, R82.1
- new net BS+ SRC: R83.1, U9.5 (ST)
- new net PD BOTTOM: Q6.5 (D), Q6.6 (D), Q6.7 (D), Q6.8 (D)
- new net PD EN BOTTOM: R77.2
- new net PD EN LEFT: R78.2
- new net PD EN RIGHT: R76.2
- new net PD EN TOP: R75.2
- new net PD LEFT: Q7.5 (D), Q7.6 (D), Q7.7 (D), Q7.8 (D)
- new net PD RIGHT: Q5.5 (D), Q5.6 (D), Q5.7 (D), Q5.8 (D)
- new net PD TOP: Q4.5 (D), Q4.6 (D), Q4.7 (D), Q4.8 (D)
- new net SM BS EN: R92.2, U12.4 (EN)
- new net SM+: C121.2, U16.1 (OUT)
- new net SM+ EN: R95.2, U16.4 (EN)
- new net SM+ FLT: R96.2, U16.3 (~{FLG})
- no-connect marks 24 -> 26
Other:
- note added: "BS+: Bootstrap rail(5V) PD+: Power Delivery rail (9-20V) +5VA: 5V Analog/clean 5V +5VP: 5V Power/Noisy 5V (for rgb) SM+: Sub-Module power (5V)"
- note added: "Bottom"
- note added: "Enable/Disable Sub-modules"
- note added: "Ideal diode to stop BS+ flowing onto +5VP"
- note added: "Left"
- note added: "PD+ Per-Side Switches"
- note added: "Right"
- note added: "Sub-Module Switching"
- note added: "Switch BS+ -> Sub-Modules"
- note added: "Top"
- moved on the sheet: C115, C23, C24, C25, C26, C27, C28, C29, C30, C31, C32, C33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

Commit message: drc rules and stuff
Parts:
- removed U10: TLV431B, Package_TO_SOT_SMD:SOT-23, symbol Reference_Voltage:TL431DBV
- removed USB1, USB2: USB_C_Receptacle, Connector_USB:USB_C_Receptacle_Molex_105450-0101, symbol Connector:USB_C_Receptacle
- added U10: TLV431BQDBZR, Package_TO_SOT_SMD:SOT-23, symbol Reference_Voltage:TL431DBZ
- added USB1, USB2: USB_C_Receptacle_USB2.0_16P, Connector_USB:USB_C_Receptacle_HCTL_HC-TYPE-C-16P-01A, symbol Connector:USB_C_Receptacle_USB2.0_16P
- C114, C120, C24, C41, C76: LCSC (none) -> C52923; MPN (none) -> CL05A105KA5NQNC; Manufacturer (none) -> Samsung Electro-Mechanics
- C115, C116, C117, C118, C119, C38, C39, C44: LCSC (none) -> C307331; MPN (none) -> CL05B104KB54PNC; Manufacturer (none) -> Samsung Electro-Mechanics
- C121, C40, C77: footprint Capacitor_SMD:C_0402_1005Metric -> Capacitor_SMD:C_1206_3216Metric; LCSC (none) -> C315248; MPN (none) -> CL05A106MP5NUNC; Manufacturer (none) -> Samsung Electro-Mechanics
- C23: LCSC (none) -> C23733; MPN (none) -> CL05A475MP5NRNC; Manufacturer (none) -> Samsung Electro-Mechanics
- C25, C27, C32, C33, C42, C43: value 0.1µF -> 100nF; LCSC (none) -> C307331; MPN (none) -> CL05B104KB54PNC; Manufacturer (none) -> Samsung Electro-Mechanics
- C26, C28, C29, C31, C34, C35: footprint Capacitor_SMD:C_0402_1005Metric -> Capacitor_SMD:C_1206_3216Metric
- C30, C36: LCSC (none) -> C37809; MPN (none) -> 0402CG750J500NT; Manufacturer (none) -> FH (Guangdong Fenghua)
- C45: LCSC (none) -> C53547; MPN (none) -> 0402CG102J500NT; Manufacturer (none) -> FH (Guangdong Fenghua)
- D1, D2: LCSC (none) -> C18199188; MPN (none) -> SS54C; Manufacturer (none) -> hongjiacheng
- D3: LCSC (none) -> C545375; MPN (none) -> BZV55B3V3; Manufacturer (none) -> LGE
- D4, D5: LCSC (none) -> C19077470; MPN (none) -> BZX84C10; Manufacturer (none) -> hongjiacheng
- L2, L3: footprint (none) -> Inductor_SMD:L_APV_APH0630; LCSC (none) -> C5349698; MPN (none) -> APH0630T100M; Manufacturer (none) -> APV
- PD1, PD2: LCSC (none) -> C132291; MPN (none) -> FUSB302BMPX; Manufacturer (none) -> onsemi
- Q1: LCSC C181091 -> C15127; MPN (none) -> AO3401A; Manufacturer (none) -> Alpha & Omega Semiconductor
- Q10, Q11, Q8, Q9: LCSC (none) -> C20069135; MPN (none) -> BC847B; Manufacturer (none) -> hongjiacheng
- Q2: MPN (none) -> AO4407A; Manufacturer (none) -> UMW(Youtai Semiconductor)
- Q3: LCSC (none) -> C20069137; MPN (none) -> BC857C; Manufacturer (none) -> hongjiacheng
- Q4, Q5, Q6, Q7: LCSC (none) -> C2841482; MPN (none) -> AO4407A; Manufacturer (none) -> UMW(Youtai Semiconductor)
- R12, R14, R15, R16, R17, R27: LCSC (none) -> C17168; MPN (none) -> 0402WGF0000TCE; Manufacturer (none) -> UNI-ROYAL(Uniroyal Elec)
- R18, R24: LCSC (none) -> C140147; MPN (none) -> RC-02K49R9FT; Manufacturer (none) -> FH (Guangdong Fenghua)
- R19, R25, R32, R34, R38, R39, R47, R67, R68, R69, R70, R79, R80, R81, R82, R83, R96: LCSC (none) -> C25741; MPN (none) -> 0402WGF1003TCE; Manufacturer (none) -> UNI-ROYAL(Uniroyal Elec)
- R20, R26: LCSC (none) -> C2974007; MPN (none) -> FRC0402F1332TS; Manufacturer (none) -> FOJAN
- R21: LCSC (none) -> C25765; MPN (none) -> 0402WGF2002TCE; Manufacturer (none) -> UNI-ROYAL(Uniroyal Elec)
- R22: value 10kΩ -> 5.1kΩ; LCSC (none) -> C25905
- R29, R33, R36, R37, R75, R76, R77, R78: LCSC (none) -> C25744; MPN (none) -> 0402WGF1002TCE; Manufacturer (none) -> UNI-ROYAL(Uniroyal Elec)
- R30: value 44.2kΩ -> 35.7kΩ; LCSC (none) -> C2681604; MPN (none) -> ARG02BTC4422; Manufacturer (none) -> Viking Tech
- R31: value 12.2kΩ -> 10kΩ; LCSC (none) -> C2902636
- R35, R46: LCSC (none) -> C26083; MPN (none) -> 0402WGF1004TCE; Manufacturer (none) -> UNI-ROYAL(Uniroyal Elec)
- R40, R41, R42, R43, R44, R45, R71, R72, R73, R74, R92, R95: LCSC (none) -> C25900; MPN (none) -> 0402WGF4701TCE; Manufacturer (none) -> UNI-ROYAL(Uniroyal Elec)
- R48, R49, R50, R51: LCSC (none) -> C25076; MPN (none) -> 0402WGF1000TCE; Manufacturer (none) -> UNI-ROYAL(Uniroyal Elec)
- U11: MPN (none) -> LM2903DR; Manufacturer (none) -> Texas Instruments
- U12, U16: LCSC (none) -> C110466; MPN (none) -> AP2171WG-7; Manufacturer (none) -> Diodes Incorporated
- U13, U14: LCSC (none) -> C1972959; MPN (none) -> TPD2E2U06DRLR; Manufacturer (none) -> Texas Instruments
- U15, U9: LCSC (none) -> C2832141; MPN (none) -> LM66100DCKT; Manufacturer (none) -> Texas Instruments
- U2: LCSC (none) -> C73880; MPN (none) -> TS3USB30ERSWR; Manufacturer (none) -> Texas Instruments
- U5, U6: LCSC (none) -> C311983; MPN (none) -> TPS54302DDCR; Manufacturer (none) -> Texas Instruments
- U7: LCSC (none) -> C2848334; MPN (none) -> TLV76733DRVR; Manufacturer (none) -> Texas Instruments
Connections:
- net +1V24ref: now also U10.1 (K)
- net GND: now also U10.3 (A), USB1.A1 (GND), USB1.A12 (GND), USB1.B1 (GND), USB1.B12 (GND), USB1.SH (SHIELD), USB2.A1 (GND), USB2.A12 (GND), USB2.B1 (GND), USB2.B12 (GND), USB2.SH (SHIELD)
- net USB1 D+: now also USB1.A6 (D+), USB1.B6 (D+)
- net USB1 D-: now also USB1.A7 (D-), USB1.B7 (D-)
- net USB2 D+: now also USB2.A6 (D+), USB2.B6 (D+)
- net USB2 D-: now also USB2.A7 (D-), USB2.B7 (D-)
- net SM BUS: now reaches C120.1, C77.2, R16.1, U12.1 (OUT), U15.6 (VOUT), U16.5 (IN)
- net at R27.1, R28.2: now also U10.2 (REF)
- net at D1.2 (A), PD1.2 (VBUS): now also USB1.A4 (VBUS), USB1.A9 (VBUS), USB1.B4 (VBUS), USB1.B9 (VBUS)
- net at R49.2: now also USB1.A5 (CC1)
- net at R48.1: now also USB1.B5 (CC2)
- net at D2.2 (A), PD2.2 (VBUS), R37.1: now also USB2.A4 (VBUS), USB2.A9 (VBUS), USB2.B4 (VBUS), USB2.B9 (VBUS)
- net at PD1.10 (CC1), PD1.11 (CC1): now also R49.1; no longer R48.2
- net at PD1.1 (CC2), PD1.14 (CC2): now also R48.2; no longer R49.1
- net at R51.2: now also USB2.A5 (CC1)
- net at R50.1: now also USB2.B5 (CC2)
- net SW NOISY: now reaches C33.2, L3.1, U6.2 (SW)
- net SW CLEAN: now reaches C27.2, L2.1, U5.2 (SW)
- net at PD2.1 (CC2), PD2.14 (CC2): now also R50.2; no longer R51.1
- net at PD2.10 (CC1), PD2.11 (CC1): now also R51.1; no longer R50.2
- net PD BOTTOM renamed PD+ BOTTOM
- net PD LEFT renamed PD+ LEFT
- net PD RIGHT renamed PD+ RIGHT
- net PD TOP renamed PD+ TOP
- no-connect marks 26 -> 10

Commit message: checkpoint
Parts:
- added TP37: TestPoint, TestPoint:TestPoint_Pad_D1.0mm, symbol Connector:TestPoint
Connections:
- net SM BUS: now also TP37.1
Changed lines of the file:
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@@
 	(wire
 		(pts
+			(xy 309.88 100.33) (xy 309.88 110.49)
+		)
+		(stroke
+			(width 0)
+			(type default)
+		)
+	)
+	(wire
+		(pts
 			(xy 38.1 173.99) (xy 43.18 173.99)
 		)
@@
 	)
 	(label "SM BUS"
+		(at 309.88 110.49 90)
+		(effects
+			(font
+				(size 1.27 1.27)
+			)
+			(justify left)
+		)
+	)
+	(label "SM BUS"
 		(at 241.3 228.6 0)
 		(effects
@@
 					(unit 1)
 				)
+			)
+		)
+	)
+	(symbol
+		(lib_id "Connector:TestPoint")
+		(at 309.88 100.33 0)
+		(unit 1)
+		(body_style 1)
+		(exclude_from_sim no)
+		(in_bom yes)
+		(on_board yes)
+		(in_pos_files yes)
+		(dnp no)
+		(property "Reference" "TP37"
+			(at 309.88 95.25 0)
+			(show_name no)
+			(do_not_autoplace no)
+			(effects
+				(font
+					(size 1.27 1.27)
+				)
+			)
+		)
+		(property "Value" "TestPoint"
+			(at 309.88 97.79 0)
+			(hide yes)
+			(show_name no)
+			(do_not_autoplace no)
+			(effects
+				(font
+					(size 1.27 1.27)
+				)
+			)
+		)
+		(property "Footprint" "TestPoint:TestPoint_Pad_D1.0mm"
+			(at 309.88 100.33 0)
+			(hide yes)
+			(show_name no)
+			(do_not_autoplace no)
+			(effects
+				(font
+					(size 1.27 1.27)
+				)
+			)
+		)
+		(property "Datasheet" "~"
+			(at 309.88 100.33 0)
+			(hide yes)
+			(show_name no)
+			(do_not_autoplace no)
+			(effects
+				(font
+					(size 1.27 1.27)
+				)
+			)
+		)
+		(property "Description" "test point"
+			(at 309.88 100.33 0)
+			(hide yes)
+			(show_name no)
+			(do_not_autoplace no)
+			(effects
+				(font
+					(size 1.27 1.27)
+				)
+			)
+		)
+		(pin "1"
+		)
+		(instances
+			(project "Voided-Oblivion"
+				(path "/d39297fe-343b-4cf0-9c31-a16e101c76da/889be6bb-77c0-4884-a2da-d27e1f17090a"
+					(reference "TP37")
+					(unit 1)
+				)

Commit message: blaaa why does placeing and routing things take so looonnggggggggg >:c
Connections:
- net USB1 D+: now also U2.2 (D2+); no longer U2.1 (D1+)
- net USB1 D-: now also U2.6 (D2-); no longer U2.7 (D1-)
- net USB2 D+: now also U2.1 (D1+); no longer U2.2 (D2+)
- net USB2 D-: now also U2.7 (D1-); no longer U2.6 (D2-)

Commit message: i swear bro its for the smaller hitbot
Connections:
- net VBUS2: now reaches D2.2 (A), PD2.2 (VBUS), R37.1, USB2.A4 (VBUS), USB2.A9 (VBUS), USB2.B4 (VBUS), USB2.B9 (VBUS)
- net VBUS1: now reaches D1.2 (A), PD1.2 (VBUS), USB1.A4 (VBUS), USB1.A9 (VBUS), USB1.B4 (VBUS), USB1.B9 (VBUS)
Changed lines of the file:
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@@
+		)
+	)
+	(global_label "VBUS2"
+		(shape input)
+		(at 265.43 162.56 270)
+		(fields_autoplaced yes)
+		(effects
+			(font
+				(size 1.27 1.27)
+			)
+			(justify right)
+		)
+		(property "Intersheetrefs" "${INTERSHEET_REFS}"
+			(at 265.43 171.6533 90)
+			(hide yes)
+			(show_name no)
+			(do_not_autoplace no)
+			(effects
+				(font
+					(size 1.27 1.27)
+				)
+				(justify right)
+			)
 		)
 	)
@@
 			(hide yes)
 			(show_name no)
+			(do_not_autoplace no)
+			(effects
+				(font
+					(size 1.27 1.27)
+				)
+				(justify right)
+			)
+		)
+	)
+	(global_label "VBUS1"
+		(shape input)
+		(at 265.43 90.17 270)
+		(fields_autoplaced yes)
+		(effects
+			(font
+				(size 1.27 1.27)
+			)
+			(justify right)
+		)
+		(property "Intersheetrefs" "${INTERSHEET_REFS}"
+			(at 265.43 99.2633 90)
+			(hide yes)
+			(show_name no)

Commit message: still cis tho
Parts:
- removed D1, D2: SS54, Diode_SMD:D_SMC, symbol Diode:SS34
- removed R17: 0Ω, Resistor_SMD:R_0402_1005Metric, symbol Device:R
- added C127, C128, C129, C130: 100nF, Capacitor_SMD:C_0402_1005Metric, symbol Device:C
- added Q13, Q14: NCE4009S, Package_SO:SOP-8_3.76x4.96mm_P1.27mm, symbol Transistor_FET:IRF8721PBF-1
- added R102, R103: 0Ω, Resistor_SMD:R_0402_1005Metric, symbol Device:R
- added U17, U18: LM74700QDDF, Package_TO_SOT_SMD:SOT-23-8, symbol Voided-Oblivion-misc:LM74700QDDF
Connections:
- net GND: now also U2.8 (~{OE}), C127.2, C130.2, U17.2 (GND), U18.2 (GND)
- net VBUS: now also Q13.5 (D), Q13.6 (D), Q13.7 (D), Q13.8 (D), Q14.5 (D), Q14.6 (D), Q14.7 (D), Q14.8 (D), U17.8 (CATHODE), U18.8 (CATHODE)
- net VBUS1: now also C129.1, C130.1, Q14.1 (S), Q14.2 (S), Q14.3 (S), R103.1, U18.5 (ANODE)
- net VBUS2: now also C127.1, C128.1, Q13.1 (S), Q13.2 (S), Q13.3 (S), R102.1, U17.5 (ANODE)
- new net: Q13.4 (G), U17.6 (GATE)
- new net: R103.2, U18.1 (EN)
- new net: C129.2, U18.4 (VCAP)
- new net: Q14.4 (G), U18.6 (GATE)
- new net: R102.2, U17.1 (EN)
- new net: C128.2, U17.4 (VCAP)
- no-connect marks 10 -> 14
Other:
- note removed: "~5.73V"
- moved on the sheet: C114, C120, C121, C39, C76, C77, D3, R16, R37, R92, R95, R96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
