File: Voided-Oblivion/keys.kicad_sch (KiCad schematic)
At the start: 162 parts, among them U8 SN74LVC2T45DCUR

Commit message: BOMB update  (ignore the "B" on the end of that first word, it has no significant meaning) and some library linking
Connections:
- no-connect marks 0 -> 2
Changed lines of the file:
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@@
 		(color 0 0 0 0)
+	)
+	(no_connect
+		(at 398.78 30.48)
+	)
+	(no_connect
+		(at 384.81 30.48)
 	)
 	(wire

Commit message: firmware stuff i thinkg a lil bit
Other:
- note added: "Col 0"
- note added: "Col 1"
- note added: "Col 2"
- note added: "Col 3"
- note added: "Col 4"
- note added: "Row 0"
- note added: "Row 1"
- note added: "Row 2"
- note added: "Row 3"
- note added: "Row 4"
- note added: "Row 5"
- note removed: "0,0"
- note removed: "0,1"
- note removed: "0,2"
- note removed: "0,3"
- note removed: "0,4"
- note removed: "0,5"
- note removed: "1,0"
- note removed: "1,1"
- note removed: "1,2"
- note removed: "1,3"
- note removed: "1,4"
- note removed: "1,5"
- note removed: "2,0"
- note removed: "2,1"
- note removed: "2,2"
- note removed: "2,3"
- note removed: "2,4"
- note removed: "2,5"
- note removed: "3,0"
- note removed: "3,1"
- note removed: "3,2"
- note removed: "3,3"
- note removed: "3,4"
- note removed: "3,5"
- note removed: "4,0"
- note removed: "4,1"
- note removed: "4,2"
- note removed: "4,3"
- note removed: "4,4"
- note removed: "4,5"
